File: hardware/project/ETH3CDAQ1/Channel1.sch (KiCad schematic (older format))
At the start: 32 parts, among them U801 DG211, U802 DG419LDY, U803 DG419LDY, U804 AD8251, U805 SN74LVC1G14DBVR, U806 SN74LVC1G14DBVR, U807 ADAQ798x, U808 74HCT595, U809 OPA140, U810 SN74LVC1G14DBVR

Commit message: Schematic design
Parts:
- removed RN801, RN802: 1k, Resistor_THT:R_Array_SIP8, symbol Device:R_Pack04_SIP_Split
- added C701, C702, C703, C704, C705, C706, C707, C708, C709, C710, C712, C713, C714, C715, C717, C718, C719, C720, C722: 100n, Capacitor_SMD:C_0603_1608Metric_Pad1.08x0.95mm_HandSolder, symbol Device:C
- added C711: 330p, Capacitor_SMD:C_0603_1608Metric_Pad1.08x0.95mm_HandSolder, symbol Device:C
- added C716: 100p, Capacitor_SMD:C_0603_1608Metric_Pad1.08x0.95mm_HandSolder, symbol Device:C
- added C721: 1000p, Capacitor_SMD:C_0603_1608Metric_Pad1.08x0.95mm_HandSolder, symbol Device:C
- added C724: 47p, Capacitor_SMD:C_0603_1608Metric_Pad1.08x0.95mm_HandSolder, symbol Device:C
- added D701: MMBZ15VDL, Package_TO_SOT_SMD:SOT-23, symbol Diode:MMBZxx
- added R708, R710: 6k81, Resistor_SMD:R_0603_1608Metric_Pad0.98x0.95mm_HandSolder, symbol Device:R
- added R709: 11k3, Resistor_SMD:R_0603_1608Metric_Pad0.98x0.95mm_HandSolder, symbol Device:R
- added R711, R713: 5k23, Resistor_SMD:R_0603_1608Metric_Pad0.98x0.95mm_HandSolder, symbol Device:R
- added R712: 10k2, Resistor_SMD:R_0603_1608Metric_Pad0.98x0.95mm_HandSolder, symbol Device:R
- added RN701, RN702: 1k, Resistor_SMD:R_Array_Concave_4x0603, symbol Device:R_Pack04_Split
- added U701: LT1355, Package_SO:SOIC-8_3.9x4.9mm_P1.27mm, symbol ETH3CDAQ1:LT1355
- C723: renamed from C802; footprint (none) -> Capacitor_SMD:C_0603_1608Metric_Pad1.08x0.95mm_HandSolder
- C725: renamed from C801; footprint (none) -> Capacitor_SMD:C_0603_1608Metric_Pad1.08x0.95mm_HandSolder
- C726: renamed from C803; footprint (none) -> Capacitor_SMD:C_0603_1608Metric_Pad1.08x0.95mm_HandSolder
- R701: renamed from R?; value R -> 0; footprint (none) -> Resistor_SMD:R_0603_1608Metric_Pad0.98x0.95mm_HandSolder
- R702: renamed from R?; value R -> DNP; footprint (none) -> Resistor_SMD:R_0603_1608Metric_Pad0.98x0.95mm_HandSolder
- R703: renamed from R813; value R -> OPT; footprint (none) -> Resistor_SMD:R_0603_1608Metric_Pad0.98x0.95mm_HandSolder
- R704: renamed from R814; value R -> 0; footprint (none) -> Resistor_SMD:R_0603_1608Metric_Pad0.98x0.95mm_HandSolder
- R705: renamed from R801; footprint (none) -> Resistor_SMD:R_0603_1608Metric_Pad0.98x0.95mm_HandSolder
- R706: renamed from R802; footprint (none) -> Resistor_SMD:R_0603_1608Metric_Pad0.98x0.95mm_HandSolder
- R707: renamed from R803; footprint (none) -> Resistor_SMD:R_0603_1608Metric_Pad0.98x0.95mm_HandSolder
- R714: renamed from R804; value R -> 0; footprint (none) -> Resistor_SMD:R_0603_1608Metric_Pad0.98x0.95mm_HandSolder
- R715: renamed from R805; value R -> DNP; footprint (none) -> Resistor_SMD:R_0603_1608Metric_Pad0.98x0.95mm_HandSolder
- R716: renamed from R806; footprint (none) -> Resistor_SMD:R_0603_1608Metric_Pad0.98x0.95mm_HandSolder
- R717: renamed from R807; footprint (none) -> Resistor_SMD:R_0603_1608Metric_Pad0.98x0.95mm_HandSolder
- R718: renamed from R808; footprint (none) -> Resistor_SMD:R_0603_1608Metric_Pad0.98x0.95mm_HandSolder
- R719: renamed from R809; footprint (none) -> Resistor_SMD:R_0603_1608Metric_Pad0.98x0.95mm_HandSolder
- R720: renamed from R810; footprint (none) -> Resistor_SMD:R_0603_1608Metric_Pad0.98x0.95mm_HandSolder
- R721: renamed from R811; footprint (none) -> Resistor_SMD:R_0603_1608Metric_Pad0.98x0.95mm_HandSolder
- R722: renamed from R812; footprint (none) -> Resistor_SMD:R_0603_1608Metric_Pad0.98x0.95mm_HandSolder
- U702: renamed from U801; footprint (none) -> Package_SO:TSSOP-16_4.4x5mm_P0.65mm
- U704: renamed from U809; footprint (none) -> Package_SO:SOIC-8_3.9x4.9mm_P1.27mm
- U706: renamed from U804; footprint (none) -> Package_SO:MSOP-10_3x3mm_P0.5mm
- U710: renamed from U807; footprint (none) -> ETH3CDAQ1:LGA-24_5x4mm_P0.5mm
- renumbered D801 to D702, U802 to U703, U803 to U705, U805 to U707, U806 to U708, U810 to U709, U808 to U711
Connections:
- net +15V: now also C712.1, C714.1, C717.1, C719.1, C722.1, U701.8 (V+)
- net +5V: now also C702.1, C704.1, C706.1, C708.1, C710.1, C713.1, C715.1, C718.1
- net +5VP: now also RN702.8 (R1.2)
- net -15V: now also C701.1, C703.1, C705.1, C707.1, C709.1, U701.4 (V-)
- net -2V5: now also C720.1
- net GND: now also U711.13 (~OE)
- net GNDA: now also C701.2, C702.2, C703.2, C704.2, C705.2, C706.2, C707.2, C708.2, C709.2, C710.2, C711.2, C712.2, C713.2, C714.2, C715.2, C717.2, C718.2, C719.2, C720.2, C721.2, C722.2, D701.1 (K), RN702.4 (R4.1), U701.3 (+), U701.5 (+)
- net at C725.1, U710.1 (IN+): now also RN702.5 (R4.2), RN702.6 (R3.2), RN702.7 (R2.2)
- net at C726.2, U710.2 (IN-): now also RN701.3 (R3.1), RN701.4 (R4.1), RN701.7 (R2.2)
- net at C726.1, D702.3, U710.3 (AMP_OUT): now also RN701.5 (R4.2), RN701.6 (R3.2)
- net at U706.7 (OUT): now also RN701.1 (R1.1)
- net at U702.14: now also R705.1
- net at U703.8: now also R708.2
- net at U705.8: now also C724.1, R713.1, U701.7
- net SR_CLK: now reaches U711.11 (SRCLK)
- net SR_LAT: now reaches U711.12 (RCLK)
- net SR_DAT: now reaches U711.14 (SER)
- net SR_QH1: now reaches U711.9 (QH')
- net at R703.1, R704.2, U704.2 (-)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: no longer R703.2
- net at R701.1, R702.1, U704.3 (+): now also R703.2, D701.2 (K)
- new net: C716.1, R710.1, R711.2, U701.1
- new net: C716.2, R709.1, U701.2 (-)
- new net: C724.2, R712.1, U701.6 (-)
- new net: C711.1, R708.1, R709.2, R710.2
- new net: RN702.1 (R1.1), RN702.2 (R2.1), RN702.3 (R3.1)
- new net: RN701.2 (R2.1), RN701.8 (R1.2)
- new net: C721.1, R711.1, R712.2, R713.2
- no-connect marks 4 -> 5
Other:
- moved on the sheet: C723, R701, R702, R703, R704, R705, R706, R707, R716, R717, R718, R719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
