File: hardware/project/ETH3CDAQ1/Connector.sch (KiCad schematic (older format))
At the start: 1 part, among them J601 C64AC

Commit message: Schematic design
Parts:
- renumbered J601 to J501
Changed lines of the file:
@@
 $Descr A4 11693 8268
 encoding utf-8
-Sheet 6 9
+Sheet 5 11
 Title "Connector"
 Date "2020-03-07"
@@
 	4900 3850 4950 3850
 $Comp
-L ETH3CDAQ1:GND_TRIG #PWR0605
+L ETH3CDAQ1:GND_TRIG #PWR0505
 U 1 1 5EC065BC
 P 4900 3850
-F 0 "#PWR0605" H 4900 3600 50  0001 C CNN
+F 0 "#PWR0505" H 4900 3600 50  0001 C CNN
 F 1 "GND_TRIG" V 4905 3722 50  0000 R CNN
 F 2 "" H 4900 3850 50  0001 C CNN
@@
 	4850 4200 4900 4200
 $Comp
-L power:Earth #PWR0601
+L power:Earth #PWR0501
 U 1 1 5DED2C4C
 P 4850 4200
-F 0 "#PWR0601" H 4850 3950 50  0001 C CNN
+F 0 "#PWR0501" H 4850 3950 50  0001 C CNN
 F 1 "Earth" H 4850 4050 50  0001 C CNN
 F 2 "" H 4850 4200 50  0001 C CNN
@@
 	4850 5000 4900 5000
 $Comp
-L power:Earth #PWR0602
+L power:Earth #PWR0502
 U 1 1 5DECE77F
 P 4850 5000
-F 0 "#PWR0602" H 4850 4750 50  0001 C CNN
+F 0 "#PWR0502" H 4850 4750 50  0001 C CNN
 F 1 "Earth" H 4850 4850 50  0001 C CNN
 F 2 "" H 4850 5000 50  0001 C CNN
@@
 	4850 6900 4900 6900
 $Comp
-L power:+24V #PWR0604
+L power:+24V #PWR0504
 U 1 1 5DE97137
 P 4850 6900
-F 0 "#PWR0604" H 4850 6750 50  0001 C CNN
+F 0 "#PWR0504" H 4850 6750 50  0001 C CNN
 F 1 "+24V" V 4865 7028 50  0000 L CNN
 F 2 "" H 4850 6900 50  0001 C CNN
@@
 	4950 7050 4900 7050
 $Comp
-L Connector:C64AC J601
+L Connector:C64AC J501
 U 1 1 5DE8758D
 P 5250 3950
-F 0 "J601" H 5430 4046 50  0000 L CNN
+F 0 "J501" H 5430 4046 50  0000 L CNN
 F 1 "C64AC" H 5430 3955 50  0000 L CNN
 F 2 "ETH3CDAQ1:Socket_DIN41612-CaseC1-AC-Male-64Pin-2rows" H 5250 4000 50  0001 C CNN
@@
 NoConn ~ 4950 950
 $Comp
-L power:GND #PWR0603
+L power:GND #PWR0503
 U 1 1 602571EB
 P 4850 6100
-F 0 "#PWR0603" H 4850 5850 50  0001 C CNN
+F 0 "#PWR0503" H 4850 5850 50  0001 C CNN
 F 1 "GND" V 4855 5972 50  0000 R CNN
 F 2 "" H 4850 6100 50  0001 C CNN
