File: hardware/project/ETH3CDAQ1/Ethernet.sch (KiCad schematic (older format))
At the start: 43 parts, among them U201 LAN8742A, U202 LC03-3.3, U203 LC03-3.3, Y201 NX5032GA-25.000M-LN-CD-1

Commit message: Schematic design
Parts:
- C201, C202, C203, C204, C205, C206, C207, C208, C209, C210, C211, C212: footprint Capacitor_SMD:C_0603_1608Metric_Pad1.05x0.95mm_HandSolder -> Capacitor_SMD:C_0603_1608Metric_Pad1.08x0.95mm_HandSolder
- C213, C214: footprint Capacitor_SMD:C_1206_3216Metric_Pad1.42x1.75mm_HandSolder -> Capacitor_SMD:C_1206_3216Metric_Pad1.33x1.80mm_HandSolder
- R201, R202, R203, R204, R205, R206, R207, R208, R209, R210, R211, R212, R213, R214, R215, R216, R217, R218, R220, R221: footprint Resistor_SMD:R_0603_1608Metric_Pad1.05x0.95mm_HandSolder -> Resistor_SMD:R_0603_1608Metric_Pad0.98x0.95mm_HandSolder
- R219: footprint Resistor_SMD:R_1206_3216Metric_Pad1.42x1.75mm_HandSolder -> Resistor_SMD:R_1206_3216Metric_Pad1.30x1.75mm_HandSolder
