File: hardware/project/ETH3CDAQ1/MCU.sch (KiCad schematic (older format))
At the start: 42 parts, among them J501 Conn_02x01, J502 20021111-00010T4LF, U501 HDC1080, U502 STM32H743ZI, U503 24LC08B-E/MS, Y501 NX3225GD-8MHZ-STD-CRA-3

Commit message: Schematic design
Parts:
- removed C505, C507: 8p, Capacitor_SMD:C_0603_1608Metric_Pad1.05x0.95mm_HandSolder, symbol Device:C
- removed C508, C510: 2u2, Capacitor_SMD:C_0805_2012Metric_Pad1.15x1.40mm_HandSolder, symbol Device:C
- added C404, C405: 8p, Capacitor_SMD:C_0603_1608Metric_Pad1.08x0.95mm_HandSolder, symbol Device:C
- added C408, C409: 2u2, Capacitor_SMD:C_0603_1608Metric_Pad1.08x0.95mm_HandSolder, symbol Device:C
- added C411, C413, C415, C417, C419, C421: 100n, Capacitor_SMD:C_0603_1608Metric_Pad1.08x0.95mm_HandSolder, symbol Device:C
- added U402, U403, U404: SN74LVC1T45DBV, Package_TO_SOT_SMD:SOT-23-6, symbol Logic_LevelTranslator:SN74LVC1T45DBV
- C401: renamed from C502; footprint Capacitor_SMD:C_0603_1608Metric_Pad1.05x0.95mm_HandSolder -> Capacitor_SMD:C_0603_1608Metric_Pad1.08x0.95mm_HandSolder
- C402: renamed from C504; footprint Capacitor_SMD:C_0603_1608Metric_Pad1.05x0.95mm_HandSolder -> Capacitor_SMD:C_0603_1608Metric_Pad1.08x0.95mm_HandSolder
- C403: renamed from C506; footprint Capacitor_SMD:C_0603_1608Metric_Pad1.05x0.95mm_HandSolder -> Capacitor_SMD:C_0603_1608Metric_Pad1.08x0.95mm_HandSolder
- C406: renamed from C509; footprint Capacitor_SMD:C_0603_1608Metric_Pad1.05x0.95mm_HandSolder -> Capacitor_SMD:C_0603_1608Metric_Pad1.08x0.95mm_HandSolder
- C407: renamed from C511; footprint Capacitor_SMD:C_0603_1608Metric_Pad1.05x0.95mm_HandSolder -> Capacitor_SMD:C_0603_1608Metric_Pad1.08x0.95mm_HandSolder
- C410: renamed from C512; footprint Capacitor_SMD:C_0603_1608Metric_Pad1.05x0.95mm_HandSolder -> Capacitor_SMD:C_0603_1608Metric_Pad1.08x0.95mm_HandSolder
- C412: renamed from C513; footprint Capacitor_SMD:C_0603_1608Metric_Pad1.05x0.95mm_HandSolder -> Capacitor_SMD:C_0603_1608Metric_Pad1.08x0.95mm_HandSolder
- C414: renamed from C514; footprint Capacitor_SMD:C_0603_1608Metric_Pad1.05x0.95mm_HandSolder -> Capacitor_SMD:C_0603_1608Metric_Pad1.08x0.95mm_HandSolder
- C416: renamed from C515; footprint Capacitor_SMD:C_0603_1608Metric_Pad1.05x0.95mm_HandSolder -> Capacitor_SMD:C_0603_1608Metric_Pad1.08x0.95mm_HandSolder
- C418: renamed from C516; footprint Capacitor_SMD:C_0603_1608Metric_Pad1.05x0.95mm_HandSolder -> Capacitor_SMD:C_0603_1608Metric_Pad1.08x0.95mm_HandSolder
- C420: renamed from C517; footprint Capacitor_SMD:C_0603_1608Metric_Pad1.05x0.95mm_HandSolder -> Capacitor_SMD:C_0603_1608Metric_Pad1.08x0.95mm_HandSolder
- C422: renamed from C518; footprint Capacitor_SMD:C_0603_1608Metric_Pad1.05x0.95mm_HandSolder -> Capacitor_SMD:C_0603_1608Metric_Pad1.08x0.95mm_HandSolder
- C423: renamed from C501; footprint Capacitor_SMD:C_0603_1608Metric_Pad1.05x0.95mm_HandSolder -> Capacitor_SMD:C_0603_1608Metric_Pad1.08x0.95mm_HandSolder
- C424: renamed from C519; footprint Capacitor_SMD:C_0603_1608Metric_Pad1.05x0.95mm_HandSolder -> Capacitor_SMD:C_0603_1608Metric_Pad1.08x0.95mm_HandSolder
- C425: renamed from C503; footprint Capacitor_SMD:C_0603_1608Metric_Pad1.05x0.95mm_HandSolder -> Capacitor_SMD:C_0603_1608Metric_Pad1.08x0.95mm_HandSolder
- C426: renamed from C520; footprint Capacitor_SMD:C_0603_1608Metric_Pad1.05x0.95mm_HandSolder -> Capacitor_SMD:C_0603_1608Metric_Pad1.08x0.95mm_HandSolder
- C427: renamed from C521; footprint Capacitor_SMD:C_0603_1608Metric_Pad1.05x0.95mm_HandSolder -> Capacitor_SMD:C_0603_1608Metric_Pad1.08x0.95mm_HandSolder
- C428: renamed from C522; footprint Capacitor_SMD:C_0603_1608Metric_Pad1.05x0.95mm_HandSolder -> Capacitor_SMD:C_0603_1608Metric_Pad1.08x0.95mm_HandSolder
- R401: renamed from R502; footprint Resistor_SMD:R_0603_1608Metric_Pad1.05x0.95mm_HandSolder -> Resistor_SMD:R_0603_1608Metric_Pad0.98x0.95mm_HandSolder
- R402: renamed from R503; footprint Resistor_SMD:R_0603_1608Metric_Pad1.05x0.95mm_HandSolder -> Resistor_SMD:R_0603_1608Metric_Pad0.98x0.95mm_HandSolder
- R403: renamed from R504; footprint Resistor_SMD:R_0603_1608Metric_Pad1.05x0.95mm_HandSolder -> Resistor_SMD:R_0603_1608Metric_Pad0.98x0.95mm_HandSolder
- R404: renamed from R505; footprint Resistor_SMD:R_0603_1608Metric_Pad1.05x0.95mm_HandSolder -> Resistor_SMD:R_0603_1608Metric_Pad0.98x0.95mm_HandSolder
- R405: renamed from R506; footprint Resistor_SMD:R_0603_1608Metric_Pad1.05x0.95mm_HandSolder -> Resistor_SMD:R_0603_1608Metric_Pad0.98x0.95mm_HandSolder
- R406: renamed from R507; footprint Resistor_SMD:R_0603_1608Metric_Pad1.05x0.95mm_HandSolder -> Resistor_SMD:R_0603_1608Metric_Pad0.98x0.95mm_HandSolder
- R407: renamed from R508; footprint Resistor_SMD:R_0603_1608Metric_Pad1.05x0.95mm_HandSolder -> Resistor_SMD:R_0603_1608Metric_Pad0.98x0.95mm_HandSolder
- R408: renamed from R509; footprint Resistor_SMD:R_0603_1608Metric_Pad1.05x0.95mm_HandSolder -> Resistor_SMD:R_0603_1608Metric_Pad0.98x0.95mm_HandSolder
- R409: renamed from R510; footprint Resistor_SMD:R_0603_1608Metric_Pad1.05x0.95mm_HandSolder -> Resistor_SMD:R_0603_1608Metric_Pad0.98x0.95mm_HandSolder
- R410: renamed from R501; footprint Resistor_SMD:R_0603_1608Metric_Pad1.05x0.95mm_HandSolder -> Resistor_SMD:R_0603_1608Metric_Pad0.98x0.95mm_HandSolder
- Y401: renamed from Y501; value NX3225GD-8MHZ-STD-CRA-3 -> NX3225GD-8MHZ
- renumbered D501 to D401, D502 to D402, D503 to D403, FB501 to FB401, J502 to J401, J501 to J402, U501 to U401, U502 to U405, U503 to U406
Connections:
- net +3V3: now also C417.1, C419.1, C421.1, U402.6 (VCCB), U403.6 (VCCB), U404.6 (VCCB)
- net TRIG_EN: now also U405.73 (PB12,TIM1_BKIN,I2C2_SMBA,SPI2_NSS,I2S2_WS,DFSDM1_DATIN1,USART3_CK,UART5_RX,CAN2_RX,OTG_HS_ULPI_D5,ETH_MII_TXD0,ETH_RMII_TXD0,OTG_HS_ID,EVENTOUT); no longer U405.75 (PB14,TIM1_CH2N,TIM8_CH2N,USART1_TX,SPI2_MISO,DFSDM1_DATIN2,USART3_RTS,UART4_RTS,TIM12_CH1,SDMMC2_D0,OTG_HS_DM,EVENTOUT)
- net TRIG_IN: now also U405.69 (PB10,TIM2_CH3,I2C2_SCL,SPI2_SCK,I2S2_CK,DFSDM1_DATIN7,USART3_TX,QUADSPI_BK1_NCS,OTG_HS_ULPI_D3,ETH_MII_RX_ER,LCD_G4,EVENTOUT); no longer U405.73 (PB12,TIM1_BKIN,I2C2_SMBA,SPI2_NSS,I2S2_WS,DFSDM1_DATIN1,USART3_CK,UART5_RX,CAN2_RX,OTG_HS_ULPI_D5,ETH_MII_TXD0,ETH_RMII_TXD0,OTG_HS_ID,EVENTOUT)
- net TRIG_OUT: now also U405.70 (PB11,TIM2_CH4,I2C2_SDA,DFSDM1_CKIN7,USART3_RX,OTG_HS_ULPI_D4,ETH_MII_TX_EN,ETH_RMII_TX_EN,_DSI_TE,LCD_G5,EVENTOUT); no longer U405.74 (PB13,TIM1_CH1N,SPI2_SCK,I2S2_CK,DFSDM1_CKIN1,USART3_CTS,UART5_TX,CAN2_TX,OTG_HS_ULPI_D6,ETH_MII_TXD1,ETH_RMII_TXD1,EVENTOUT,OTG_HS_VBUS)
- net at U405.106 (VCAP_2): now also C409.1
- net at U405.71 (VCAP_1): now also C408.1
- net at U405.23 (PH0,EVENTOUT,OSC_IN), Y401.1: now also C404.1
- net at U405.24 (PH1,EVENTOUT,OSC_OUT), Y401.2: now also C405.1
- net MCU_CNV: now reaches U405.110 (PA15,JTDI,TIM2_CH1,TIM2_ETR,HDMI_CEC,SPI1_NSS,I2S1_WS,SPI3_NSS,I2S3_WS,SPI6_NSS,UART4_RTS,CAN3_TX,UART7_TX,EVENTOUT)
- net MCU_CLK: now reaches U405.111 (PC10,DFSDM1_CKIN5,SPI3_SCK,I2S3_CK,USART3_TX,UART4_TX,QUADSPI_BK1_IO1,SDMMC1_D2,DCMI_D8,LCD_R2,EVENTOUT)
- net MCU_MISO: now reaches U405.112 (PC11,DFSDM1_DATIN5,SPI3_MISO,USART3_RX,UART4_RX,QUADSPI_BK2_NCS,SDMMC1_D3,DCMI_D4,EVENTOUT)
- net MCU_~CS1: now reaches U405.116 (PD2,TRACED2,TIM3_ETR,UART5_RX,SDMMC1_CMD,DCMI_D11,EVENTOUT)
- net MCU_~CS2: now reaches U405.117 (PD3,DFSDM1_CKOUT,SPI2_SCK,I2S2_CK,DFSDM1_DATIN0,USART2_CTS,FMC_CLK,DCMI_D5,LCD_G7,EVENTOUT)
- net MCU_~CS3: now reaches U405.118 (PD4,DFSDM1_CKIN0,USART2_RTS,FMC_NOE,EVENTOUT)
- net at U405.46 (PB0,TIM1_CH2N,TIM3_CH3,TIM8_CH2N,DFSDM1_CKOUT,UART4_CTS,_LCD_R3,OTG_HS_ULPI_D1,ETH_MII_RXD2,LCD_G1,EVENTOUT,ADC1_IN8,ADC2_IN8): now also J402.1 (Pin_1), R410.1
- net MCU_SR_DAT: now reaches U405.96 (PC6,TIM3_CH1,TIM8_CH1,I2S2_MCK,DFSDM1_CKIN3,USART6_TX,FMC_NWAIT,SDMMC2_D6,SDMMC1_D6,DCMI_D0,LCD_HSYNC,EVENTOUT)
- net MCU_SR_DAT: now also U402.4 (B)
- net MCU_SR_CLK: now reaches U405.97 (PC7,TIM3_CH2,TIM8_CH2,I2S3_MCK,DFSDM1_DATIN3,USART6_RX,FMC_NE1,SDMMC2_D7,SDMMC1_D7,DCMI_D1,LCD_G6,EVENTOUT)
- net MCU_SR_CLK: now also U403.4 (B)
- net MCU_SR_LAT: now reaches U405.98 (PC8,TRACED1,TIM3_CH3,TIM8_CH3,UART5_RTS,USART6_CK,FMC_NE2,FMC_NCE,SDMMC1_D0,DCMI_D2,EVENTOUT)
- net MCU_SR_LAT: now also U404.4 (B)
- net DGNDF renamed GND
- net GND: now also C404.2, C405.2, C408.2, C409.2, C411.2, C413.2, C415.2, C417.2, C419.2, C421.2, U402.2 (GND), U402.5 (DIR), U403.2 (GND), U403.5 (DIR), U404.2 (GND), U404.5 (DIR)
- removed net MCU_DEFAULT: J402.1 (Pin_1), R410.1, U405.34 (PA0,TIM2_CH1,TIM2_ETR,TIM5_CH1,TIM8_ETR,USART2_CTS,UART4_TX,SAI2_SD_B,ETH_MII_CRS,EVENTOUT,ADC1_IN0,ADC2_IN0,ADC3_IN0,WKUP1)
- new net +5V: C411.1, C413.1, C415.1, U402.1 (VCCA), U403.1 (VCCA), U404.1 (VCCA)
- new net SD_CLK: U403.3 (A)
- new net SD_DAT: U402.3 (A)
- new net SD_LAT: U404.3 (A)
- no-connect marks 55 -> 46
Other:
- moved on the sheet: C401, C402, C403, C406, C407, C410, C412, C414, C416, C418, C420, C422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
