File: hardware/project/ETH3CDAQ1/Power.sch (KiCad schematic (older format))
At the start: 113 parts, among them Q701 IRFR5410, U701 LT8330_S6, U702 LT8330_S6, U703 LT8330_S6, U704 LT8330_S6, U705 ADP7118_LFCSP6, U706 ADP7182_LFCSP6, U707 ADP7118_LFCSP6, U708 ADP7182_LFCSP6, U709 MAX5902, U710 ADP7118_LFCSP6, U711 TSR1-2490, U712 TSR1-2450, U713 LM1117DTX-5.0/NOPB, U714 LM1117DTX-3.3/NOPB

Commit message: Schematic design
Parts:
- removed C703, C704, C731, C732: 10u/50V, Capacitor_SMD:C_1206_3216Metric_Pad1.42x1.75mm_HandSolder, symbol Device:C
- removed C707, C708, C723, C724, C727, C728: 4u7/50V, Capacitor_SMD:C_1206_3216Metric_Pad1.42x1.75mm_HandSolder, symbol Device:C
- removed C711, C712: 1u, Capacitor_SMD:C_0603_1608Metric_Pad1.05x0.95mm_HandSolder, symbol Device:C
- removed C715, C716: 1u/HC, Capacitor_SMD:C_1206_3216Metric_Pad1.42x1.75mm_HandSolder, symbol Device:C
- removed C719, C720: 4p7, Capacitor_SMD:C_0603_1608Metric_Pad1.05x0.95mm_HandSolder, symbol Device:C
- removed C735, C736: 100n, symbol Device:C
- removed C739, C740: 10u/35V, Capacitor_SMD:C_1206_3216Metric_Pad1.42x1.75mm_HandSolder, symbol Device:C
- removed C750, C751: 10u/16V, Capacitor_SMD:C_1206_3216Metric_Pad1.42x1.75mm_HandSolder, symbol Device:C
- removed D702, D704: PMEG6010EP,115, Diode_SMD:D_SOD-128, symbol Device:D_Schottky
- removed L703, L704: 74489440068, ETH3CDAQ1:74489440068, symbol ETH3CDAQ1:74489440068
- removed R705, R707, R713, R715: 1M, Resistor_SMD:R_0603_1608Metric_Pad1.05x0.95mm_HandSolder, symbol Device:R
- removed R706, R708: 287k, Resistor_SMD:R_0603_1608Metric_Pad1.05x0.95mm_HandSolder, symbol Device:R
- removed R714: 111k, Resistor_SMD:R_0603_1608Metric_Pad1.05x0.95mm_HandSolder, symbol Device:R
- removed R716: 53k, Resistor_SMD:R_0603_1608Metric_Pad1.05x0.95mm_HandSolder, symbol Device:R
- removed R721: 100k, symbol Device:R
- removed R722: 49k9, symbol Device:R
- removed R723: 150k, symbol Device:R
- removed R724: 13k3, symbol Device:R
- removed R727, R728: R, symbol Device:R
- removed U703, U704: LT8330_S6, Package_TO_SOT_SMD:TSOT-23-6_HandSoldering, symbol ETH3CDAQ1:LT8330_S6
- removed U707: ADP7118_LFCSP6, symbol ETH3CDAQ1:ADP7118_LFCSP6
- removed U708: ADP7182_LFCSP6, symbol ETH3CDAQ1:ADP7182_LFCSP6
- removed U711: TSR1-2490, ETH3CDAQ1:TSR1, symbol ETH3CDAQ1:TSR1-2450
- removed U713: LM1117DTX-5.0/NOPB, Package_TO_SOT_SMD:TO-252-2, symbol Regulator_Linear:LM1117-3.3
- removed U714: LM1117DTX-3.3/NOPB, Package_TO_SOT_SMD:TO-252-2, symbol Regulator_Linear:LM1117-3.3
- added C624: 10u, Capacitor_SMD:C_1206_3216Metric_Pad1.33x1.80mm_HandSolder, symbol Device:C
- added C629: 4u7, Capacitor_SMD:C_1206_3216Metric_Pad1.33x1.80mm_HandSolder, symbol Device:C
- added U607: ADP7182-2V5_LFCSP6, ETH3CDAQ1:LFCSP-6_2x2mm_1EP_P0.65mm, symbol ETH3CDAQ1:ADP7182-2V5_LFCSP6
- added U608: TSR1-2433, ETH3CDAQ1:TSR1, symbol ETH3CDAQ1:TSR1-2450
- C601: renamed from C701; footprint Capacitor_SMD:C_1206_3216Metric_Pad1.42x1.75mm_HandSolder -> Capacitor_SMD:C_1206_3216Metric_Pad1.33x1.80mm_HandSolder
- C602: renamed from C702; footprint Capacitor_SMD:C_1206_3216Metric_Pad1.42x1.75mm_HandSolder -> Capacitor_SMD:C_1206_3216Metric_Pad1.33x1.80mm_HandSolder
- C603: renamed from C705; footprint Capacitor_SMD:C_1206_3216Metric_Pad1.42x1.75mm_HandSolder -> Capacitor_SMD:C_1206_3216Metric_Pad1.33x1.80mm_HandSolder
- C604: renamed from C706; footprint Capacitor_SMD:C_1206_3216Metric_Pad1.42x1.75mm_HandSolder -> Capacitor_SMD:C_1206_3216Metric_Pad1.33x1.80mm_HandSolder
- C605: renamed from C709; footprint Capacitor_SMD:C_0603_1608Metric_Pad1.05x0.95mm_HandSolder -> Capacitor_SMD:C_0603_1608Metric_Pad1.08x0.95mm_HandSolder
- C606: renamed from C710; footprint Capacitor_SMD:C_0603_1608Metric_Pad1.05x0.95mm_HandSolder -> Capacitor_SMD:C_0603_1608Metric_Pad1.08x0.95mm_HandSolder
- C607: renamed from C713; footprint Capacitor_SMD:C_1206_3216Metric_Pad1.42x1.75mm_HandSolder -> Capacitor_SMD:C_1206_3216Metric_Pad1.33x1.80mm_HandSolder
- C608: renamed from C714; footprint Capacitor_SMD:C_1206_3216Metric_Pad1.42x1.75mm_HandSolder -> Capacitor_SMD:C_1206_3216Metric_Pad1.33x1.80mm_HandSolder
- C609: renamed from C717; footprint Capacitor_SMD:C_0603_1608Metric_Pad1.05x0.95mm_HandSolder -> Capacitor_SMD:C_0603_1608Metric_Pad1.08x0.95mm_HandSolder
- C610: renamed from C718; footprint Capacitor_SMD:C_0603_1608Metric_Pad1.05x0.95mm_HandSolder -> Capacitor_SMD:C_0603_1608Metric_Pad1.08x0.95mm_HandSolder
- C611: renamed from C721; footprint Capacitor_SMD:C_1206_3216Metric_Pad1.42x1.75mm_HandSolder -> Capacitor_SMD:C_1206_3216Metric_Pad1.33x1.80mm_HandSolder
- C612: renamed from C722; footprint Capacitor_SMD:C_1206_3216Metric_Pad1.42x1.75mm_HandSolder -> Capacitor_SMD:C_1206_3216Metric_Pad1.33x1.80mm_HandSolder
- C613: renamed from C725; footprint Capacitor_SMD:C_1206_3216Metric_Pad1.42x1.75mm_HandSolder -> Capacitor_SMD:C_1206_3216Metric_Pad1.33x1.80mm_HandSolder
- C614: renamed from C726; footprint Capacitor_SMD:C_1206_3216Metric_Pad1.42x1.75mm_HandSolder -> Capacitor_SMD:C_1206_3216Metric_Pad1.33x1.80mm_HandSolder
- C615: renamed from C729; footprint Capacitor_SMD:C_1206_3216Metric_Pad1.42x1.75mm_HandSolder -> Capacitor_SMD:C_1206_3216Metric_Pad1.33x1.80mm_HandSolder
- C616: renamed from C730; footprint Capacitor_SMD:C_1206_3216Metric_Pad1.42x1.75mm_HandSolder -> Capacitor_SMD:C_1206_3216Metric_Pad1.33x1.80mm_HandSolder
- C617: renamed from C733; footprint (none) -> Capacitor_SMD:C_0603_1608Metric_Pad1.08x0.95mm_HandSolder
- C618: renamed from C734; footprint (none) -> Capacitor_SMD:C_0603_1608Metric_Pad1.08x0.95mm_HandSolder
- C619: renamed from C737; footprint Capacitor_SMD:C_1206_3216Metric_Pad1.42x1.75mm_HandSolder -> Capacitor_SMD:C_1206_3216Metric_Pad1.33x1.80mm_HandSolder
- C620: renamed from C738; footprint Capacitor_SMD:C_1206_3216Metric_Pad1.42x1.75mm_HandSolder -> Capacitor_SMD:C_1206_3216Metric_Pad1.33x1.80mm_HandSolder
- C621: renamed from C743; footprint Capacitor_SMD:C_1206_3216Metric_Pad1.42x1.75mm_HandSolder -> Capacitor_SMD:C_1206_3216Metric_Pad1.33x1.80mm_HandSolder
- C622: renamed from C742; footprint Capacitor_SMD:C_1206_3216Metric_Pad1.42x1.75mm_HandSolder -> Capacitor_SMD:C_1206_3216Metric_Pad1.33x1.80mm_HandSolder
- C623: renamed from C741; value 4u7/16V -> 4u7/25V; footprint Capacitor_SMD:C_1206_3216Metric_Pad1.42x1.75mm_HandSolder -> Capacitor_SMD:C_1206_3216Metric_Pad1.33x1.80mm_HandSolder
- C625: renamed from C745; footprint Capacitor_SMD:C_1206_3216Metric_Pad1.42x1.75mm_HandSolder -> Capacitor_SMD:C_1206_3216Metric_Pad1.33x1.80mm_HandSolder
- C626: renamed from C744; footprint Capacitor_SMD:C_1206_3216Metric_Pad1.42x1.75mm_HandSolder -> Capacitor_SMD:C_1206_3216Metric_Pad1.33x1.80mm_HandSolder
- C627: renamed from C746; footprint Capacitor_SMD:C_1206_3216Metric_Pad1.42x1.75mm_HandSolder -> Capacitor_SMD:C_1206_3216Metric_Pad1.33x1.80mm_HandSolder
- C628: renamed from C747; footprint Capacitor_SMD:C_1206_3216Metric_Pad1.42x1.75mm_HandSolder -> Capacitor_SMD:C_1206_3216Metric_Pad1.33x1.80mm_HandSolder
- C630: renamed from C748; footprint (none) -> Capacitor_SMD:C_0603_1608Metric_Pad1.08x0.95mm_HandSolder
- C631: renamed from C749; footprint Capacitor_SMD:C_1206_3216Metric_Pad1.42x1.75mm_HandSolder -> Capacitor_SMD:C_1206_3216Metric_Pad1.33x1.80mm_HandSolder
- R601: renamed from R701; footprint Resistor_SMD:R_0603_1608Metric_Pad1.05x0.95mm_HandSolder -> Resistor_SMD:R_0603_1608Metric_Pad0.98x0.95mm_HandSolder
- R602: renamed from R702; footprint Resistor_SMD:R_0603_1608Metric_Pad1.05x0.95mm_HandSolder -> Resistor_SMD:R_0603_1608Metric_Pad0.98x0.95mm_HandSolder
- R603: renamed from R703; footprint Resistor_SMD:R_0603_1608Metric_Pad1.05x0.95mm_HandSolder -> Resistor_SMD:R_0603_1608Metric_Pad0.98x0.95mm_HandSolder
- R604: renamed from R704; footprint Resistor_SMD:R_0603_1608Metric_Pad1.05x0.95mm_HandSolder -> Resistor_SMD:R_0603_1608Metric_Pad0.98x0.95mm_HandSolder
- R605: renamed from R729; footprint (none) -> Resistor_SMD:R_0603_1608Metric_Pad0.98x0.95mm_HandSolder
- R606: renamed from R709; footprint Resistor_SMD:R_0603_1608Metric_Pad1.05x0.95mm_HandSolder -> Resistor_SMD:R_0603_1608Metric_Pad0.98x0.95mm_HandSolder
- R607: renamed from R710; footprint Resistor_SMD:R_0603_1608Metric_Pad1.05x0.95mm_HandSolder -> Resistor_SMD:R_0603_1608Metric_Pad0.98x0.95mm_HandSolder
- R608: renamed from R711; footprint Resistor_SMD:R_0603_1608Metric_Pad1.05x0.95mm_HandSolder -> Resistor_SMD:R_0603_1608Metric_Pad0.98x0.95mm_HandSolder
- R609: renamed from R712; footprint Resistor_SMD:R_0603_1608Metric_Pad1.05x0.95mm_HandSolder -> Resistor_SMD:R_0603_1608Metric_Pad0.98x0.95mm_HandSolder
- R610: renamed from R733; footprint Resistor_SMD:R_0603_1608Metric_Pad1.05x0.95mm_HandSolder -> Resistor_SMD:R_0603_1608Metric_Pad0.98x0.95mm_HandSolder
- R611: renamed from R717; footprint (none) -> Resistor_SMD:R_0603_1608Metric_Pad0.98x0.95mm_HandSolder
- R612: renamed from R718; footprint (none) -> Resistor_SMD:R_0603_1608Metric_Pad0.98x0.95mm_HandSolder
- R613: renamed from R719; footprint (none) -> Resistor_SMD:R_0603_1608Metric_Pad0.98x0.95mm_HandSolder
- R614: renamed from R720; footprint (none) -> Resistor_SMD:R_0603_1608Metric_Pad0.98x0.95mm_HandSolder
- R615: renamed from R725; footprint (none) -> Resistor_SMD:R_0603_1608Metric_Pad0.98x0.95mm_HandSolder
- R616: renamed from R726; footprint (none) -> Resistor_SMD:R_0603_1608Metric_Pad0.98x0.95mm_HandSolder
- R617: renamed from R730; footprint (none) -> Resistor_SMD:R_0603_1608Metric_Pad0.98x0.95mm_HandSolder
- R618: renamed from R731; footprint (none) -> Resistor_SMD:R_0603_1608Metric_Pad0.98x0.95mm_HandSolder
- R619: renamed from R732; footprint (none) -> Resistor_SMD:R_0603_1608Metric_Pad0.98x0.95mm_HandSolder
- U603: renamed from U709; footprint (none) -> Package_TO_SOT_SMD:SOT-23-6_Handsoldering
- U604: renamed from U705; footprint (none) -> ETH3CDAQ1:LFCSP-6_2x2mm_1EP_P0.65mm
- U605: renamed from U706; footprint (none) -> ETH3CDAQ1:LFCSP-6_2x2mm_1EP_P0.65mm
- U606: renamed from U710; footprint (none) -> ETH3CDAQ1:LFCSP-6_2x2mm_1EP_P0.65mm
- renumbered D705 to D601, D701 to D602, D703 to D603, D706 to D604, D707 to D605, F701 to F601, L701 to L601, L702 to L602, L706 to L603, L705 to L604, Q701 to Q601, U701 to U601, U702 to U602, U712 to U609
Connections:
- net +3V3: now also C627.1, U608.3 (VO)
- net +5V: now also C628.1, U609.3 (VO)
- net +9V: no longer C627.1
- net GND: now also D602.1 (K), C624.2, C629.2, U607.5 (GND), U608.2 (GND)
- net at C625.1, L603.2: now also U608.1 (VI)
- net DGNDF: no longer names the net of L601.3
- net DGNDF: no longer D602.1 (K)
- new net -2V5: C629.1, U607.1 (VOUT)
- new net -5V: C624.1, U607.3 (EN), U607.6 (VIN), U607.7 (PAD)
- no-connect marks 4 -> 3
Other:
- moved on the sheet: C601, C602, C603, C604, C605, C606, C607, C608, C609, C610, C611, C612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
