File: hardware/project/ETH3CDAQ1/SDRAM.sch (KiCad schematic (older format))
At the start: 8 parts, among them U301 IS42S16400J-xC

Commit message: Schematic design
Parts:
- C1001: renamed from C301; footprint Capacitor_SMD:C_0603_1608Metric_Pad1.05x0.95mm_HandSolder -> Capacitor_SMD:C_0603_1608Metric_Pad1.08x0.95mm_HandSolder
- C1002: renamed from C302; footprint Capacitor_SMD:C_0603_1608Metric_Pad1.05x0.95mm_HandSolder -> Capacitor_SMD:C_0603_1608Metric_Pad1.08x0.95mm_HandSolder
- C1003: renamed from C303; footprint Capacitor_SMD:C_0603_1608Metric_Pad1.05x0.95mm_HandSolder -> Capacitor_SMD:C_0603_1608Metric_Pad1.08x0.95mm_HandSolder
- C1004: renamed from C304; footprint Capacitor_SMD:C_0603_1608Metric_Pad1.05x0.95mm_HandSolder -> Capacitor_SMD:C_0603_1608Metric_Pad1.08x0.95mm_HandSolder
- C1005: renamed from C305; footprint Capacitor_SMD:C_0603_1608Metric_Pad1.05x0.95mm_HandSolder -> Capacitor_SMD:C_0603_1608Metric_Pad1.08x0.95mm_HandSolder
- C1006: renamed from C306; footprint Capacitor_SMD:C_0603_1608Metric_Pad1.05x0.95mm_HandSolder -> Capacitor_SMD:C_0603_1608Metric_Pad1.08x0.95mm_HandSolder
- C1007: renamed from C307; footprint Capacitor_SMD:C_0603_1608Metric_Pad1.05x0.95mm_HandSolder -> Capacitor_SMD:C_0603_1608Metric_Pad1.08x0.95mm_HandSolder
- renumbered U301 to U1001
Changed lines of the file:
@@
 $Descr A4 11693 8268
 encoding utf-8
-Sheet 3 9
+Sheet 10 11
 Title "SDRAM"
 Date "2020-03-07"
@@
 $EndDescr
 $Comp
-L Memory_RAM:IS42S16400J-xC U301
+L Memory_RAM:IS42S16400J-xC U1001
 U 1 1 5EB98CAA
 P 5650 3200
-F 0 "U301" H 6400 4600 50  0000 C CNN
+F 0 "U1001" H 6400 4600 50  0000 C CNN
 F 1 "IS42S16400J-xC" H 6400 4500 50  0000 C CNN
 F 2 "ETH3CDAQ1:TSSOP-54" H 5650 3200 50  0001 C CNN
@@
 D[0..15]
 $Comp
-L Device:C C301
+L Device:C C1001
 U 1 1 5F12988C
 P 1000 7250
-F 0 "C301" H 1115 7296 50  0000 L CNN
+F 0 "C1001" H 1115 7296 50  0000 L CNN
 F 1 "100n" H 1115 7205 50  0000 L CNN
-F 2 "Capacitor_SMD:C_0603_1608Metric_Pad1.05x0.95mm_HandSolder" H 1038 7100 50  0001 C CNN
+F 2 "Capacitor_SMD:C_0603_1608Metric_Pad1.08x0.95mm_HandSolder" H 1038 7100 50  0001 C CNN
 F 3 "~" H 1000 7250 50  0001 C CNN
 	1    1000 7250
@@
 $EndComp
 $Comp
-L Device:C C302
+L Device:C C1002
 U 1 1 5F12BD5A
 P 1500 7250
-F 0 "C302" H 1615 7296 50  0000 L CNN
+F 0 "C1002" H 1615 7296 50  0000 L CNN
 F 1 "100n" H 1615 7205 50  0000 L CNN
-F 2 "Capacitor_SMD:C_0603_1608Metric_Pad1.05x0.95mm_HandSolder" H 1538 7100 50  0001 C CNN
+F 2 "Capacitor_SMD:C_0603_1608Metric_Pad1.08x0.95mm_HandSolder" H 1538 7100 50  0001 C CNN
 F 3 "~" H 1500 7250 50  0001 C CNN
 	1    1500 7250
@@
 $EndComp
 $Comp
-L Device:C C303
+L Device:C C1003
 U 1 1 5F12CAA5
 P 2000 7250
-F 0 "C303" H 2115 7296 50  0000 L CNN
+F 0 "C1003" H 2115 7296 50  0000 L CNN
 F 1 "100n" H 2115 7205 50  0000 L CNN
-F 2 "Capacitor_SMD:C_0603_1608Metric_Pad1.05x0.95mm_HandSolder" H 2038 7100 50  0001 C CNN
+F 2 "Capacitor_SMD:C_0603_1608Metric_Pad1.08x0.95mm_HandSolder" H 2038 7100 50  0001 C CNN
 F 3 "~" H 2000 7250 50  0001 C CNN
 	1    2000 7250
@@
 $EndComp
 $Comp
-L Device:C C304
+L Device:C C1004
 U 1 1 5F12CAAB
 P 2500 7250
-F 0 "C304" H 2615 7296 50  0000 L CNN
+F 0 "C1004" H 2615 7296 50  0000 L CNN
 F 1 "100n" H 2615 7205 50  0000 L CNN
-F 2 "Capacitor_SMD:C_0603_1608Metric_Pad1.05x0.95mm_HandSolder" H 2538 7100 50  0001 C CNN
+F 2 "Capacitor_SMD:C_0603_1608Metric_Pad1.08x0.95mm_HandSolder" H 2538 7100 50  0001 C CNN
 F 3 "~" H 2500 7250 50  0001 C CNN
 	1    2500 7250
@@
 $EndComp
 $Comp
-L Device:C C305
+L Device:C C1005
 U 1 1 5F12F1B4
 P 3000 7250
-F 0 "C305" H 3115 7296 50  0000 L CNN
+F 0 "C1005" H 3115 7296 50  0000 L CNN
 F 1 "100n" H 3115 7205 50  0000 L CNN
-F 2 "Capacitor_SMD:C_0603_1608Metric_Pad1.05x0.95mm_HandSolder" H 3038 7100 50  0001 C CNN
+F 2 "Capacitor_SMD:C_0603_1608Metric_Pad1.08x0.95mm_HandSolder" H 3038 7100 50  0001 C CNN
 F 3 "~" H 3000 7250 50  0001 C CNN
 	1    3000 7250
@@
 $EndComp
 $Comp
-L Device:C C306
+L Device:C C1006
 U 1 1 5F12F1BA
 P 3500 7250
-F 0 "C306" H 3615 7296 50  0000 L CNN
+F 0 "C1006" H 3615 7296 50  0000 L CNN
 F 1 "100n" H 3615 7205 50  0000 L CNN
-F 2 "Capacitor_SMD:C_0603_1608Metric_Pad1.05x0.95mm_HandSolder" H 3538 7100 50  0001 C CNN
+F 2 "Capacitor_SMD:C_0603_1608Metric_Pad1.08x0.95mm_HandSolder" H 3538 7100 50  0001 C CNN
 F 3 "~" H 3500 7250 50  0001 C CNN
 	1    3500 7250
@@
 $EndComp
 $Comp
-L Device:C C307
+L Device:C C1007
 U 1 1 5F12F1C0
 P 4000 7250
-F 0 "C307" H 4115 7296 50  0000 L CNN
+F 0 "C1007" H 4115 7296 50  0000 L CNN
 F 1 "100n" H 4115 7205 50  0000 L CNN
-F 2 "Capacitor_SMD:C_0603_1608Metric_Pad1.05x0.95mm_HandSolder" H 4038 7100 50  0001 C CNN
+F 2 "Capacitor_SMD:C_0603_1608Metric_Pad1.08x0.95mm_HandSolder" H 4038 7100 50  0001 C CNN
 F 3 "~" H 4000 7250 50  0001 C CNN
 	1    4000 7250
@@
 Wire Wire Line
 	2500 7000 2500 7050
+$Comp
+L power:GND #PWR01002
+U 1 1 6038237F
+P 2500 7500
+F 0 "#PWR01002" H 2500 7250 50  0001 C CNN
+F 1 "GND" H 2505 7327 50  0000 C CNN
+F 2 "" H 2500 7500 50  0001 C CNN
+F 3 "" H 2500 7500 50  0001 C CNN
+	1    2500 7500
+	1    0    0    -1
+$EndComp
+$Comp
+L power:GND #PWR01004
+U 1 1 603828AC
+P 5650 4700
+F 0 "#PWR01004" H 5650 4450 50  0001 C CNN
+F 1 "GND" H 5655 4527 50  0000 C CNN
+F 2 "" H 5650 4700 50  0001 C CNN
+F 3 "" H 5650 4700 50  0001 C CNN
+	1    5650 4700
+	1    0    0    -1
+$EndComp
+$Comp
+L power:+3.3V #PWR01003
+U 1 1 60383841
+P 5650 1700
+F 0 "#PWR01003" H 5650 1550 50  0001 C CNN
+F 1 "+3.3V" H 5665 1873 50  0000 C CNN
+F 2 "" H 5650 1700 50  0001 C CNN
+F 3 "" H 5650 1700 50  0001 C CNN
+	1    5650 1700
+	1    0    0    -1
+$EndComp
+$Comp
+L power:+3.3V #PWR01001
+U 1 1 60384354
+P 2500 7000
+F 0 "#PWR01001" H 2500 6850 50  0001 C CNN
+F 1 "+3.3V" H 2515 7173 50  0000 C CNN
+F 2 "" H 2500 7000 50  0001 C CNN
+F 3 "" H 2500 7000 50  0001 C CNN
+	1    2500 7000
+	1    0    0    -1
+$EndComp
 Wire Bus Line
 	4500 2200 4500 3500
 Wire Bus Line
 	6800 2100 6800 3700
-$Comp
-L power:GND #PWR0302
-U 1 1 6038237F
-P 2500 7500
-F 0 "#PWR0302" H 2500 7250 50  0001 C CNN
-F 1 "GND" H 2505 7327 50  0000 C CNN
-F 2 "" H 2500 7500 50  0001 C CNN
-F 3 "" H 2500 7500 50  0001 C CNN
-	1    2500 7500
-	1    0    0    -1
-$EndComp
-$Comp
-L power:GND #PWR0304
-U 1 1 603828AC
-P 5650 4700
-F 0 "#PWR0304" H 5650 4450 50  0001 C CNN
-F 1 "GND" H 5655 4527 50  0000 C CNN
-F 2 "" H 5650 4700 50  0001 C CNN
-F 3 "" H 5650 4700 50  0001 C CNN
-	1    5650 4700
-	1    0    0    -1
-$EndComp
-$Comp
-L power:+3.3V #PWR0303
-U 1 1 60383841
-P 5650 1700
-F 0 "#PWR0303" H 5650 1550 50  0001 C CNN
-F 1 "+3.3V" H 5665 1873 50  0000 C CNN
-F 2 "" H 5650 1700 50  0001 C CNN
-F 3 "" H 5650 1700 50  0001 C CNN
-	1    5650 1700
-	1    0    0    -1
-$EndComp
-$Comp
-L power:+3.3V #PWR0301
-U 1 1 60384354
-P 2500 7000
-F 0 "#PWR0301" H 2500 6850 50  0001 C CNN
-F 1 "+3.3V" H 2515 7173 50  0000 C CNN
-F 2 "" H 2500 7000 50  0001 C CNN
-F 3 "" H 2500 7000 50  0001 C CNN
-	1    2500 7000
-	1    0    0    -1
-$EndComp
 $EndSCHEMATC
