File: hardware/project/ETH3CDAQ1/VREF.sch (KiCad schematic (older format))
At the start: 5 parts, among them U901 ADR4550

Commit message: Schematic design
Parts:
- added C801, C802: 100n, Capacitor_SMD:C_0603_1608Metric_Pad1.08x0.95mm_HandSolder, symbol Device:C
- added R801, R802, R804: 10k, Resistor_SMD:R_0603_1608Metric_Pad0.98x0.95mm_HandSolder, symbol Device:R
- added R803: 20k, Resistor_SMD:R_0603_1608Metric_Pad0.98x0.95mm_HandSolder, symbol Device:R
- added U801: OPA2277, Package_SO:SOIC-8_3.9x4.9mm_P1.27mm, symbol Amplifier_Operational:OPA2277
- C803: renamed from C901; footprint (none) -> Capacitor_SMD:C_0603_1608Metric_Pad1.08x0.95mm_HandSolder
- C804: renamed from C902; footprint (none) -> Capacitor_SMD:C_1206_3216Metric_Pad1.33x1.80mm_HandSolder
- C805: renamed from C903; footprint (none) -> Capacitor_SMD:C_0603_1608Metric_Pad1.08x0.95mm_HandSolder
- C806: renamed from C904; footprint (none) -> Capacitor_SMD:C_1206_3216Metric_Pad1.33x1.80mm_HandSolder
- renumbered U901 to U802
Connections:
- net +5VP: now also R801.2, U801.5 (+)
- net GND renamed GNDA
- net GNDA: now also C801.2, C802.2, R802.2, U801.3 (+)
- new net: R801.1, R803.2, U801.2 (-)
- new net: R802.1, R804.2, U801.6 (-)
- new net +10V: R804.1, U801.7
- new net +15V: C801.1, U801.8 (V+)
- new net -10V: R803.1, U801.1
- new net -15V: C802.1, U801.4 (V-)
Other:
- moved on the sheet: C803, C804, C805, C806, U802
