File: hardware/project/ETH3CDAQ1/ETH3CDAQ1.kicad_pcb (KiCad board)
At the start: 2 copper layers, 160 x 100 mm, 270 parts, among them J401 20021111-00010T4LF, J402 Conn_02x01, J501 C64AC, Q601 IRFR5410, U1001 IS42S16400J-xC, U201 LAN8742A, U202 LC03-3.3, U203 LC03-3.3, U301 TXB0104PW, U302 ADuM5402, U303 74AC125, U401 HDC1080, U402 SN74LVC1T45DBV, U403 SN74LVC1T45DBV, U404 SN74LVC1T45DBV, U405 STM32H743ZI, U406 24LC08B-E/MS, U601 LT8330_S6, U602 LT8330_S6, U603 MAX5902, U604 ADP7118_LFCSP6, U605 ADP7182_LFCSP6, U606 ADP7118_LFCSP6, U607 ADP7182-2V5_LFCSP6, U608 TSR1-2433, U609 TSR1-2450, U701 LT1355, U702 DG211, U703 DG419LDY, U704 OPA140, U705 DG419LDY, U706 AD8251, U707 SN74LVC1G14DBVR, U708 SN74LVC1G14DBVR, U709 SN74LVC1G14DBVR, U710 ADAQ798x, U711 74HCT595, U801 OPA2277, U802 ADR4550, Y201 NX5032GA-25.000M-LN-CD-1, Y401 NX3225GD-8MHZ

Commit message: Schematic design.
Parts:
- removed the C625 at (-124.2, 101.7)
- removed the C626 at (-130.2, 108.4)
- removed L603, L604: TCK-141, ETH3CDAQ1:TCK-141
- added C628: 10u/50V, Capacitor_SMD:C_1206_3216Metric_Pad1.33x1.80mm_HandSolder, F.Cu at (188.6, 156.0)
- added C631: 10u/16V, Capacitor_SMD:C_1206_3216Metric_Pad1.33x1.80mm_HandSolder, F.Cu at (179.6, 154.0)
- added U610: TSR1-2490, ETH3CDAQ1:TSR1, F.Cu at (192.0, 139.0)
- moved R302 333.4 mm to (198.0, 93.0), turned to 90 degrees
- moved J401 261.1 mm to (202.0, 56.0), turned to 90 degrees
- moved U710 16.2 mm to (147.0, 56.7), turned to 90 degrees
- moved U704 14.8 mm to (147.5, 76.5), turned to 90 degrees
- moved U711 14.3 mm to (155.1, 57.4), turned to 90 degrees
- moved U702 14.1 mm to (155.1, 76.5), turned to 90 degrees
- moved RN702 12.4 mm to (145.0, 61.7), turned to 90 degrees
- moved U609 11.9 mm to (192.0, 130.0)
- moved RN701 8.53 mm to (149.1, 61.7), turned to 90 degrees
- moved D601 7.28 mm to (205.0, 142.0), turned to 90 degrees
- moved Q601 7.07 mm to (203.0, 131.0), turned to 90 degrees
- moved U706 6.26 mm to (147.8, 68.3), turned to 90 degrees
- moved U608 6.02 mm to (192.0, 121.0)
- moved U601 5.66 mm to (178.0, 140.0)
- moved U603 5.39 mm to (200.0, 142.0), turned to 90 degrees
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- renumbered C623 to C621, C624 to C622, C621 to C623, C622 to C624, C627 to C625, C628 to C626, C629 to C627, C630 to C629, C631 to C630
Connections:
- U608 pad 1: Net-(C625-Pad1) -> +24VF
- U609 pad 1: Net-(C626-Pad1) -> +24VF
- U704 pad 1: Net-(U704-Pad1) -> (no net)
- U704 pad 5: Net-(U704-Pad5) -> (no net)
- U704 pad 8: Net-(U704-Pad8) -> (no net)
- U708 pad 1: Net-(U708-Pad1) -> (no net)
- U710 pad 12: Net-(U710-Pad12) -> (no net)
- U710 pad 23: /Channel 1/VREF -> (no net)
- U711 pad 7: Net-(U711-Pad7) -> (no net)
- U711 pad 9: /Channel 1/SR_QH1 -> (no net)
Other:
- outline, holes or cut-outs redrawn
- copper layers 2 -> 4
- board text added: "MODULE 1"
- board text added: "MODULE 2"
- board text added: "MODULE 3"
