File: hardware/project/ETH3CDAQ1_BASE/Power.sch (KiCad schematic (older format))
At the start: 107 parts, among them Q601 IRFR5410, U601 LT8330_S6, U602 LT8330_S6, U603 LT8330_S6, U604 LT8330_S6, U605 MAX5902, U606 ADP7118_LFCSP6, U607 ADP7182_LFCSP6, U608 ADP7118_LFCSP6, U609 ADP7182_LFCSP6, U611 TSR1-2450, U613 TSR1-2490

Commit message: Schematic design.
Parts:
- gave numbers to parts that had none: 1
- renumbered C601 to C201, C602 to C202, C603 to C203, C604 to C204, C605 to C205, C606 to C206, C607 to C207, C608 to C208, C609 to C209, C610 to C210, C611 to C211, C612 to C212, C613 to C213, C614 to C214, C615 to C215, C616 to C216, C617 to C217, C618 to C218, C619 to C219, C620 to C220, C621 to C221, C622 to C222, C623 to C223, C624 to C224, C625 to C225, C626 to C226, C627 to C227, C628 to C228, C629 to C229, C630 to C230, C631 to C231, C632 to C232, C633 to C233, C634 to C234, C635 to C235, C636 to C236, C637 to C237, C638 to C238, C639 to C239, C640 to C240, C641 to C241, C642 to C242, C648 to C243, C643 to C244, C644 to C245, C650 to C246, C645 to C247, C646 to C248, C652 to C249, D602 to D201, D603 to D202, D604 to D203, D605 to D204, D601 to D205, D606 to D206, D607 to D207, F601 to F201, L601 to L201, L602 to L202, L603 to L203, L604 to L204, L605 to L205, L606 to L206, L608 to L207, Q601 to Q201, R601 to R201, R602 to R202, R603 to R203, R604 to R204, R605 to R205, R606 to R206, R607 to R207, R608 to R208, R610 to R209, R611 to R210, R612 to R211, R613 to R212, R614 to R213, R615 to R214, R616 to R215, R617 to R216, R619 to R217, R620 to R218, R621 to R219, R622 to R220, R623 to R221, R624 to R222, R625 to R223, R626 to R224, R627 to R225, R628 to R226, R629 to R227, R630 to R228, R609 to R229, R618 to R230, U601 to U201, U602 to U202, U603 to U203, U604 to U204, U606 to U205, U607 to U206, U608 to U207, U609 to U208, U611 to U210, U613 to U211, U605 to U212
Connections:
- net GND: now also L201.3, L203.3
Other:
- moved on the sheet: C241, C242, C243, C244, C245, C246, C247, C248, C249, D205, D206, D207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

Commit message: Schematic design
Parts:
- removed C244: 10u/50V, Capacitor_SMD:C_1206_3216Metric_Pad1.33x1.80mm_HandSolder, symbol Device:C
- removed C247: 10u/16V, Capacitor_SMD:C_1206_3216Metric_Pad1.33x1.80mm_HandSolder, symbol Device:C
- removed U209: TSR2-2433, ETH3CDAQ1:TSR2, symbol ETH3CDAQ1:TSR2
- removed U210: TSR1-2450, ETH3CDAQ1:TSR1, symbol ETH3CDAQ1:TSR1-2450
- removed U211: TSR1-2490, ETH3CDAQ1:TSR1, symbol ETH3CDAQ1:TSR1-2450
- added C243: 10u/50V, Capacitor_SMD:C_1206_3216Metric_Pad1.33x1.80mm_HandSolder, symbol Device:C
- added C245: 10u/16V, Capacitor_SMD:C_1206_3216Metric_Pad1.33x1.80mm_HandSolder, symbol Device:C
- added U209: TSR1-2433SM, ETH3CDAQ1:TSR1SM, symbol ETH3CDAQ1:TSR1SM
- added U210: TSR1-2450SM, ETH3CDAQ1:TSR1SM, symbol ETH3CDAQ1:TSR1SM
- added U212: TSR1-2490SM, ETH3CDAQ1:TSR1SM, symbol ETH3CDAQ1:TSR1SM
- R210, R214: value 111k -> 82k5
- R212, R216: value 53k -> 39k2
- renumbered C245 to C244, C248 to C246, C243 to C247, C246 to C248, U212 to U211
Connections:
- net +3V3: now also C245.1, U209.5 (VO)
- net +5V: now also U210.5 (VO)
- net +9V: now also U212.5 (VO)
- net GND: now also C243.2, C245.2, U209.7 (GND), U209.9 (GND), U210.7 (GND), U210.9 (GND), U212.7 (GND), U212.9 (GND)
- net at C244.1, L206.2: now also U210.1 (VI)
- net at L205.2: now also C243.1, U209.1 (VI)
- net at C248.1, L207.2: now also U212.1 (VI)
Other:
- moved on the sheet: C247, C248, C249, L207

Commit message: PCB layout
Parts:
- removed C233, C234, C235, C236: 100n, Capacitor_SMD:C_0603_1608Metric_Pad1.08x0.95mm_HandSolder, symbol Device:C
- removed R225, R226, R227, R228: R, Resistor_SMD:R_0603_1608Metric_Pad0.98x0.95mm_HandSolder, symbol Device:R
- removed U205, U207: ADP7118_LFCSP6, ETH3CDAQ1:LFCSP-6_2x2mm_1EP_P0.65mm, symbol ETH3CDAQ1:ADP7118_LFCSP6
- removed U206, U208: ADP7182_LFCSP6, ETH3CDAQ1:LFCSP-6_2x2mm_1EP_P0.65mm, symbol ETH3CDAQ1:ADP7182_LFCSP6
- added U205, U207: LM317_TO263, Package_TO_SOT_SMD:TO-263-3_TabPin2, symbol Regulator_Linear:LM317_3PinPackage
- added U206, U208: LM337_TO263, Package_TO_SOT_SMD:TO-263-2, symbol Regulator_Linear:LM337_TO263
- R217: value 100k -> 3k2; footprint Resistor_SMD:R_0603_1608Metric_Pad0.98x0.95mm_HandSolder -> Resistor_SMD:R_0603_1608Metric_Pad1.05x0.95mm_HandSolder
- R218: value 49k9 -> 1k6; footprint Resistor_SMD:R_0603_1608Metric_Pad0.98x0.95mm_HandSolder -> Resistor_SMD:R_0603_1608Metric_Pad1.05x0.95mm_HandSolder
- R219: value 150k -> 3k2; footprint Resistor_SMD:R_0603_1608Metric_Pad0.98x0.95mm_HandSolder -> Resistor_SMD:R_0603_1608Metric_Pad1.05x0.95mm_HandSolder
- R220: value 13k3 -> 1k6; footprint Resistor_SMD:R_0603_1608Metric_Pad0.98x0.95mm_HandSolder -> Resistor_SMD:R_0603_1608Metric_Pad1.05x0.95mm_HandSolder
- R221: value 100k -> 240; footprint Resistor_SMD:R_0603_1608Metric_Pad0.98x0.95mm_HandSolder -> Resistor_SMD:R_0603_1608Metric_Pad1.05x0.95mm_HandSolder
- R222: value 49k9 -> 120; footprint Resistor_SMD:R_0603_1608Metric_Pad0.98x0.95mm_HandSolder -> Resistor_SMD:R_0603_1608Metric_Pad1.05x0.95mm_HandSolder
- R223: value 150k -> 240; footprint Resistor_SMD:R_0603_1608Metric_Pad0.98x0.95mm_HandSolder -> Resistor_SMD:R_0603_1608Metric_Pad1.05x0.95mm_HandSolder
- R224: value 13k3 -> 120; footprint Resistor_SMD:R_0603_1608Metric_Pad0.98x0.95mm_HandSolder -> Resistor_SMD:R_0603_1608Metric_Pad1.05x0.95mm_HandSolder
- renumbered C237 to C233, C238 to C234, C239 to C235, C240 to C236, C241 to C237, C242 to C238, C243 to C239, C244 to C240, C245 to C241, C246 to C242, C247 to C243, C248 to C244, C249 to C245, R229 to R225, R230 to R226
Connections:
- net GND: now also R217.2, R219.2; no longer R222.2, R224.2
- net at C217.1, C221.1, C225.1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: now also U205.3 (VI)
- net at C218.1, C222.1, C226.1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: now also U206.2 (VI)
- net at C219.1, C223.1, C227.1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: now also U207.3 (VI)
- net at C220.1, C224.1, C228.1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: now also U208.2 (VI)
- net at R221.2: now also R217.1, U205.1 (ADJ); no longer R222.1
- net at R223.2: now also R219.1, U207.1 (ADJ); no longer R224.1
- net at R218.1: now also R222.2, U206.1 (ADJ); no longer R217.2
- net at R220.1: now also R224.2, U208.1 (ADJ); no longer R219.2
- net +15V renamed +18V
- net +18V: now also R221.1, U205.2 (VO); no longer R217.1
- net +15VF renamed +18VF
- net +18VF: now also R223.1, U207.2 (VO); no longer R221.1
- net -15V renamed -18V
- net -18V: now also R222.1, U206.3 (VO); no longer R219.1
- net -15VF renamed -18VF
- net -18VF: now also R224.1, U208.3 (VO); no longer R223.1
- no-connect marks 3 -> 1
Other:
- moved on the sheet: C233, C234, C235, C236
