File: hardware/project/ETH3CDAQ1_BASE/Connector.sch (KiCad schematic (older format))
At the start: 3 parts, among them J301 Conn_02x02_Odd_Even, J302 Conn_02x04_Odd_Even, J303 C64AC

Commit message: PCB layout
Changed lines of the file:
@@
+	1    0    0    -1
+$EndComp
+$Comp
+L power:PWR_FLAG #FLG0301
+U 1 1 60030887
+P 1150 6950
+F 0 "#FLG0301" H 1150 7025 50  0001 C CNN
+F 1 "PWR_FLAG" H 1150 7123 50  0000 C CNN
+F 2 "" H 1150 6950 50  0001 C CNN
+F 3 "~" H 1150 6950 50  0001 C CNN
+	1    1150 6950
+	1    0    0    -1
+$EndComp
+$Comp
+L power:Earth #PWR0312
+U 1 1 60030E52
+P 1150 6950
+F 0 "#PWR0312" H 1150 6700 50  0001 C CNN
+F 1 "Earth" H 1150 6800 50  0001 C CNN
+F 2 "" H 1150 6950 50  0001 C CNN
+F 3 "~" H 1150 6950 50  0001 C CNN
+	1    1150 6950
+	1    0    0    -1
+$EndComp
+$Comp
+L power:PWR_FLAG #FLG0302
+U 1 1 6003B275
+P 1600 6950
+F 0 "#FLG0302" H 1600 7025 50  0001 C CNN
+F 1 "PWR_FLAG" H 1600 7123 50  0000 C CNN
+F 2 "" H 1600 6950 50  0001 C CNN
+F 3 "~" H 1600 6950 50  0001 C CNN
+	1    1600 6950
+	1    0    0    -1
+$EndComp
+$Comp
+L ETH3CDAQ1:GND_TRIG #PWR0313
+U 1 1 6003C15F
+P 1600 6950
+F 0 "#PWR0313" H 1600 6700 50  0001 C CNN
+F 1 "GND_TRIG" H 1605 6777 50  0000 C CNN
+F 2 "" H 1600 6950 50  0001 C CNN
+F 3 "" H 1600 6950 50  0001 C CNN
+	1    1600 6950
 	1    0    0    -1
 $EndComp
