File: hardware/project/ETH3CDAQ1_BASE/Selftest.sch (KiCad schematic (older format))
At the start: 24 parts, among them U701 TL074, U702 TL071, U703 TLA2528

Commit message: Modifications in PCB and schematic in the base module.
Parts:
- removed U702: TL071, Package_SO:SO-8_3.9x4.9mm_P1.27mm, symbol Amplifier_Operational:TL071
- added U702: TL072, Package_SO:SO-8_3.9x4.9mm_P1.27mm, symbol Amplifier_Operational:TL072
- R701, R705: value 200k -> 250k
- R703: value 200k -> 33k
- R704: value 200k -> 100k
- R711: value R -> 0
- R712: value R -> DNP
Connections:
- net +18V: now also U702.8 (V+); no longer R701.2
- net -18V: now also R701.2, U702.4 (V-)
- net AIN2: now also U702.1
- net GND: now also U702.3 (+)
- net at R709.1, R710.2: now also U702.2 (-)
- net at R701.1, R702.1: now also U702.5 (+); no longer R709.2
- new net: R709.2, U702.6 (-), U702.7
- no-connect marks 5 -> 3
Other:
- moved on the sheet: C701, C702, C703, C704, C705, C706, R701, R702, R703, R704, R705, R706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

Commit message: Modification in PCBs. Created BOM files.
Parts:
- C705: value 100n -> 1u
- R701, R705: value 250k -> 249k
- R702, R706, R707, R708: value 50k -> 49k9
Other:
- moved on the sheet: C703, C704, C705, C706
Changed lines of the file:
@@
 P 4400 2050
 F 0 "R706" H 4470 2096 50  0000 L CNN
-F 1 "50k" H 4470 2005 50  0000 L CNN
+F 1 "49k9" H 4470 2005 50  0000 L CNN
 F 2 "Resistor_SMD:R_0603_1608Metric_Pad0.98x0.95mm_HandSolder" V 4330 2050 50  0001 C CNN
 F 3 "~" H 4400 2050 50  0001 C CNN
@@
 P 4400 3050
 F 0 "R707" H 4470 3096 50  0000 L CNN
-F 1 "50k" H 4470 3005 50  0000 L CNN
+F 1 "49k9" H 4470 3005 50  0000 L CNN
 F 2 "Resistor_SMD:R_0603_1608Metric_Pad0.98x0.95mm_HandSolder" V 4330 3050 50  0001 C CNN
 F 3 "~" H 4400 3050 50  0001 C CNN
@@
 P 4200 3850
 F 0 "R705" V 3993 3850 50  0000 C CNN
-F 1 "250k" V 4084 3850 50  0000 C CNN
+F 1 "249k" V 4084 3850 50  0000 C CNN
 F 2 "Resistor_SMD:R_0603_1608Metric_Pad0.98x0.95mm_HandSolder" V 4130 3850 50  0001 C CNN
 F 3 "~" H 4200 3850 50  0001 C CNN
@@
 P 4400 4050
 F 0 "R708" H 4470 4096 50  0000 L CNN
-F 1 "50k" H 4470 4005 50  0000 L CNN
+F 1 "49k9" H 4470 4005 50  0000 L CNN
 F 2 "Resistor_SMD:R_0603_1608Metric_Pad0.98x0.95mm_HandSolder" V 4330 4050 50  0001 C CNN
 F 3 "~" H 4400 4050 50  0001 C CNN
@@
 P 3100 5700
 F 0 "R701" V 2893 5700 50  0000 C CNN
-F 1 "250k" V 2984 5700 50  0000 C CNN
+F 1 "249k" V 2984 5700 50  0000 C CNN
 F 2 "Resistor_SMD:R_0603_1608Metric_Pad0.98x0.95mm_HandSolder" V 3030 5700 50  0001 C CNN
 F 3 "~" H 3100 5700 50  0001 C CNN
@@
 P 3300 5900
 F 0 "R702" H 3370 5946 50  0000 L CNN
-F 1 "50k" H 3370 5855 50  0000 L CNN
+F 1 "49k9" H 3370 5855 50  0000 L CNN
 F 2 "Resistor_SMD:R_0603_1608Metric_Pad0.98x0.95mm_HandSolder" V 3230 5900 50  0001 C CNN
 F 3 "~" H 3300 5900 50  0001 C CNN
@@
 L Device:C C705
 U 1 1 5FEAE636
-P 3550 7150
-F 0 "C705" H 3435 7104 50  0000 R CNN
-F 1 "100n" H 3435 7195 50  0000 R CNN
-F 2 "Capacitor_SMD:C_0603_1608Metric_Pad1.08x0.95mm_HandSolder" H 3588 7000 50  0001 C CNN
-F 3 "~" H 3550 7150 50  0001 C CNN
-	1    3550 7150
+P 3600 7150
+F 0 "C705" H 3485 7104 50  0000 R CNN
+F 1 "1u" H 3485 7195 50  0000 R CNN
+F 2 "Capacitor_SMD:C_0603_1608Metric_Pad1.08x0.95mm_HandSolder" H 3638 7000 50  0001 C CNN
+F 3 "~" H 3600 7150 50  0001 C CNN
+	1    3600 7150
 	-1   0    0    1
 $EndComp
@@
 L Device:C C706
 U 1 1 5FEAEEBE
-P 4000 7150
-F 0 "C706" H 3885 7104 50  0000 R CNN
-F 1 "100n" H 3885 7195 50  0000 R CNN
-F 2 "Capacitor_SMD:C_0603_1608Metric_Pad1.08x0.95mm_HandSolder" H 4038 7000 50  0001 C CNN
-F 3 "~" H 4000 7150 50  0001 C CNN
-	1    4000 7150
+P 4050 7150
+F 0 "C706" H 3935 7104 50  0000 R CNN
+F 1 "100n" H 3935 7195 50  0000 R CNN
+F 2 "Capacitor_SMD:C_0603_1608Metric_Pad1.08x0.95mm_HandSolder" H 4088 7000 50  0001 C CNN
+F 3 "~" H 4050 7150 50  0001 C CNN
+	1    4050 7150
 	-1   0    0    1
 $EndComp
@@
 L Device:C C703
 U 1 1 5FEB5A11
-P 2650 7150
-F 0 "C703" H 2535 7104 50  0000 R CNN
-F 1 "100n" H 2535 7195 50  0000 R CNN
-F 2 "Capacitor_SMD:C_0603_1608Metric_Pad1.08x0.95mm_HandSolder" H 2688 7000 50  0001 C CNN
-F 3 "~" H 2650 7150 50  0001 C CNN
-	1    2650 7150
+P 2700 7150
+F 0 "C703" H 2585 7104 50  0000 R CNN
+F 1 "100n" H 2585 7195 50  0000 R CNN
+F 2 "Capacitor_SMD:C_0603_1608Metric_Pad1.08x0.95mm_HandSolder" H 2738 7000 50  0001 C CNN
+F 3 "~" H 2700 7150 50  0001 C CNN
+	1    2700 7150
 	-1   0    0    1
 $EndComp
@@
 L Device:C C704
 U 1 1 5FEB5A17
-P 3100 7150
-F 0 "C704" H 2985 7104 50  0000 R CNN
-F 1 "100n" H 2985 7195 50  0000 R CNN
-F 2 "Capacitor_SMD:C_0603_1608Metric_Pad1.08x0.95mm_HandSolder" H 3138 7000 50  0001 C CNN
-F 3 "~" H 3100 7150 50  0001 C CNN
-	1    3100 7150
+P 3150 7150
+F 0 "C704" H 3035 7104 50  0000 R CNN
+F 1 "100n" H 3035 7195 50  0000 R CNN
+F 2 "Capacitor_SMD:C_0603_1608Metric_Pad1.08x0.95mm_HandSolder" H 3188 7000 50  0001 C CNN
+F 3 "~" H 3150 7150 50  0001 C CNN
+	1    3150 7150
 	-1   0    0    1
 $EndComp
@@
 L ETH3CDAQ1:+18V #PWR0707
 U 1 1 5FEBE64C
-P 2650 7000
-F 0 "#PWR0707" H 2650 6850 50  0001 C CNN
-F 1 "+18V" H 2665 7173 50  0000 C CNN
-F 2 "" H 2650 7000 50  0001 C CNN
-F 3 "" H 2650 7000 50  0001 C CNN
-	1    2650 7000
+P 2700 7000
+F 0 "#PWR0707" H 2700 6850 50  0001 C CNN
+F 1 "+18V" H 2715 7173 50  0000 C CNN
+F 2 "" H 2700 7000 50  0001 C CNN
+F 3 "" H 2700 7000 50  0001 C CNN
+	1    2700 7000
 	1    0    0    -1
 $EndComp
@@
 L ETH3CDAQ1:-18V #PWR0709
 U 1 1 5FEBF8F1
-P 3100 7000
-F 0 "#PWR0709" H 3100 6850 50  0001 C CNN
-F 1 "-18V" H 3115 7173 50  0000 C CNN
-F 2 "" H 3100 7000 50  0001 C CNN
-F 3 "" H 3100 7000 50  0001 C CNN
-	1    3100 7000
+P 3150 7000
+F 0 "#PWR0709" H 3150 6850 50  0001 C CNN
+F 1 "-18V" H 3165 7173 50  0000 C CNN
+F 2 "" H 3150 7000 50  0001 C CNN
+F 3 "" H 3150 7000 50  0001 C CNN
+	1    3150 7000
 	1    0    0    -1
 $EndComp
@@
 L power:GND #PWR0708
 U 1 1 5FEC2559
-P 2650 7300
-F 0 "#PWR0708" H 2650 7050 50  0001 C CNN
-F 1 "GND" H 2655 7127 50  0000 C CNN
-F 2 "" H 2650 7300 50  0001 C CNN
-F 3 "" H 2650 7300 50  0001 C CNN
-	1    2650 7300
+P 2700 7300
+F 0 "#PWR0708" H 2700 7050 50  0001 C CNN
+F 1 "GND" H 2705 7127 50  0000 C CNN
+F 2 "" H 2700 7300 50  0001 C CNN
+F 3 "" H 2700 7300 50  0001 C CNN
+	1    2700 7300
 	1    0    0    -1
 $EndComp
@@
 L power:GND #PWR0710
 U 1 1 5FEC32F6
-P 3100 7300
-F 0 "#PWR0710" H 3100 7050 50  0001 C CNN
-F 1 "GND" H 3105 7127 50  0000 C CNN
-F 2 "" H 3100 7300 50  0001 C CNN
-F 3 "" H 3100 7300 50  0001 C CNN
-	1    3100 7300
+P 3150 7300
+F 0 "#PWR0710" H 3150 7050 50  0001 C CNN
+F 1 "GND" H 3155 7127 50  0000 C CNN
+F 2 "" H 3150 7300 50  0001 C CNN
+F 3 "" H 3150 7300 50  0001 C CNN
+	1    3150 7300
 	1    0    0    -1
 $EndComp
@@
 L power:GND #PWR0712
 U 1 1 5FEC4254
-P 3550 7300
-F 0 "#PWR0712" H 3550 7050 50  0001 C CNN
-F 1 "GND" H 3555 7127 50  0000 C CNN
-F 2 "" H 3550 7300 50  0001 C CNN
-F 3 "" H 3550 7300 50  0001 C CNN
-	1    3550 7300
+P 3600 7300
+F 0 "#PWR0712" H 3600 7050 50  0001 C CNN
+F 1 "GND" H 3605 7127 50  0000 C CNN
+F 2 "" H 3600 7300 50  0001 C CNN
+F 3 "" H 3600 7300 50  0001 C CNN
+	1    3600 7300
 	1    0    0    -1
 $EndComp
@@
 L power:GND #PWR0715
 U 1 1 5FEC4698
-P 4000 7300
-F 0 "#PWR0715" H 4000 7050 50  0001 C CNN
-F 1 "GND" H 4005 7127 50  0000 C CNN
-F 2 "" H 4000 7300 50  0001 C CNN
-F 3 "" H 4000 7300 50  0001 C CNN
-	1    4000 7300
+P 4050 7300
+F 0 "#PWR0715" H 4050 7050 50  0001 C CNN
+F 1 "GND" H 4055 7127 50  0000 C CNN
+F 2 "" H 4050 7300 50  0001 C CNN
+F 3 "" H 4050 7300 50  0001 C CNN
+	1    4050 7300
 	1    0    0    -1
 $EndComp
@@
 L power:+3.3V #PWR0714
 U 1 1 5FECCA76
-P 4000 7000
-F 0 "#PWR0714" H 4000 6850 50  0001 C CNN
-F 1 "+3.3V" H 4000 7150 50  0000 C CNN
-F 2 "" H 4000 7000 50  0001 C CNN
-F 3 "" H 4000 7000 50  0001 C CNN
-	1    4000 7000
+P 4050 7000
+F 0 "#PWR0714" H 4050 6850 50  0001 C CNN
+F 1 "+3.3V" H 4050 7150 50  0000 C CNN
+F 2 "" H 4050 7000 50  0001 C CNN
+F 3 "" H 4050 7000 50  0001 C CNN
+	1    4050 7000
 	1    0    0    -1
 $EndComp
@@
 L power:+5V #PWR0711
 U 1 1 5FED0A67
-P 3550 7000
-F 0 "#PWR0711" H 3550 6850 50  0001 C CNN
-F 1 "+5V" H 3550 7150 50  0000 C CNN
-F 2 "" H 3550 7000 50  0001 C CNN
-F 3 "" H 3550 7000 50  0001 C CNN
-	1    3550 7000
-	1    0    0    -1
-$EndComp
+P 3600 7000
+F 0 "#PWR0711" H 3600 6850 50  0001 C CNN
+F 1 "+5V" H 3600 7150 50  0000 C CNN
+F 2 "" H 3600 7000 50  0001 C CNN
+F 3 "" H 3600 7000 50  0001 C CNN
+	1    3600 7000
+	1    0    0    -1
+$EndComp

Commit message: PCB modifications
Other:
- note added: "Need to add 18VF and -18VF. Replace TL072 with TL074."
Changed lines of the file:
@@
 Wire Wire Line
 	3250 5700 3300 5700
+Text Notes 5950 5200 0    50   ~ 0
+Need to add 18VF and -18VF. Replace TL072 with TL074.
 $EndSCHEMATC

Commit message: PCB and software development.
Parts:
- removed U702: TL072, Package_SO:SO-8_3.9x4.9mm_P1.27mm, symbol Amplifier_Operational:TL072
- added C705, C706: 100n, Capacitor_SMD:C_0603_1608Metric_Pad1.08x0.95mm_HandSolder, symbol Device:C
- added R702, R714: 249k, Resistor_SMD:R_0603_1608Metric_Pad0.98x0.95mm_HandSolder, symbol Device:R
- added R704, R716: 49k9, Resistor_SMD:R_0603_1608Metric_Pad0.98x0.95mm_HandSolder, symbol Device:R
- added R710, R712: 1k, Resistor_SMD:R_0603_1608Metric_Pad0.98x0.95mm_HandSolder, symbol Device:R
- added U702: TL074, Package_SO:TSSOP-14_4.4x5mm_P0.65mm, symbol Amplifier_Operational:TL074
- added U703: TL071, Package_SO:SOIC-8_3.9x4.9mm_P1.27mm, symbol Amplifier_Operational:TL071
- renumbered C705 to C707, C706 to C708, C707 to C709, R702 to R703, R703 to R705, R705 to R706, R706 to R707, R710 to R711, R704 to R713, R707 to R715, R711 to R717, R712 to R718, R713 to R719, R714 to R720, U703 to U704
Connections:
- net +18V: now also C705.2, U702.4 (V+), U703.7 (V+)
- net -18V: now also C706.2, U702.11 (V-), U703.4 (V-)
- net AIN2: now also U702.1
- net GND: now also C705.1, C706.1, R704.2, R716.2, U702.10 (+), U702.3 (+)
- net AIN5: now reaches U704.4 (AIN5/GPIO5)
- net AIN5: now also R712.1, U702.8
- net AIN6: now reaches U704.5 (AIN6/GPIO6)
- net AIN6: now also U703.2 (-), U703.6
- net at R709.1, R711.2: now also U702.2 (-)
- net at R701.1, R703.1: now also U702.5 (+)
- net at R709.2: now also U702.6 (-), U702.7
- new net: R710.1, R712.2, U702.9 (-)
- new net: R702.1, R704.1, U702.12 (+)
- new net: R710.2, U702.13 (-), U702.14
- new net: R714.1, R716.1, U703.3 (+)
- new net +18VF: R714.2
- new net -18VF: R702.2
Other:
- moved on the sheet: C707, C708, R701, R703, R705, R706, R707, R708, R709, R711, R713, R715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
