File: hardware/project/ETH3CDAQ1_MEASURE/Power.sch (KiCad schematic (older format))
At the start: 0 parts

Commit message: Measurement module development.
Parts:
- added C901, C902: 10u, Capacitor_SMD:C_1206_3216Metric_Pad1.33x1.80mm_HandSolder, symbol Device:C
- added U901: LM1117-5.0, Package_TO_SOT_SMD:SOT-223-3_TabPin2, symbol Regulator_Linear:LM1117-5.0
Connections:
- new net +5VF: C902.1, U901.2 (VO)
- new net +9V: C901.1, U901.3 (VI)
- new net GND: C901.2, C902.2, U901.1 (GND)
