File: hardware/project/ETH3CDAQ1_MEASURE/Power.sch (KiCad schematic (older format))
At the start: 3 parts, among them U901 LM1117-5.0

Commit message: PCB layout
Parts:
- renumbered C901 to C601, C902 to C602, U901 to U601
Changed lines of the file:
@@
 $EndDescr
 $Comp
-L Regulator_Linear:LM1117-5.0 U901
+L Regulator_Linear:LM1117-5.0 U601
 U 1 1 5FE0E2E8
 P 2850 1900
-F 0 "U901" H 2850 2142 50  0000 C CNN
+F 0 "U601" H 2850 2142 50  0000 C CNN
 F 1 "LM1117-5.0" H 2850 2051 50  0000 C CNN
 F 2 "Package_TO_SOT_SMD:SOT-223-3_TabPin2" H 2850 1900 50  0001 C CNN
@@
 $EndComp
 $Comp
-L power:GNDA #PWR0907
+L power:GNDA #PWR0607
 U 1 1 5FE0EA9E
 P 2850 2350
-F 0 "#PWR0907" H 2850 2100 50  0001 C CNN
+F 0 "#PWR0607" H 2850 2100 50  0001 C CNN
 F 1 "GNDA" H 2855 2177 50  0000 C CNN
 F 2 "" H 2850 2350 50  0001 C CNN
@@
 $EndComp
 $Comp
-L Device:C C901
+L Device:C C601
 U 1 1 5FE0EF0E
 P 2250 2100
-F 0 "C901" H 2365 2146 50  0000 L CNN
+F 0 "C601" H 2365 2146 50  0000 L CNN
 F 1 "10u" H 2365 2055 50  0000 L CNN
 F 2 "Capacitor_SMD:C_1206_3216Metric_Pad1.33x1.80mm_HandSolder" H 2288 1950 50  0001 C CNN
@@
 $EndComp
 $Comp
-L Device:C C902
+L Device:C C602
 U 1 1 5FE0F335
 P 3400 2100
-F 0 "C902" H 3515 2146 50  0000 L CNN
+F 0 "C602" H 3515 2146 50  0000 L CNN
 F 1 "10u" H 3515 2055 50  0000 L CNN
 F 2 "Capacitor_SMD:C_1206_3216Metric_Pad1.33x1.80mm_HandSolder" H 3438 1950 50  0001 C CNN
@@
 	2850 2300 3400 2300
 $Comp
-L power:+9V #PWR0904
+L power:+9V #PWR0604
 U 1 1 5FE11F66
 P 2250 1850
-F 0 "#PWR0904" H 2250 1700 50  0001 C CNN
+F 0 "#PWR0604" H 2250 1700 50  0001 C CNN
 F 1 "+9V" H 2265 2023 50  0000 C CNN
 F 2 "" H 2250 1850 50  0001 C CNN
@@
 Connection ~ 2250 1900
 $Comp
-L ETH3CDAQ1:+5VF #PWR0909
+L ETH3CDAQ1:+5VF #PWR0609
 U 1 1 5FE12C26
 P 3400 1850
-F 0 "#PWR0909" H 3400 1700 50  0001 C CNN
+F 0 "#PWR0609" H 3400 1700 50  0001 C CNN
 F 1 "+5VF" H 3415 2023 50  0000 C CNN
 F 2 "" H 3400 1850 50  0001 C CNN
@@
 Connection ~ 3400 1900
 $Comp
-L ETH3CDAQ1:+18V #PWR0902
+L ETH3CDAQ1:+18V #PWR0602
 U 1 1 5FED1831
 P 1400 7350
-F 0 "#PWR0902" H 1400 7200 50  0001 C CNN
+F 0 "#PWR0602" H 1400 7200 50  0001 C CNN
 F 1 "+18V" H 1415 7523 50  0000 C CNN
 F 2 "" H 1400 7350 50  0001 C CNN
@@
 $EndComp
 $Comp
-L ETH3CDAQ1:-18V #PWR0903
+L ETH3CDAQ1:-18V #PWR0603
 U 1 1 5FED1DF4
 P 1850 7350
-F 0 "#PWR0903" H 1850 7200 50  0001 C CNN
+F 0 "#PWR0603" H 1850 7200 50  0001 C CNN
 F 1 "-18V" H 1865 7523 50  0000 C CNN
 F 2 "" H 1850 7350 50  0001 C CNN
@@
 $EndComp
 $Comp
-L power:PWR_FLAG #FLG0902
+L power:PWR_FLAG #FLG0602
 U 1 1 5FED22FB
 P 1400 7350
-F 0 "#FLG0902" H 1400 7425 50  0001 C CNN
+F 0 "#FLG0602" H 1400 7425 50  0001 C CNN
 F 1 "PWR_FLAG" H 1400 7523 50  0000 C CNN
 F 2 "" H 1400 7350 50  0001 C CNN
@@
 $EndComp
 $Comp
-L power:PWR_FLAG #FLG0903
+L power:PWR_FLAG #FLG0603
 U 1 1 5FED2734
 P 1850 7350
-F 0 "#FLG0903" H 1850 7425 50  0001 C CNN
+F 0 "#FLG0603" H 1850 7425 50  0001 C CNN
 F 1 "PWR_FLAG" H 1850 7523 50  0000 C CNN
 F 2 "" H 1850 7350 50  0001 C CNN
@@
 $EndComp
 $Comp
-L power:PWR_FLAG #FLG0904
+L power:PWR_FLAG #FLG0604
 U 1 1 5FED43BD
 P 2300 7350
-F 0 "#FLG0904" H 2300 7425 50  0001 C CNN
+F 0 "#FLG0604" H 2300 7425 50  0001 C CNN
 F 1 "PWR_FLAG" H 2300 7523 50  0000 C CNN
 F 2 "" H 2300 7350 50  0001 C CNN
@@
 $EndComp
 $Comp
-L power:+5V #PWR0905
+L power:+5V #PWR0605
 U 1 1 5FED47A8
 P 2300 7350
-F 0 "#PWR0905" H 2300 7200 50  0001 C CNN
+F 0 "#PWR0605" H 2300 7200 50  0001 C CNN
 F 1 "+5V" H 2315 7523 50  0000 C CNN
 F 2 "" H 2300 7350 50  0001 C CNN
@@
 $EndComp
 $Comp
-L power:PWR_FLAG #FLG0905
+L power:PWR_FLAG #FLG0605
 U 1 1 5FED655C
 P 2750 7350
-F 0 "#FLG0905" H 2750 7425 50  0001 C CNN
+F 0 "#FLG0605" H 2750 7425 50  0001 C CNN
 F 1 "PWR_FLAG" H 2750 7523 50  0000 C CNN
 F 2 "" H 2750 7350 50  0001 C CNN
@@
 $EndComp
 $Comp
-L power:+3.3V #PWR0906
+L power:+3.3V #PWR0606
 U 1 1 5FED69C1
 P 2750 7350
-F 0 "#PWR0906" H 2750 7200 50  0001 C CNN
+F 0 "#PWR0606" H 2750 7200 50  0001 C CNN
 F 1 "+3.3V" H 2765 7523 50  0000 C CNN
 F 2 "" H 2750 7350 50  0001 C CNN
@@
 $EndComp
 $Comp
-L power:GND #PWR0908
+L power:GND #PWR0608
 U 1 1 5FEF388D
 P 3200 7350
-F 0 "#PWR0908" H 3200 7100 50  0001 C CNN
+F 0 "#PWR0608" H 3200 7100 50  0001 C CNN
 F 1 "GND" H 3205 7177 50  0000 C CNN
 F 2 "" H 3200 7350 50  0001 C CNN
@@
 $EndComp
 $Comp
-L power:GNDA #PWR0910
+L power:GNDA #PWR0610
 U 1 1 5FEF40C4
 P 3500 7350
-F 0 "#PWR0910" H 3500 7100 50  0001 C CNN
+F 0 "#PWR0610" H 3500 7100 50  0001 C CNN
 F 1 "GNDA" H 3505 7177 50  0000 C CNN
 F 2 "" H 3500 7350 50  0001 C CNN
@@
 	3500 7300 3500 7350
 $Comp
-L power:PWR_FLAG #FLG0901
+L power:PWR_FLAG #FLG0601
 U 1 1 5FEF796D
 P 950 7350
-F 0 "#FLG0901" H 950 7425 50  0001 C CNN
+F 0 "#FLG0601" H 950 7425 50  0001 C CNN
 F 1 "PWR_FLAG" H 950 7523 50  0000 C CNN
 F 2 "" H 950 7350 50  0001 C CNN
@@
 $EndComp
 $Comp
-L power:+9V #PWR0901
+L power:+9V #PWR0601
 U 1 1 5FEF80D2
 P 950 7350
-F 0 "#PWR0901" H 950 7200 50  0001 C CNN
+F 0 "#PWR0601" H 950 7200 50  0001 C CNN
 F 1 "+9V" H 965 7523 50  0000 C CNN
 F 2 "" H 950 7350 50  0001 C CNN
@@
 $EndComp
 $Comp
-L power:PWR_FLAG #FLG0906
+L power:PWR_FLAG #FLG0606
 U 1 1 5FF02954
 P 3350 7250
-F 0 "#FLG0906" H 3350 7325 50  0001 C CNN
+F 0 "#FLG0606" H 3350 7325 50  0001 C CNN
 F 1 "PWR_FLAG" H 3350 7423 50  0000 C CNN
 F 2 "" H 3350 7250 50  0001 C CNN
