File: hardware/project/ETH3CDAQ1_MEASURE/ETH3CDAQ1_MEASURE.kicad_pcb (KiCad board)
At the start: 4 copper layers, 73 x 100 mm, 194 parts, among them J201 20021111-00010T4LF, J202 Conn_02x01, J701 Conn_02x10_Odd_Even, J702 Conn_02x02_Odd_Even, J703 Conn_02x10_Odd_Even, J704 Conn_02x04_Odd_Even, J705 Conn_02x10_Odd_Even, U201 HDC1080, U202 SN74LVC1T45DBV, U203 SN74LVC1T45DBV, U204 SN74LVC1T45DBV, U205 STM32H743ZI, U206 24LC08B-E/MS, U301 LT1355, U302 DG211, U303 DG419LDY, U304 OPA140, U305 DG419LDY, U306 AD8251, U307 SN74LVC1G14DBVR, U308 SN74LVC1G14DBVR, U309 SN74LVC1G14DBVR, U310 ADAQ798x, U311 74HCT595, U401 TXB0104PW, U402 ADuM5402, U403 74AC125, U501 IS42S16400J-xC, U601 LAN8742A, U602 LC03-3.3, U603 LC03-3.3, Y201 NX3225GD-8MHZ, Y601 NX5032GA-25.000M-LN-CD-1

Commit message: Measurement module development.
Parts:
- removed the C308 at (125.8, -32.4)
- removed the C319 at (95.2, -8.12)
- removed C326: C, Capacitor_SMD:C_0603_1608Metric_Pad1.08x0.95mm_HandSolder
- removed D301: MMBZ15VDL, Package_TO_SOT_SMD:SOT-23
- removed D302: BAT54SW, Package_TO_SOT_SMD:SOT-323_SC-70
- removed J701, J703, J705: Conn_02x10_Odd_Even, Connector_PinSocket_2.54mm:PinSocket_2x10_P2.54mm_Vertical
- removed the R301 at (121.4, -29.9)
- removed the R302 at (112.7, -25.2)
- removed the R303 at (117.0, -25.3)
- removed the R307 at (110.0, -18.6)
- removed R317, R318, R319, R320, R321, R322: 620, Resistor_SMD:R_0603_1608Metric_Pad0.98x0.95mm_HandSolder
- removed RN301, RN302: 1k, Resistor_SMD:R_Array_Concave_4x0603
- removed U309: SN74LVC1G14DBVR, Package_TO_SOT_SMD:SOT-23-5
- removed U310: ADAQ798x, ETH3CDAQ1:LGA-24_5x4mm_P0.5mm
- removed U311: 74HCT595, Package_SO:TSSOP-16_4.4x5mm_P0.65mm
- added C1401: 22u, Capacitor_SMD:C_0805_2012Metric_Pad1.18x1.45mm_HandSolder, F.Cu at (72.0, -13.0)
- added C1402: 1u, Capacitor_SMD:C_0603_1608Metric_Pad1.08x0.95mm_HandSolder, F.Cu at (81.1, 0.38)
- added C1403: 10u, Capacitor_SMD:C_0805_2012Metric_Pad1.18x1.45mm_HandSolder, F.Cu at (54.8, 0.18)
- added C1404: 100n, Capacitor_SMD:C_0603_1608Metric_Pad1.08x0.95mm_HandSolder, F.Cu at (86.7, -2.13)
- added C1405: 100n, Capacitor_SMD:C_0603_1608Metric_Pad1.08x0.95mm_HandSolder, F.Cu at (76.8, -0.20)
- added C1406: 100n, Capacitor_SMD:C_0603_1608Metric_Pad1.08x0.95mm_HandSolder, F.Cu at (59.4, -0.07)
- added C1407: 100n, Capacitor_SMD:C_0603_1608Metric_Pad1.08x0.95mm_HandSolder, F.Cu at (69.3, -6.80)
- added C1408: 330p, Capacitor_SMD:C_0603_1608Metric_Pad1.08x0.95mm_HandSolder, F.Cu at (76.6, -13.2)
- added C1409: 100n, Capacitor_SMD:C_0603_1608Metric_Pad1.08x0.95mm_HandSolder, F.Cu at (69.3, -4.29)
- added C1410: 100n, Capacitor_SMD:C_0603_1608Metric_Pad1.08x0.95mm_HandSolder, F.Cu at (63.7, -0.23)
- added C1411: 100p, Capacitor_SMD:C_0603_1608Metric_Pad1.08x0.95mm_HandSolder, F.Cu at (84.4, -19.7)
- added C1412: 100n, Capacitor_SMD:C_0603_1608Metric_Pad1.08x0.95mm_HandSolder, F.Cu at (76.1, -10.2)
- added C1413: 100n, Capacitor_SMD:C_0603_1608Metric_Pad1.08x0.95mm_HandSolder, F.Cu at (91.1, -7.15)
- added C1414: 100n, Capacitor_SMD:C_0603_1608Metric_Pad1.08x0.95mm_HandSolder, F.Cu at (73.7, -7.73)
- added C1415: 100n, Capacitor_SMD:C_0603_1608Metric_Pad1.08x0.95mm_HandSolder, F.Cu at (80.9, -14.9)
- added C1416: 1000p, Capacitor_SMD:C_0603_1608Metric_Pad1.08x0.95mm_HandSolder, F.Cu at (69.3, -1.78)
- added C1417: 100n, Capacitor_SMD:C_0603_1608Metric_Pad1.08x0.95mm_HandSolder, F.Cu at (73.7, -5.22)
- added C1418: 100n, Capacitor_SMD:C_0603_1608Metric_Pad1.08x0.95mm_HandSolder, F.Cu at (80.9, -12.4)
- added C1419: 47p, Capacitor_SMD:C_0603_1608Metric_Pad1.08x0.95mm_HandSolder, F.Cu at (88.7, -19.7)
- added C1420: 100n, Capacitor_SMD:C_0603_1608Metric_Pad1.08x0.95mm_HandSolder, F.Cu at (68.1, 0.73)
- added C1421: 100n, Capacitor_SMD:C_0603_1608Metric_Pad1.08x0.95mm_HandSolder, F.Cu at (78.0, -7.73)
- added C1422: 100n, Capacitor_SMD:C_0603_1608Metric_Pad1.08x0.95mm_HandSolder, F.Cu at (85.3, -17.2)
- added C1423: 100n, Capacitor_SMD:C_0603_1608Metric_Pad1.08x0.95mm_HandSolder, F.Cu at (73.7, -2.71)
- added C1424: 100n, Capacitor_SMD:C_0603_1608Metric_Pad1.08x0.95mm_HandSolder, F.Cu at (71.8, -10.2)
- added C1425: 330p, Capacitor_SMD:C_0603_1608Metric_Pad1.08x0.95mm_HandSolder, F.Cu at (91.1, -9.66)
- added C1501: 22u, Capacitor_SMD:C_0805_2012Metric_Pad1.18x1.45mm_HandSolder, F.Cu at (69.6, 16.0)
- added C1502: 1u, Capacitor_SMD:C_0603_1608Metric_Pad1.08x0.95mm_HandSolder, F.Cu at (78.7, 29.4)
- added C1503: 10u, Capacitor_SMD:C_0805_2012Metric_Pad1.18x1.45mm_HandSolder, F.Cu at (52.4, 29.2)
- added C1504: 100n, Capacitor_SMD:C_0603_1608Metric_Pad1.08x0.95mm_HandSolder, F.Cu at (84.3, 26.9)
- added C1505: 100n, Capacitor_SMD:C_0603_1608Metric_Pad1.08x0.95mm_HandSolder, F.Cu at (74.4, 28.8)
- added C1506: 100n, Capacitor_SMD:C_0603_1608Metric_Pad1.08x0.95mm_HandSolder, F.Cu at (57.0, 28.9)
- added C1507: 100n, Capacitor_SMD:C_0603_1608Metric_Pad1.08x0.95mm_HandSolder, F.Cu at (66.9, 22.2)
- added C1508: 330p, Capacitor_SMD:C_0603_1608Metric_Pad1.08x0.95mm_HandSolder, F.Cu at (74.2, 15.8)
- added C1509: 100n, Capacitor_SMD:C_0603_1608Metric_Pad1.08x0.95mm_HandSolder, F.Cu at (66.9, 24.7)
- added C1510: 100n, Capacitor_SMD:C_0603_1608Metric_Pad1.08x0.95mm_HandSolder, F.Cu at (61.3, 28.8)
- added C1511: 100p, Capacitor_SMD:C_0603_1608Metric_Pad1.08x0.95mm_HandSolder, F.Cu at (82.0, 9.30)
- added C1512: 100n, Capacitor_SMD:C_0603_1608Metric_Pad1.08x0.95mm_HandSolder, F.Cu at (73.7, 18.8)
- added C1513: 100n, Capacitor_SMD:C_0603_1608Metric_Pad1.08x0.95mm_HandSolder, F.Cu at (88.7, 21.9)
- added C1514: 100n, Capacitor_SMD:C_0603_1608Metric_Pad1.08x0.95mm_HandSolder, F.Cu at (71.3, 21.3)
- added C1515: 100n, Capacitor_SMD:C_0603_1608Metric_Pad1.08x0.95mm_HandSolder, F.Cu at (78.5, 14.1)
- added C1516: 1000p, Capacitor_SMD:C_0603_1608Metric_Pad1.08x0.95mm_HandSolder, F.Cu at (66.9, 27.2)
- added C1517: 100n, Capacitor_SMD:C_0603_1608Metric_Pad1.08x0.95mm_HandSolder, F.Cu at (71.3, 23.8)
- added C1518: 100n, Capacitor_SMD:C_0603_1608Metric_Pad1.08x0.95mm_HandSolder, F.Cu at (78.5, 16.6)
- added C1519: 47p, Capacitor_SMD:C_0603_1608Metric_Pad1.08x0.95mm_HandSolder, F.Cu at (86.3, 9.30)
- added C1520: 100n, Capacitor_SMD:C_0603_1608Metric_Pad1.08x0.95mm_HandSolder, F.Cu at (65.7, 29.7)
- added C1521: 100n, Capacitor_SMD:C_0603_1608Metric_Pad1.08x0.95mm_HandSolder, F.Cu at (75.6, 21.3)
- added C1522: 100n, Capacitor_SMD:C_0603_1608Metric_Pad1.08x0.95mm_HandSolder, F.Cu at (82.9, 11.8)
- added C1523: 100n, Capacitor_SMD:C_0603_1608Metric_Pad1.08x0.95mm_HandSolder, F.Cu at (71.3, 26.3)
- added C1524: 100n, Capacitor_SMD:C_0603_1608Metric_Pad1.08x0.95mm_HandSolder, F.Cu at (69.4, 18.8)
- added C1525: 330p, Capacitor_SMD:C_0603_1608Metric_Pad1.08x0.95mm_HandSolder, F.Cu at (88.7, 19.3)
- added C321: 100n, Capacitor_SMD:C_0603_1608Metric_Pad1.08x0.95mm_HandSolder, F.Cu at (144.3, 3.55)
- added C324: 100n, Capacitor_SMD:C_0603_1608Metric_Pad1.08x0.95mm_HandSolder, F.Cu at (139.9, 3.55)
- added C701: 1u, Capacitor_SMD:C_0603_1608Metric_Pad1.08x0.95mm_HandSolder, F.Cu at (153.5, 6.99)
- added C702: 1u, Capacitor_SMD:C_0603_1608Metric_Pad1.08x0.95mm_HandSolder, F.Cu at (161.9, 3.55)
- added C703: 10u, Capacitor_SMD:C_0805_2012Metric_Pad1.18x1.45mm_HandSolder, F.Cu at (162.2, 0.79)
- added C801: 10u, Capacitor_SMD:C_0805_2012Metric_Pad1.18x1.45mm_HandSolder, F.Cu at (123.2, 33.6)
- added C802: 10u, Capacitor_SMD:C_0805_2012Metric_Pad1.18x1.45mm_HandSolder, F.Cu at (122.9, 30.6)
- added C803: 100n, Capacitor_SMD:C_0603_1608Metric_Pad1.08x0.95mm_HandSolder, F.Cu at (127.4, 36.4)
- added C804: 100n, Capacitor_SMD:C_0603_1608Metric_Pad1.08x0.95mm_HandSolder, F.Cu at (132.2, 33.4)
- added C805: 4u7, Capacitor_SMD:C_0805_2012Metric_Pad1.18x1.45mm_HandSolder, F.Cu at (131.4, 24.2)
- added C806: 4u7, Capacitor_SMD:C_0805_2012Metric_Pad1.18x1.45mm_HandSolder, F.Cu at (127.8, 30.6)
- added C807: 100n, Capacitor_SMD:C_0603_1608Metric_Pad1.08x0.95mm_HandSolder, F.Cu at (136.7, 28.9)
- added C808: 220n, Capacitor_SMD:C_0603_1608Metric_Pad1.08x0.95mm_HandSolder, F.Cu at (140.3, 26.4)
- added C809: 220n, Capacitor_SMD:C_0603_1608Metric_Pad1.08x0.95mm_HandSolder, F.Cu at (127.4, 38.9)
- added C810: 220n, Capacitor_SMD:C_0603_1608Metric_Pad1.08x0.95mm_HandSolder, F.Cu at (131.7, 35.9)
- added C811: 1n, Capacitor_SMD:C_0603_1608Metric_Pad1.08x0.95mm_HandSolder, F.Cu at (136.5, 31.9)
- added C812: 1n, Capacitor_SMD:C_0603_1608Metric_Pad1.08x0.95mm_HandSolder, F.Cu at (144.7, 23.9)
- added C813: 1n, Capacitor_SMD:C_0603_1608Metric_Pad1.08x0.95mm_HandSolder, F.Cu at (141.0, 28.9)
- added C901: 10u, Capacitor_SMD:C_1206_3216Metric_Pad1.33x1.80mm_HandSolder, F.Cu at (162.7, 24.3)
- added C902: 10u, Capacitor_SMD:C_1206_3216Metric_Pad1.33x1.80mm_HandSolder, F.Cu at (162.7, 27.7)
- added FB801: MPZ1608S221ATA00, Resistor_SMD:R_0603_1608Metric_Pad0.98x0.95mm_HandSolder, F.Cu at (131.7, 38.4)
- added FB802: MPZ1608S221ATA00, Resistor_SMD:R_0603_1608Metric_Pad0.98x0.95mm_HandSolder, F.Cu at (140.4, 37.0)
- added J1101: Conn_02x10_Odd_Even, Connector_PinSocket_2.54mm:PinSocket_2x10_P2.54mm_Vertical, B.Cu at (153.0, 56.0)
- added J1201: Conn_02x10_Odd_Even, Connector_PinSocket_2.54mm:PinSocket_2x10_P2.54mm_Vertical, B.Cu at (153.0, 89.0)
- added J1301: Conn_02x10_Odd_Even, Connector_PinSocket_2.54mm:PinSocket_2x10_P2.54mm_Vertical, B.Cu at (153.0, 122.0)
- added R1401: 0, Resistor_SMD:R_0603_1608Metric_Pad0.98x0.95mm_HandSolder, F.Cu at (89.6, -17.2)
- added R1402: 10k, Resistor_SMD:R_0603_1608Metric_Pad0.98x0.95mm_HandSolder, F.Cu at (85.3, -12.2)
- added R1403: 10k, Resistor_SMD:R_0603_1608Metric_Pad0.98x0.95mm_HandSolder, F.Cu at (72.4, 0.73)
- added R1404: 49R9, Resistor_SMD:R_0603_1608Metric_Pad0.98x0.95mm_HandSolder, F.Cu at (82.4, -9.66)
- added R1405: 0R22, Resistor_SMD:R_0603_1608Metric_Pad0.98x0.95mm_HandSolder, F.Cu at (78.0, -2.71)
- added R1406: 0R47, Resistor_SMD:R_0603_1608Metric_Pad0.98x0.95mm_HandSolder, F.Cu at (82.4, -7.15)
- added R1407: 6k81, Resistor_SMD:R_0603_1608Metric_Pad0.98x0.95mm_HandSolder, F.Cu at (89.6, -14.7)
- added R1408: 11k3, Resistor_SMD:R_0603_1608Metric_Pad0.98x0.95mm_HandSolder, F.Cu at (86.7, -9.66)
- added R1409: 6k81, Resistor_SMD:R_0603_1608Metric_Pad0.98x0.95mm_HandSolder, F.Cu at (89.6, -12.2)
- added R1410: 5k23, Resistor_SMD:R_0603_1608Metric_Pad0.98x0.95mm_HandSolder, F.Cu at (78.0, -5.22)
- added R1411: 10k2, Resistor_SMD:R_0603_1608Metric_Pad0.98x0.95mm_HandSolder, F.Cu at (82.4, -4.64)
- added R1412: 5k23, Resistor_SMD:R_0603_1608Metric_Pad0.98x0.95mm_HandSolder, F.Cu at (86.7, -7.15)
- added R1413: 0, Resistor_SMD:R_0603_1608Metric_Pad0.98x0.95mm_HandSolder, F.Cu at (85.3, -14.7)
- added R1414: 680, Resistor_SMD:R_Array_Convex_4x0603, F.Cu at (80.1, -18.6)
- added R1415: 10k, Resistor_SMD:R_0603_1608Metric_Pad0.98x0.95mm_HandSolder, F.Cu at (82.4, -2.13)
- added R1416: 10k, Resistor_SMD:R_0603_1608Metric_Pad0.98x0.95mm_HandSolder, F.Cu at (86.7, -4.64)
- added R1501: 0, Resistor_SMD:R_0603_1608Metric_Pad0.98x0.95mm_HandSolder, F.Cu at (87.2, 11.8)
- added R1502: 10k, Resistor_SMD:R_0603_1608Metric_Pad0.98x0.95mm_HandSolder, F.Cu at (82.9, 16.8)
- added R1503: 10k, Resistor_SMD:R_0603_1608Metric_Pad0.98x0.95mm_HandSolder, F.Cu at (70.0, 29.7)
- added R1504: 49R9, Resistor_SMD:R_0603_1608Metric_Pad0.98x0.95mm_HandSolder, F.Cu at (80.0, 19.3)
- added R1505: 0R22, Resistor_SMD:R_0603_1608Metric_Pad0.98x0.95mm_HandSolder, F.Cu at (75.6, 26.3)
- added R1506: 0R47, Resistor_SMD:R_0603_1608Metric_Pad0.98x0.95mm_HandSolder, F.Cu at (80.0, 21.9)
- added R1507: 6k81, Resistor_SMD:R_0603_1608Metric_Pad0.98x0.95mm_HandSolder, F.Cu at (87.2, 14.3)
- added R1508: 11k3, Resistor_SMD:R_0603_1608Metric_Pad0.98x0.95mm_HandSolder, F.Cu at (84.3, 19.3)
- added R1509: 6k81, Resistor_SMD:R_0603_1608Metric_Pad0.98x0.95mm_HandSolder, F.Cu at (87.2, 16.8)
- added R1510: 5k23, Resistor_SMD:R_0603_1608Metric_Pad0.98x0.95mm_HandSolder, F.Cu at (75.6, 23.8)
- added R1511: 10k2, Resistor_SMD:R_0603_1608Metric_Pad0.98x0.95mm_HandSolder, F.Cu at (80.0, 24.4)
- added R1512: 5k23, Resistor_SMD:R_0603_1608Metric_Pad0.98x0.95mm_HandSolder, F.Cu at (84.3, 21.9)
- added R1513: 0, Resistor_SMD:R_0603_1608Metric_Pad0.98x0.95mm_HandSolder, F.Cu at (82.9, 14.3)
- added R1514: 680, Resistor_SMD:R_Array_Convex_4x0603, F.Cu at (77.7, 10.4)
- added R1515: 10k, Resistor_SMD:R_0603_1608Metric_Pad0.98x0.95mm_HandSolder, F.Cu at (80.0, 26.9)
- added R1516: 10k, Resistor_SMD:R_0603_1608Metric_Pad0.98x0.95mm_HandSolder, F.Cu at (84.3, 24.4)
- added R304: 49R9, Resistor_SMD:R_0603_1608Metric_Pad0.98x0.95mm_HandSolder, F.Cu at (129.0, 15.9)
- added R305: 0R22, Resistor_SMD:R_0603_1608Metric_Pad0.98x0.95mm_HandSolder, F.Cu at (135.8, 10.00)
- added R306: 0R47, Resistor_SMD:R_0603_1608Metric_Pad0.98x0.95mm_HandSolder, F.Cu at (133.4, 12.5)
- added R314: 680, Resistor_SMD:R_Array_Convex_4x0603, F.Cu at (163.7, 76.5)
- added R701: 0R22, Resistor_SMD:R_0603_1608Metric_Pad0.98x0.95mm_HandSolder, F.Cu at (157.8, 6.99)
- added R801: 27, Resistor_SMD:R_0603_1608Metric_Pad0.98x0.95mm_HandSolder, F.Cu at (123.0, 36.4)
- added R802: 27, Resistor_SMD:R_0603_1608Metric_Pad0.98x0.95mm_HandSolder, F.Cu at (118.6, 40.7)
- added R803: 27, Resistor_SMD:R_0603_1608Metric_Pad0.98x0.95mm_HandSolder, F.Cu at (131.2, 26.9)
- added R804: 27, Resistor_SMD:R_0603_1608Metric_Pad0.98x0.95mm_HandSolder, F.Cu at (136.5, 34.4)
- added R805: 10, Resistor_SMD:R_0603_1608Metric_Pad0.98x0.95mm_HandSolder, F.Cu at (127.8, 33.4)
- added R806: 1k, Resistor_SMD:R_0603_1608Metric_Pad0.98x0.95mm_HandSolder, F.Cu at (136.1, 39.5)
- added R807: 1k, Resistor_SMD:R_0603_1608Metric_Pad0.98x0.95mm_HandSolder, F.Cu at (140.9, 33.9)
- added R808: 1k, Resistor_SMD:R_0603_1608Metric_Pad0.98x0.95mm_HandSolder, F.Cu at (136.1, 37.0)
- added R809: 24k9, Resistor_SMD:R_0603_1608Metric_Pad0.98x0.95mm_HandSolder, F.Cu at (131.7, 40.9)
- added R810: 33k2, Resistor_SMD:R_0603_1608Metric_Pad0.98x0.95mm_HandSolder, F.Cu at (140.9, 31.4)
- added R811: 24k9, Resistor_SMD:R_0603_1608Metric_Pad0.98x0.95mm_HandSolder, F.Cu at (140.3, 23.9)
- added R812: 33k2, Resistor_SMD:R_0603_1608Metric_Pad0.98x0.95mm_HandSolder, F.Cu at (144.7, 26.4)
- added R813: 24k9, Resistor_SMD:R_0603_1608Metric_Pad0.98x0.95mm_HandSolder, F.Cu at (123.0, 38.9)
- added R814: 33k2, Resistor_SMD:R_0603_1608Metric_Pad0.98x0.95mm_HandSolder, F.Cu at (136.0, 26.4)
- added R815: 100k, Resistor_SMD:R_0603_1608Metric_Pad0.98x0.95mm_HandSolder, F.Cu at (132.3, 29.4)
- added R816: 100k, Resistor_SMD:R_0603_1608Metric_Pad0.98x0.95mm_HandSolder, F.Cu at (136.0, 23.9)
- added R817: 100k, Resistor_SMD:R_0603_1608Metric_Pad0.98x0.95mm_HandSolder, F.Cu at (114.3, 40.7)
- added U1401: LT1355, Package_SO:SOIC-8_3.9x4.9mm_P1.27mm, F.Cu at (73.8, -17.7)
- added U1402: DG211, Package_SO:TSSOP-16_4.4x5mm_P0.65mm, F.Cu at (56.8, -11.1)
- added U1403: DG419LDY, Package_SO:SOIC-8_3.9x4.9mm_P1.27mm, F.Cu at (65.4, -11.3)
- added U1404: DG419LDY, Package_SO:SOIC-8_3.9x4.9mm_P1.27mm, F.Cu at (56.6, -4.55)
- added U1405: OPA192, Package_SO:SOIC-8_3.9x4.9mm_P1.27mm, F.Cu at (65.4, -17.7)
- added U1406: 74LVC1GU04DRL, Package_TO_SOT_SMD:SOT-553, F.Cu at (90.6, -4.27)
- added U1407: ADS8681RUM, Package_DFN_QFN:QFN-16-1EP_4x4mm_P0.65mm_EP2.7x2.7mm, F.Cu at (64.0, -4.63)
- added U1408: 74HCT595, Package_SO:TSSOP-16_4.4x5mm_P0.65mm, F.Cu at (56.8, -17.7)
- added U1501: LT1355, Package_SO:SOIC-8_3.9x4.9mm_P1.27mm, F.Cu at (71.4, 11.3)
- added U1502: DG211, Package_SO:TSSOP-16_4.4x5mm_P0.65mm, F.Cu at (54.4, 17.9)
- added U1503: DG419LDY, Package_SO:SOIC-8_3.9x4.9mm_P1.27mm, F.Cu at (63.0, 17.7)
- added U1504: DG419LDY, Package_SO:SOIC-8_3.9x4.9mm_P1.27mm, F.Cu at (54.2, 24.5)
- added U1505: OPA192, Package_SO:SOIC-8_3.9x4.9mm_P1.27mm, F.Cu at (63.0, 11.3)
- added U1506: 74LVC1GU04DRL, Package_TO_SOT_SMD:SOT-553, F.Cu at (88.2, 24.7)
- added U1507: ADS8681RUM, Package_DFN_QFN:QFN-16-1EP_4x4mm_P0.65mm_EP2.7x2.7mm, F.Cu at (61.6, 24.4)
- added U1508: 74HCT595, Package_SO:TSSOP-16_4.4x5mm_P0.65mm, F.Cu at (54.4, 11.3)
- added U701: REF5040ID, Package_SO:SOIC-8_3.9x4.9mm_P1.27mm, F.Cu at (182.4, 126.4)
- added U801: TL074, Package_SO:SOIC-14_3.9x8.7mm_P1.27mm, F.Cu at (190.8, 135.4)
- added U802: DAC8564, Package_SO:TSSOP-16_4.4x5mm_P0.65mm, F.Cu at (201.5, 131.3)
- added U803: TL071, Package_SO:SOIC-8_3.9x4.9mm_P1.27mm, F.Cu at (190.8, 126.4)
- added U901: LM1117-5.0, Package_TO_SOT_SMD:SOT-223-3_TabPin2, F.Cu at (211.3, 133.7)
- C301: value 100n -> 22u; footprint Capacitor_SMD:C_0603_1608Metric_Pad1.08x0.95mm_HandSolder -> Capacitor_SMD:C_0805_2012Metric_Pad1.18x1.45mm_HandSolder
- C302: value 100n -> 1u
- C303: value 100n -> 10u; footprint Capacitor_SMD:C_0603_1608Metric_Pad1.08x0.95mm_HandSolder -> Capacitor_SMD:C_0805_2012Metric_Pad1.18x1.45mm_HandSolder
- C323: value 2u2 -> 100n
- C325: value C -> 330p
- R315: value DNP -> 10k
- R316: value 620 -> 10k
- R405: moved to B.Cu
- U304: value OPA140 -> DG419LDY
- U305: value DG419LDY -> OPA192
- U306: value AD8251 -> 74LVC1GU04DRL; footprint Package_SO:MSOP-10_3x3mm_P0.5mm -> Package_TO_SOT_SMD:SOT-553
- U307: value SN74LVC1G14DBVR -> ADS8681RUM; footprint Package_TO_SOT_SMD:SOT-23-5 -> Package_DFN_QFN:QFN-16-1EP_4x4mm_P0.65mm_EP2.7x2.7mm
- U308: value SN74LVC1G14DBVR -> 74HCT595; footprint Package_TO_SOT_SMD:SOT-23-5 -> Package_SO:TSSOP-16_4.4x5mm_P0.65mm
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- renumbered C311 to C308, C316 to C311, C321 to C316, C324 to C319, J702 to J1001, J704 to J1002, R304 to R301, R305 to R302, R306 to R303, R308 to R307, R309 to R308, R310 to R309, R311 to R310, R312 to R311, R313 to R312, R314 to R313
Connections:
- C228 pad 1: /MCU/NRST -> /Ethernet/NRST
- C301 pad 1: -15V -> Net-(C301-Pad1)
- C301 pad 2: GNDA -> GND
- C302 pad 1: +5V -> Net-(C301-Pad1)
- C302 pad 2: GNDA -> GND
- C303 pad 1: -15V -> Net-(C303-Pad1)
- C303 pad 2: GNDA -> GND
- C304 pad 2: GNDA -> GND
- C305 pad 1: -15V -> +18V
- C305 pad 2: GNDA -> GND
- C306 pad 2: GNDA -> GND
- C307 pad 1: -15V -> +18V
- C307 pad 2: GNDA -> GND
- C308 pad 2: GNDA -> GND
- C309 pad 1: -15V -> +5V
- C309 pad 2: GNDA -> GND
- C310 pad 1: +5V -> +18V
- C310 pad 2: GNDA -> GND
- C312 pad 1: +15V -> +5V
- C312 pad 2: GNDA -> GND
- C313 pad 1: +5V -> +18V
- C313 pad 2: GNDA -> GND
- C314 pad 1: +15V -> +5V
- C314 pad 2: GNDA -> GND
- C315 pad 1: +5V -> +18V
- C315 pad 2: GNDA -> GND
- C316 pad 2: GNDA -> GND
- C317 pad 1: +15V -> +5V
- C317 pad 2: GNDA -> GND
- C318 pad 1: +5V -> -18V
- C318 pad 2: GNDA -> GND
- C319 pad 1: Net-(C324-Pad1) -> Net-(C319-Pad1)
- C320 pad 1: -2V5 -> +3V3
- C320 pad 2: GNDA -> GND
- C322 pad 1: +15V -> -18V
- C322 pad 2: GNDA -> GND
- C323 pad 1: +5V -> -18V
- C323 pad 2: GNDA -> GND
- C325 pad 2: GNDA -> GND
- C409 pad 1: /Trigger/EXT_TRIG -> /Connector 1/EXT_TRIG
- D403 pad 1: /Trigger/EXT_TRIG -> /Connector 1/EXT_TRIG
- J1001 pad 1: (no net) -> /Connector 1/EXT_TRIG
- J1001 pad 2: (no net) -> /Connector 1/EXT_TRIG
- J1001 pad 3: (no net) -> GND_TRIG
- J1001 pad 4: (no net) -> GND_TRIG
- J1002 pad 1: (no net) -> Earth
- J1002 pad 2: (no net) -> Earth
- J1002 pad 3: (no net) -> /Connector 1/RX+
- J1002 pad 4: (no net) -> /Connector 1/TX+
- J1002 pad 5: (no net) -> /Connector 1/RX-
- J1002 pad 6: (no net) -> /Connector 1/TX-
- J1002 pad 7: (no net) -> Earth
- J1002 pad 8: (no net) -> Earth
- J201 pad 10: /MCU/NRST -> /Ethernet/NRST
- L401 pad 1: /Trigger/EXT_TRIG -> /Connector 1/EXT_TRIG
- R209 pad 2: /MCU/NRST -> /Ethernet/NRST
- R301 pad 2: Net-(R303-Pad1) (its old number) -> /CH1 Connector/CH1_IN
- R302 pad 2: GNDA -> GND
- R303 pad 2: (no net) -> /Channel 1/DAC_V1
- R312 pad 1: Net-(C324-Pad1) -> Net-(C319-Pad1)
- R313 pad 1: Net-(R314-Pad1) -> Net-(C325-Pad1)
- R313 pad 2: Net-(R314-Pad2) -> Net-(R313-Pad2)
- R315 pad 1: GNDA -> +3V3
- R315 pad 2: Net-(R314-Pad1) -> Net-(R315-Pad2)
- R316 pad 1: Net-(R316-Pad1) -> +3V3
- R316 pad 2: /Channel 1/CH1_A1 -> /Channel 1/ADC1_SDO
- R601 pad 2: (no net) -> /Ethernet/RMII_RXD0
- R602 pad 2: (no net) -> /Ethernet/RMII_RXD1
- R604 pad 2: (no net) -> /Ethernet/RMII_CRS_DV
- R605 pad 2: (no net) -> /Ethernet/REF_CLK
- U202 pad 3: (no net) -> /MCU/SD_DAT
- U203 pad 3: (no net) -> /MCU/SD_CLK
- U204 pad 3: (no net) -> /MCU/SD_LAT
- U205 pad 10: (no net) -> /MCU/A0
- U205 pad 11: (no net) -> /MCU/A1
- U205 pad 110: (no net) -> /Channel 1/ADC1_~CS
- U205 pad 111: (no net) -> /Channel 1/ADC1_SCLK
- U205 pad 113: (no net) -> /Channel 1/ADC1_SDI
- U205 pad 114: (no net) -> /MCU/D2
- U205 pad 115: (no net) -> /MCU/D3
- U205 pad 12: (no net) -> /MCU/A2
- U205 pad 126: (no net) -> /Ethernet/RMII_TXEN
- U205 pad 128: (no net) -> /Ethernet/RMII_TXD0
- U205 pad 129: (no net) -> /Ethernet/RMII_TXD1
- U205 pad 13: (no net) -> /MCU/A3
- U205 pad 132: (no net) -> /MCU/~CAS
- U205 pad 135: (no net) -> /MCU/CKE
- U205 pad 136: (no net) -> /MCU/~CS
- U205 pad 14: (no net) -> /MCU/A4
- U205 pad 141: (no net) -> /MCU/LDQM
- U205 pad 142: (no net) -> /MCU/UDQM
- U205 pad 15: (no net) -> /MCU/A5
- U205 pad 25: /MCU/NRST -> /Ethernet/NRST
- U205 pad 26: (no net) -> /MCU/~WE
- U205 pad 27: (no net) -> /Ethernet/RMII_MDC
- U205 pad 35: (no net) -> /Ethernet/REF_CLK
- U205 pad 36: (no net) -> /Ethernet/RMII_MDIO
- U205 pad 43: (no net) -> /Ethernet/RMII_CRS_DV
- U205 pad 44: (no net) -> /Ethernet/RMII_RXD0
- U205 pad 45: (no net) -> /Ethernet/RMII_RXD1
- U205 pad 49: (no net) -> /MCU/~RAS
- U205 pad 50: (no net) -> /MCU/A6
- U205 pad 53: (no net) -> /MCU/A7
- U205 pad 54: (no net) -> /MCU/A8
- U205 pad 55: (no net) -> /MCU/A9
- U205 pad 56: (no net) -> /MCU/A10
- U205 pad 57: (no net) -> /MCU/A11
- U205 pad 58: (no net) -> /MCU/D4
- U205 pad 59: (no net) -> /MCU/D5
- U205 pad 60: (no net) -> /MCU/D6
- U205 pad 63: (no net) -> /MCU/D7
- U205 pad 64: (no net) -> /MCU/D8
- U205 pad 65: (no net) -> /MCU/D9
- U205 pad 66: (no net) -> /MCU/D10
- U205 pad 67: (no net) -> /MCU/D11
- U205 pad 68: (no net) -> /MCU/D12
- U205 pad 69: (no net) -> /MCU/TRIG_IN
- U205 pad 70: (no net) -> /MCU/TRIG_OUT
- U205 pad 73: (no net) -> /MCU/TRIG_EN
- U205 pad 77: (no net) -> /MCU/D13
- U205 pad 78: (no net) -> /MCU/D14
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Routing:
- added copper zone on GND, net GND
Other:
- copper layers 4 -> 6

Commit message: PCB layout
Parts:
- removed the R801 at (123.0, 36.4)
- removed the R802 at (118.6, 40.7)
- removed the R803 at (131.2, 26.9)
- removed the R804 at (136.5, 34.4)
- C1405, C1406, C1407, C1408, C1409, C1410, C1413, C1415, C1417, C1418, C1419, C1421, C1422, C1423, C1424, C201, C202, C203, C204, C205, C206, C207, C208, C209, C210, C211, C212, C213, C214, C215, C216, C217, C218, C219, C220, C221, C222, C223, C224, C225, C226, C227, C228, C301, C303, C304, C305, C306, C307, C308, C309, C310, C312, C313, C314, C315, C317, C318, C319, C320, C321, C322, C323, C324, C325, C401, C402, C403, C404, C405, C406, C407, C408, C409, C501, C502, C503, C504, C505, C506, C507, C601, C602, C603, C604, C605, C610, C611, C612, C613, C614, C701, C702, C801, C901, C902, FB201, FB601, R1409, R1414, R201, R202, R203, R204, R205, R206, R207, R208, R209, R210, R302, R304, R309, R311, R313, R314, R315, R316, R401, R402, R403, R404, R406, R606, R607, R608, R609, R611, R612, R613, R614, R615, R616, R617, R618, R619, R620, R621, U1406, U306, Y201: moved to B.Cu
- D403: moved to F.Cu
- U501: value IS42S16400J-xC -> IS42S16400J-xC/MT48LC16M16A2P-6A
- moved R801 182.7 mm to (258.2, 161.4), turned to 90 degrees
- moved C801 175.2 mm to (251.0, 153.5)
- moved C805 170.9 mm to (270.8, 123.0)
- moved C810 170.9 mm to (271.2, 134.7)
- moved C811 170.9 mm to (276.0, 130.7)
- moved C813 170.9 mm to (280.5, 127.7)
- moved R805 170.9 mm to (271.2, 139.7)
- moved R811 170.9 mm to (271.8, 128.2)
- moved C803 170.9 mm to (266.8, 135.2)
- moved C804 170.9 mm to (271.6, 132.2)
- moved C807 170.9 mm to (276.1, 127.7)
- moved C809 170.9 mm to (266.8, 137.7)
- moved C812 170.9 mm to (284.1, 122.7)
- moved FB801 170.9 mm to (271.2, 137.2)
- moved FB802 170.9 mm to (279.9, 135.8)
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- renumbered R805 to R801, R806 to R802, R807 to R803, R808 to R804, R809 to R805, R810 to R806, R811 to R807, R812 to R808, R813 to R809, R814 to R810, R815 to R811, R816 to R812, R817 to R813
Connections:
- U307 pad 16: +5VF -> +5V
- U802 pad 10: Net-(R803-Pad1) -> (no net)
- U802 pad 11: Net-(R802-Pad1) -> (no net)
- U802 pad 16: Net-(R804-Pad1) -> (no net)
- U802 pad 9: Net-(R801-Pad1) -> (no net)
Routing:
- added copper zone on B.Cu, net Earth
- added copper zone on F.Cu, net Earth
- added copper zone on B.Cu, net GND_TRIG
- added copper zone on F.Cu, net GND_TRIG
- added copper zone on GND, net GND_TRIG
Other:
- outline, holes or cut-outs redrawn

Commit message: PCB design
Parts:
- added C814: 100n, Capacitor_SMD:C_0603_1608Metric_Pad1.08x0.95mm_HandSolder, F.Cu at (186.7, 127.0)
- added C815: 100n, Capacitor_SMD:C_0603_1608Metric_Pad1.08x0.95mm_HandSolder, F.Cu at (198.6, 127.0)
- C1401, C1403, C1404, C1412, C1414, C1416, C1420, C1425, C1501, C1503, C1504, C1505, C1506, C1507, C1508, C1509, C1510, C1512, C1513, C1514, C1515, C1516, C1517, C1518, C1519, C1520, C1521, C1522, C1523, C1524, C1525, C316, C703, C802, C803, C804, C805, C806, C808, C809, C810, C811, C812, C813, FB801, FB802, R1402, R1404, R1411, R1413, R1415, R1416, R1502, R1504, R1509, R1511, R1513, R1514, R1515, R1516, R701, R802, R803, R804, R806, R808, R810, U1506: moved to B.Cu
- moved R1514 182.7 mm to (159.9, 142.9), turned to 180 degrees
- moved U1508 182.3 mm to (161.5, 143.9)
- moved C1515 175.2 mm to (159.0, 138.8), turned to 90 degrees
- moved C1501 174.5 mm to (167.3, 141.0), turned to 90 degrees
- moved R1501 173.9 mm to (159.5, 134.2), turned to 180 degrees
- moved U1506 173.1 mm to (159.3, 146.2)
- moved C1517 172.1 mm to (162.2, 146.2), turned to 90 degrees
- moved C1525 171.8 mm to (170.4, 140.8)
- moved R1513 170.3 mm to (163.6, 134.2), turned to 180 degrees
- moved C1519 169.3 mm to (174.8, 128.8), turned to 270 degrees
- moved C1522 169.1 mm to (158.6, 129.9), turned to 270 degrees
- moved C1511 169.1 mm to (174.8, 128.8), turned to 90 degrees
- moved U1501 167.7 mm to (170.1, 129.4)
- moved C1521 167.4 mm to (164.0, 138.8), turned to 270 degrees
- moved C1514 167.3 mm to (161.4, 138.8), turned to 90 degrees
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Connections:
- C813 pad 1: /DAC/DAC_V3 -> /Channel 3/DAC_V3
- R1501 pad 2: (no net) -> /CH3 Connector/CH3_IN
- R1503 pad 2: (no net) -> /Channel 3/DAC_V3
- R813 pad 1: /DAC/DAC_V3 -> /Channel 3/DAC_V3
- U1407 pad 16: +5VF -> +5V
- U1408 pad 9: (no net) -> /Channel 2/SR2_QH
- U1507 pad 10: (no net) -> /Channel 1/ADC1_SCLK
- U1507 pad 16: +5VF -> +5V
- U1507 pad 8: (no net) -> /Channel 2/ADC2_SDO
- U1507 pad 9: (no net) -> /Channel 1/ADC1_~CS
- U1508 pad 11: (no net) -> /MCU/SD_CLK
- U1508 pad 12: (no net) -> /MCU/SD_LAT
- U1508 pad 14: (no net) -> /Channel 2/SR2_QH
- U205 pad 112: (no net) -> /Channel 3/ADC3_SDO
- U801 pad 8: /DAC/DAC_V3 -> /Channel 3/DAC_V3
Routing:
- net +3V3: track 0.00 -> 69.9 mm, vias 0 -> 30
- net /Ethernet/NRST: track 0.00 -> 61.0 mm, vias 0 -> 3
- net Net-(U303-Pad6): track 0.00 -> 33.8 mm, vias 0 -> 1
- net /Ethernet/RMII_TXD0: track 0.00 -> 32.5 mm, vias 0 -> 2
- net /Ethernet/RMII_RXD0: track 0.00 -> 32.4 mm, vias 0 -> 2
- net /Ethernet/RMII_RXD1: track 0.00 -> 32.4 mm, vias 0 -> 2
- net /Ethernet/RMII_CRS_DV: track 0.00 -> 32.4 mm, vias 0 -> 2
- net /Ethernet/REF_CLK: track 0.00 -> 32.4 mm, vias 0 -> 2
- net /Ethernet/RMII_TXD1: track 0.00 -> 32.4 mm, vias 0 -> 2
- net /Ethernet/RMII_TXEN: track 0.00 -> 32.3 mm, vias 0 -> 2
- net /Ethernet/RMII_MDC: track 0.00 -> 31.8 mm, vias 0 -> 2
- net /MCU/TCK_SWCLK: track 0.00 -> 28.9 mm, vias 0 -> 1
- net /MCU/TMS_SWDIO: track 0.00 -> 25.1 mm, vias 0 -> 1
- net +5V: track 0.00 -> 24.4 mm, vias 0 -> 8
- net Net-(U303-Pad2): track 0.00 -> 22.4 mm
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- added copper zone on POWER_A, net (none)
- added copper zone on POWER_A, net +18V
- added copper zone on POWER_B, net +3V3
- added copper zone on POWER_B, net +5V
- added copper zone on B.Cu, net +5VF
- added copper zone on F.Cu, net +5VF
- added copper zone on POWER_A, net +5V_TRIG
- added copper zone on B.Cu, net +9V
- added copper zone on F.Cu, net +9V
- added copper zone on POWER_B, net +9V
- added copper zone on POWER_A, net -18V
- added copper zone on B.Cu, net GND
- added copper zone on F.Cu, net GND
- added copper zone on POWER_A, net VCCQ
- removed copper zone on B.Cu, net Earth
Other:
- outline, holes or cut-outs redrawn
- net class Default: clearance 0.2 -> 0.127; trace_width 0.25 -> 0.127; via_dia 0.8 -> 0.5; via_drill 0.4 -> 0.2
- rule trace_clearance: 0.2 -> 0.127
- rule trace_min: 0.2 -> 0.12
- rule via_min_drill: 0.3 -> 0.2
- rule via_min_size: 0.4 -> 0.5

Commit message: PCB design
Parts:
- H101, H102: footprint MountingHole:MountingHole_2.7mm_M2.5_DIN965_Pad -> MountingHole:MountingHole_3.2mm_M3_DIN965_Pad
- moved C503 25.4 mm to (181.4, 58.3), turned to 90 degrees
- moved C504 13.3 mm to (183.5, 58.3)
- moved C505 13.0 mm to (202.7, 58.3)
- moved C507 6.86 mm to (191.8, 58.4)
- moved R201 2.84 mm to (186.1, 55.8), turned to 0 degrees
- moved R202 2.62 mm to (189.5, 55.8), turned to 180 degrees
- moved C502 2.03 mm to (190.6, 74.4)
- moved C501 1.02 mm to (192.2, 74.4)
- moved C211 0.89 mm to (179.2, 83.8)
- moved C213 0.89 mm to (179.2, 87.5)
- moved C215 0.89 mm to (179.2, 80.1)
- moved C221 0.89 mm to (181.5, 83.8)
- moved C223 0.89 mm to (181.5, 80.1)
- moved C225 0.89 mm to (181.5, 87.5)
- moved U202 0.89 mm to (180.3, 80.1)
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Routing:
- net /MCU/A2: track 0.00 -> 28.2 mm, vias 0 -> 1
- net /MCU/A3: track 0.00 -> 27.0 mm, vias 0 -> 1
- net /MCU/D15: track 0.00 -> 26.5 mm, vias 0 -> 1
- net /MCU/A0: track 0.00 -> 26.3 mm, vias 0 -> 1
- net /MCU/A1: track 0.00 -> 26.2 mm, vias 0 -> 1
- net /MCU/CLK: track 0.53 -> 26.6 mm
- net /MCU/D14: track 0.52 -> 26.4 mm
- net /MCU/D13: track 0.54 -> 26.2 mm
- net /MCU/D12: track 0.00 -> 25.6 mm, vias 0 -> 1
- net /MCU/D11: track 0.00 -> 24.8 mm, vias 0 -> 1
- net /MCU/D10: track 0.00 -> 23.8 mm, vias 0 -> 1
- net /MCU/TCK_SWCLK: track 28.9 -> 5.48 mm
- net /MCU/D9: track 0.00 -> 22.9 mm, vias 0 -> 1
- net /MCU/CKE: track 0.53 -> 23.2 mm
- net /MCU/~CS: track 0.00 -> 22.7 mm, vias 0 -> 1
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- removed copper zone on POWER_A, net VCCQ
Other:
- outline, holes or cut-outs redrawn

Commit message: PCB layout
Parts:
- moved C506 17.4 mm to (189.2, 58.4), turned to 90 degrees
- moved C901 1.40 mm to (209.0, 140.3)
- moved C902 1.40 mm to (202.7, 140.3)
- moved R701 1.40 mm to (191.4, 142.2)
- moved U901 1.40 mm to (205.9, 141.1)
- moved C702 1.40 mm to (194.2, 139.3)
- moved C703 1.40 mm to (194.2, 142.1)
- moved U701 1.40 mm to (194.1, 141.2)
- moved C803 1.15 mm to (210.4, 123.4)
- moved C804 1.15 mm to (208.7, 123.4)
- moved C807 1.15 mm to (204.1, 132.3)
- moved C808 1.15 mm to (191.6, 125.2)
- moved C809 1.15 mm to (191.6, 131.1)
- moved C810 1.15 mm to (193.4, 131.1)
- moved C811 1.15 mm to (187.1, 125.2)
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Connections:
- U205 pad 1: (no net) -> /MCU/MCU_SR_DAT
- U205 pad 2: (no net) -> /MCU/MCU_SR_LAT
- U205 pad 3: (no net) -> /MCU/MCU_SR_CLK
- U205 pad 40: (no net) -> /MCU/TRIG_EN
- U205 pad 41: (no net) -> /MCU/TRIG_OUT
- U205 pad 42: (no net) -> /MCU/TRIG_IN
- U205 pad 69: /MCU/TRIG_IN -> (no net)
- U205 pad 7: Net-(R203-Pad1) -> (no net)
- U205 pad 70: /MCU/TRIG_OUT -> (no net)
- U205 pad 73: /MCU/TRIG_EN -> Net-(R203-Pad1)
- U205 pad 8: Net-(R204-Pad1) -> (no net)
- U205 pad 87: (no net) -> Net-(R204-Pad1)
- U205 pad 9: Net-(R205-Pad1) -> (no net)
- U205 pad 91: (no net) -> Net-(R205-Pad1)
- U205 pad 96: /MCU/MCU_SR_DAT -> (no net)
- U205 pad 97: /MCU/MCU_SR_CLK -> (no net)
- U205 pad 98: /MCU/MCU_SR_LAT -> (no net)
Routing:
- net VREF: track 3.05 -> 111.7 mm, vias 0 -> 4
- net /Channel 1/DAC_V1: track 0.00 -> 93.5 mm, vias 0 -> 2
- net GND: track 9.78 -> 98.6 mm, vias 6 -> 46
- net +9V: track 0.00 -> 80.6 mm, vias 0 -> 8
- net +5V: track 28.7 -> 101.0 mm, vias 11 -> 21
- net /Channel 2/DAC_V2: track 0.00 -> 60.0 mm, vias 0 -> 2
- net +5VF: track 0.00 -> 58.8 mm, vias 0 -> 11
- net +3V3: track 75.7 -> 125.4 mm, vias 32 -> 43
- net -18V: track 11.2 -> 58.5 mm, vias 5 -> 16
- net +18V: track 9.75 -> 51.3 mm, vias 5 -> 16
- net /Channel 3/DAC_V3: track 0.00 -> 40.6 mm, vias 0 -> 2
- net /DAC/+2V5REF: track 0.00 -> 35.1 mm, vias 0 -> 1
- net Net-(U1503-Pad6): track 0.00 -> 34.1 mm, vias 0 -> 1
- net Net-(U1403-Pad6): track 0.00 -> 34.1 mm, vias 0 -> 1
- net /Connector 1/RX-: track 0.00 -> 33.5 mm
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- added copper zone on B.Cu, net /CH1 Connector/CH1_IN
- added copper zone on B.Cu, net /CH2 Connector/CH2_IN
- added copper zone on B.Cu, net /CH3 Connector/CH3_IN
- added copper zone on B.Cu, net Earth
- added copper zone on GND, net Earth
- added copper zone on B.Cu, net Net-(C614-Pad1)
- added copper zone on POWER_B, net VCCQ
- removed copper zone on POWER_A, net (none)
Other:
- outline, holes or cut-outs redrawn

Commit message: PCB layout
Parts:
- added C228: 100n, Capacitor_SMD:C_0603_1608Metric_Pad1.08x0.95mm_HandSolder, B.Cu at (207.4, 61.0)
- added R1506: 0, Resistor_SMD:R_0603_1608Metric_Pad0.98x0.95mm_HandSolder, F.Cu at (160.6, 53.2)
- added R203: 4k7, Resistor_SMD:R_0603_1608Metric_Pad0.98x0.95mm_HandSolder, B.Cu at (153.3, 53.2)
- added R204: 4k7, Resistor_SMD:R_0603_1608Metric_Pad0.98x0.95mm_HandSolder, B.Cu at (156.8, 53.2)
- added R806: 0, Resistor_SMD:R_0603_1608Metric_Pad0.98x0.95mm_HandSolder, F.Cu at (159.5, 119.4)
- added R906: 0, Resistor_SMD:R_0603_1608Metric_Pad0.98x0.95mm_HandSolder, F.Cu at (159.5, 86.2)
- added U205: PCA9517, Package_SO:TSSOP-8_3x3mm_P0.65mm, F.Cu at (207.3, 60.7)
- moved C223 1.27 mm to (209.8, 60.8)
- moved U206 1.27 mm to (211.2, 60.8)
- moved C209 0.92 mm to (204.6, 59.6)
- moved C206 0.65 mm to (204.6, 66.8)
- moved C205 0.63 mm to (204.6, 63.4)
- moved R205 0.38 mm to (212.3, 59.7)
- moved R206 0.38 mm to (212.3, 62.1)
- renumbered C814 to C1301, C815 to C1302, C801 to C1303, C802 to C1304, C803 to C1305, C804 to C1306, C805 to C1307, C806 to C1308, C807 to C1309, C808 to C1310, C809 to C1311, C810 to C1312, C811 to C1313, C812 to C1314, C813 to C1315, C501 to C1401, C502 to C1402, C503 to C1403, C504 to C1404, C505 to C1405, C506 to C1406, C507 to C1407, C301 to C1501, C302 to C1502, C303 to C1503, C304 to C1504, C305 to C1505, C306 to C1506, C307 to C1507, C308 to C1508, C309 to C1509, C310 to C1510, C311 to C1511, C312 to C1512, C313 to C1513, C314 to C1514, C315 to C1515, C316 to C1516, C317 to C1517, C318 to C1518, C319 to C1519, C320 to C1520, C321 to C1521, C322 to C1522, C323 to C1523, C324 to C1524, C325 to C1525, C206 to C204, C207 to C205, C212 to C206, C214 to C207, C216 to C208, C218 to C209, C220 to C210, C222 to C211, C224 to C212, C226 to C213, C227 to C214, C204 to C215, C205 to C216, C211 to C217, C213 to C218, C208 to C219, C209 to C220, C215 to C221, C210 to C222, C217 to C223, C219 to C224, C221 to C225, C223 to C226, C225 to C227, C228 to C229, C401 to C301, C402 to C302, C403 to C303, C404 to C304, C405 to C305, C406 to C306, C407 to C307, C408 to C308, C409 to C309, C601 to C401, C602 to C402, C603 to C403, C604 to C404, C605 to C405, C606 to C406, C607 to C407, C608 to C408, C609 to C409, C610 to C410, C611 to C411, C612 to C412, C613 to C413, C614 to C414, C701 to C501, C702 to C502, C703 to C503, C901 to C601, C902 to C602, C1501 to C801, C1502 to C802, C1503 to C803, C1504 to C804, C1505 to C805, C1506 to C806, C1507 to C807, C1508 to C808, C1509 to C809, C1510 to C810, C1511 to C811, C1512 to C812, C1513 to C813, C1514 to C814, C1515 to C815, C1516 to C816, C1517 to C817, C1518 to C818, C1519 to C819, C1520 to C820, C1521 to C821, C1522 to C822, C1523 to C823, C1524 to C824, C1525 to C825, C1401 to C901, C1402 to C902, C1403 to C903, C1404 to C904, C1405 to C905, C1406 to C906, C1407 to C907, C1408 to C908, C1409 to C909, C1410 to C910, C1411 to C911, C1412 to C912, C1413 to C913, C1414 to C914, C1415 to C915, C1416 to C916, C1417 to C917, C1418 to C918, C1419 to C919, C1420 to C920, C1421 to C921, C1422 to C922, C1423 to C923, C1424 to C924, C1425 to C925, D401 to D301, D402 to D302, D403 to D303, D601 to D401, D602 to D402, FB801 to FB1301, FB802 to FB1302, FB601 to FB401, J1301 to J1001, J1201 to J1101, J1101 to J1201, J1001 to J701, J1002 to J702, L401 to L301, L601 to L401, R801 to R1301, R802 to R1302, R803 to R1303, R804 to R1304, R805 to R1305, R806 to R1306, R807 to R1307, R808 to R1308, R809 to R1309, R810 to R1310, R811 to R1311, R812 to R1312, R813 to R1313, R301 to R1501, R302 to R1502, R303 to R1503, R304 to R1504, R305 to R1505, R306 to R1507, R307 to R1508, R308 to R1509, R309 to R1510, R310 to R1511, R311 to R1512, R312 to R1513, R313 to R1514, R314 to R1515, R315 to R1516, R316 to R1517, R206 to R205, R207 to R206, R208 to R207, R203 to R208, R204 to R209, R205 to R210, R209 to R211, R210 to R212, R401 to R301, R402 to R302, R403 to R303, R404 to R304, R405 to R305, R406 to R306, R601 to R401, R602 to R402, R603 to R403, R604 to R404, R605 to R405, R606 to R406, R607 to R407, R608 to R408, R609 to R409, R610 to R410, R611 to R411, R612 to R412, R613 to R413, R614 to R414, R615 to R415, R616 to R416, R617 to R417, R618 to R418, R619 to R419, R620 to R420, R621 to R421, R701 to R501, R1501 to R801, R1502 to R802, R1503 to R803, R1504 to R804, R1505 to R805, R1506 to R807, R1507 to R808, R1508 to R809, R1509 to R810, R1510 to R811, R1511 to R812, R1512 to R813, R1513 to R814, R1514 to R815, R1515 to R816, R1516 to R817, R1401 to R901, R1402 to R902, R1403 to R903, R1404 to R904, R1405 to R905, R1406 to R907, R1407 to R908, R1408 to R909, R1409 to R910, R1410 to R911, R1411 to R912, R1412 to R913, R1413 to R914, R1414 to R915, R1415 to R916, R1416 to R917, U801 to U1301, U802 to U1302, U803 to U1303, U501 to U1401, U301 to U1501, U302 to U1502, U303 to U1503, U304 to U1504, U305 to U1505, U306 to U1506, U307 to U1507, U308 to U1508, U202 to U201, U203 to U202, U204 to U203, U201 to U204, U205 to U207, U401 to U301, U402 to U302, U403 to U303, U601 to U401, U602 to U402, U603 to U403, U701 to U501, U901 to U601, U1501 to U801, U1502 to U802, U1503 to U803, U1504 to U804, U1505 to U805, U1506 to U806, U1507 to U807, U1508 to U808, U1401 to U901, U1402 to U902, U1403 to U903, U1404 to U904, U1405 to U905, U1406 to U906, U1407 to U907, U1408 to U908, Y601 to Y401
Connections:
- J1001 pad 2: (no net) -> /CH1 Connector/I2C_SCL
- J1001 pad 4: (no net) -> /CH1 Connector/I2C_SDA
- J1101 pad 2: (no net) -> /CH1 Connector/I2C_SCL
- J1101 pad 4: (no net) -> /CH1 Connector/I2C_SDA
- J1201 pad 2: (no net) -> /CH1 Connector/I2C_SCL
- J1201 pad 4: (no net) -> /CH1 Connector/I2C_SDA
- U1302 pad 10: (no net) -> /DAC/DAC_SCLK
- U1302 pad 11: (no net) -> /DAC/DAC_DIN
- U1302 pad 16: (no net) -> /DAC/DAC_LDAC
- U1302 pad 9: (no net) -> /DAC/DAC_~SYNC
- U207 pad 18: (no net) -> /DAC/DAC_~SYNC
- U207 pad 19: (no net) -> /DAC/DAC_SCLK
- U207 pad 21: (no net) -> /DAC/DAC_DIN
- U207 pad 22: (no net) -> /DAC/DAC_LDAC
Routing:
- net (no net): track 0.00 -> 184.4 mm
- net /CH1 Connector/I2C_SDA: track 0.00 -> 132.2 mm, vias 0 -> 1
- net /CH1 Connector/I2C_SCL: track 0.00 -> 130.1 mm, vias 0 -> 1
- net /MCU/SD_LAT: track 0.00 -> 114.9 mm, vias 0 -> 3
- net /MCU/SD_CLK: track 0.00 -> 106.8 mm
- net /Channel 1/ADC1_SCLK: track 0.00 -> 104.0 mm, vias 0 -> 4
- net /Channel 1/ADC1_~CS: track 0.00 -> 100.8 mm, vias 0 -> 4
- net /Channel 3/ADC3_SDO: track 2.15 -> 96.8 mm, vias 1 -> 2
- net /DAC/DAC_~SYNC: track 0.00 -> 93.7 mm, vias 0 -> 2
- net /DAC/DAC_SCLK: track 0.00 -> 92.7 mm, vias 0 -> 2
- net /DAC/DAC_DIN: track 0.00 -> 89.0 mm, vias 0 -> 2
- net /DAC/DAC_LDAC: track 0.00 -> 86.1 mm, vias 0 -> 2
- net /Channel 2/SR2_QH: track 0.00 -> 58.5 mm
- net /Channel 1/SR1_QH: track 0.00 -> 51.5 mm, vias 0 -> 2
- net /Channel 1/ADC1_SDO: track 2.15 -> 46.8 mm, vias 1 -> 2
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- added copper zone on INT3, net +18V
- added copper zone on INT2, net +3V3
- added copper zone on INT2, net +5V
- added copper zone on INT2, net +5VF
- added copper zone on INT1, net +5V_TRIG
- added copper zone on INT2, net +5V_TRIG
- added copper zone on INT3, net +5V_TRIG
- added copper zone on INT2, net +9V
- added copper zone on INT1, net -18V
- added copper zone on INT0, net Earth
- added copper zone on INT1, net Earth
- added copper zone on INT2, net Earth
- added copper zone on INT3, net Earth
- added copper zone on INT0, net GND
- added copper zone on INT1, net GND
- added copper zone on INT3, net GND
- added copper zone on INT0, net GND_TRIG
- added copper zone on INT2, net VCCQ
- removed copper zone on POWER_A, net +18V
- removed copper zone on POWER_B, net +3V3
- removed copper zone on POWER_B, net +5V
- removed copper zone on POWER_A, net +5V_TRIG
- removed copper zone on POWER_B, net +9V
- removed copper zone on POWER_A, net -18V
- removed copper zone on GND, net Earth
- removed copper zone on GND, net GND
- removed copper zone on GND, net GND_TRIG
- removed copper zone on POWER_B, net VCCQ
Other:
- board text added: "1"
- board text added: "2"
- board text added: "3"
- board text added: "4"
- board text added: "5"
- board text added: "6"
