File: hardware/project/ETH3CDAQ1_MEASURE/Channel1.sch (KiCad schematic (older format))
At the start: 63 parts, among them U301 LT1355, U302 DG211, U303 DG419LDY, U304 OPA140, U305 DG419LDY, U306 AD8251, U307 SN74LVC1G14DBVR, U308 SN74LVC1G14DBVR, U309 SN74LVC1G14DBVR, U310 ADAQ798x, U311 74HCT595

Commit message: Meas. module schematic design.
Parts:
- removed D301: MMBZ15VDL, Package_TO_SOT_SMD:SOT-23, symbol Diode:MMBZxx
- removed D302: BAT54SW, Package_TO_SOT_SMD:SOT-323_SC-70, symbol Diode:BAT54SW
- removed R302, R315: DNP, Resistor_SMD:R_0603_1608Metric_Pad0.98x0.95mm_HandSolder, symbol Device:R
- removed R303: OPT, Resistor_SMD:R_0603_1608Metric_Pad0.98x0.95mm_HandSolder, symbol Device:R
- removed R307: 10k, Resistor_SMD:R_0603_1608Metric_Pad0.98x0.95mm_HandSolder, symbol Device:R
- removed R316, R317, R318, R319, R320, R321, R322: 620, Resistor_SMD:R_0603_1608Metric_Pad0.98x0.95mm_HandSolder, symbol Device:R
- removed RN301, RN302: 1k, Resistor_SMD:R_Array_Concave_4x0603, symbol Device:R_Pack04_Split
- removed U304: OPA140, Package_SO:SOIC-8_3.9x4.9mm_P1.27mm, symbol ETH3CDAQ1:OPA140
- removed U306: AD8251, Package_SO:MSOP-10_3x3mm_P0.5mm, symbol ETH3CDAQ1:AD8251
- removed U307, U308, U309: SN74LVC1G14DBVR, Package_TO_SOT_SMD:SOT-23-5, symbol 74xGxx:SN74LVC1G14DBV
- removed U310: ADAQ798x, ETH3CDAQ1:LGA-24_5x4mm_P0.5mm, symbol ETH3CDAQ1:ADAQ798x
- removed U311: 74HCT595, Package_SO:TSSOP-16_4.4x5mm_P0.65mm, symbol 74xx:74HCT595
- added C327: 1u, symbol Device:C
- added D302: D_TVS, symbol Device:D_TVS
- added R307: 680, symbol Device:R_Pack04_Split
- added U304: 74LVC1GU04DRL, Package_TO_SOT_SMD:SOT-553, symbol 74xGxx:74LVC1GU04DRL
- added U306: ADS8681RUM, Package_DFN_QFN:QFN-16-1EP_4x4mm_P0.65mm_EP2.7x2.7mm, symbol Analog_ADC:ADS8681RUM
- added U307: 74HCT595, symbol 74xx:74HCT595
- C325: value C -> 330p; footprint Capacitor_SMD:C_0603_1608Metric_Pad1.08x0.95mm_HandSolder -> (none)
- C326: value C -> 22u; footprint Capacitor_SMD:C_0603_1608Metric_Pad1.08x0.95mm_HandSolder -> (none)
- R301: value 0 -> 49R9; footprint Resistor_SMD:R_0603_1608Metric_Pad0.98x0.95mm_HandSolder -> (none)
Connections:
- net labels added: +18V, +5VF, -18V, CH1_LPF, CH1_M_DAC, DAC_VOUT1, REFCAP1
- net labels removed: +10V, +5VP, +7.5V, -10V, CH1_A0, CH1_A1, CH1_CNV, CH1_M_LPF, CH1_M_N10V, CH1_M_P10V, CH1_SCK, CH1_SDI, CH1_SDO, LPF, REF_OUT, SR_CLK, SR_DAT, SR_LAT, SR_QH1
- wire segments 305 -> 226
Other:
- moved on the sheet: C311, C316, C321, C324, R304, R305, R306, R308, R309, R310, R311, R312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

Commit message: Measurement module development.
Parts:
- removed C301, C302, C308, C319: 100n, Capacitor_SMD:C_0603_1608Metric_Pad1.08x0.95mm_HandSolder, symbol Device:C
- removed D302: D_TVS, symbol Device:D_TVS
- added C321, C324: 100n, Capacitor_SMD:C_0603_1608Metric_Pad1.08x0.95mm_HandSolder, symbol Device:C
- added R305: 0R22, Resistor_SMD:R_0603_1608Metric_Pad0.98x0.95mm_HandSolder, symbol Device:R
- added R306: 0R47, Resistor_SMD:R_0603_1608Metric_Pad0.98x0.95mm_HandSolder, symbol Device:R
- added R315, R316: 10k, Resistor_SMD:R_0603_1608Metric_Pad0.98x0.95mm_HandSolder, symbol Device:R
- added U305: OPA192, Package_SO:SOIC-8_3.9x4.9mm_P1.27mm, symbol ETH3CDAQ1:OPA192
- C301: renamed from C326; footprint (none) -> Capacitor_SMD:C_0805_2012Metric_Pad1.18x1.45mm_HandSolder
- C302: renamed from C327; footprint (none) -> Capacitor_SMD:C_0603_1608Metric_Pad1.08x0.95mm_HandSolder
- C303: value 100n -> 10u; footprint Capacitor_SMD:C_0603_1608Metric_Pad1.08x0.95mm_HandSolder -> Capacitor_SMD:C_0805_2012Metric_Pad1.18x1.45mm_HandSolder
- C323: value 2u2 -> 100n
- C325: footprint (none) -> Capacitor_SMD:C_0603_1608Metric_Pad1.08x0.95mm_HandSolder
- R304: renamed from R301; footprint (none) -> Resistor_SMD:R_0603_1608Metric_Pad0.98x0.95mm_HandSolder
- R314: renamed from R307; footprint (none) -> Resistor_SMD:R_Array_Convex_4x0603
- U308: renamed from U307; footprint (none) -> Package_SO:TSSOP-16_4.4x5mm_P0.65mm
- renumbered C311 to C308, C316 to C311, C321 to C316, C324 to C319, R304 to R301, R305 to R302, R306 to R303, R308 to R307, R309 to R308, R310 to R309, R311 to R310, R312 to R311, R313 to R312, R314 to R313, U305 to U304, U304 to U306, U306 to U307
Connections:
- net labels added: ADC1_SCLK, ADC1_SDI, ADC1_SDO, ADC1_~CS, DAC_V1, SR1_CLK, SR1_DAT, SR1_LAT, SR1_QH
- net labels removed: +15V, -15V, -2V5, DAC_VOUT1
- wire segments 226 -> 244
- no-connect marks 5 -> 7
Other:
- moved on the sheet: C301, C302, C308, C311, C316, C319, C325, R301, R302, R303, R304, R307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

Commit message: PCB layout
Connections:
- net +5VF is gone; now on net +5V: U307.16 (AVDD)
Changed lines of the file:
@@
-$EndComp
-$Comp
-L power:+5V #PWR0342
-U 1 1 5FCE598A
-P 12700 6050
-F 0 "#PWR0342" H 12700 5900 50  0001 C CNN
-F 1 "+5V" H 12715 6223 50  0000 C CNN
-F 2 "" H 12700 6050 50  0001 C CNN
-F 3 "" H 12700 6050 50  0001 C CNN
-	1    12700 6050
-	1    0    0    -1
 $EndComp
 $Comp
@@
 $EndComp
 $Comp
-L power:+5V #PWR0334
-U 1 1 5FDF399F
-P 10300 5900
-F 0 "#PWR0334" H 10300 5750 50  0001 C CNN
-F 1 "+5V" H 10315 6073 50  0000 C CNN
-F 2 "" H 10300 5900 50  0001 C CNN
-F 3 "" H 10300 5900 50  0001 C CNN
-	1    10300 5900
-	1    0    0    -1
-$EndComp
-$Comp
 L power:GND #PWR0335
 U 1 1 5FDF3FBD
@@
 Wire Wire Line
 	4300 10800 4550 10800
-$Comp
-L ETH3CDAQ1:+5VF #PWR0338
-U 1 1 5FFE8ABB
-P 11950 4300
-F 0 "#PWR0338" H 11950 4150 50  0001 C CNN
-F 1 "+5VF" H 11965 4473 50  0000 C CNN
-F 2 "" H 11950 4300 50  0001 C CNN
-F 3 "" H 11950 4300 50  0001 C CNN
-	1    11950 4300
-	1    0    0    -1
-$EndComp
 Wire Wire Line
 	11600 4850 11050 4850
@@
 	6950 9400 6750 9400
 $Comp
-L power:+5V #PWR0326
-U 1 1 5FE9D424
-P 6950 9350
-F 0 "#PWR0326" H 6950 9200 50  0001 C CNN
-F 1 "+5V" H 6965 9523 50  0000 C CNN
-F 2 "" H 6950 9350 50  0001 C CNN
-F 3 "" H 6950 9350 50  0001 C CNN
-	1    6950 9350
-	1    0    0    -1
-$EndComp
-$Comp
 L Device:C C320
 U 1 1 5FEAAE9E
@@
 Wire Wire Line
 	10650 4850 11050 4850
+$Comp
+L power:+5V #PWR?
+U 1 1 5FCDFC33
+P 11950 4300
+F 0 "#PWR?" H 11950 4150 50  0001 C CNN
+F 1 "+5V" H 11965 4473 50  0000 C CNN
+F 2 "" H 11950 4300 50  0001 C CNN
+F 3 "" H 11950 4300 50  0001 C CNN
+	1    11950 4300
+	1    0    0    -1
+$EndComp
+$Comp
+L power:+5V #PWR?
+U 1 1 5FCE044F
+P 10300 5900
+F 0 "#PWR?" H 10300 5750 50  0001 C CNN
+F 1 "+5V" H 10315 6073 50  0000 C CNN
+F 2 "" H 10300 5900 50  0001 C CNN
+F 3 "" H 10300 5900 50  0001 C CNN
+	1    10300 5900
+	1    0    0    -1
+$EndComp
+$Comp
+L power:+5V #PWR?
+U 1 1 5FCE1801
+P 12700 6050
+F 0 "#PWR?" H 12700 5900 50  0001 C CNN
+F 1 "+5V" H 12715 6223 50  0000 C CNN
+F 2 "" H 12700 6050 50  0001 C CNN
+F 3 "" H 12700 6050 50  0001 C CNN
+	1    12700 6050
+	1    0    0    -1
+$EndComp
+$Comp
+L power:+5V #PWR?
+U 1 1 5FCE29BD
+P 6950 9350
+F 0 "#PWR?" H 6950 9200 50  0001 C CNN
+F 1 "+5V" H 6965 9523 50  0000 C CNN
+F 2 "" H 6950 9350 50  0001 C CNN
+F 3 "" H 6950 9350 50  0001 C CNN
+	1    6950 9350
+	1    0    0    -1
+$EndComp
 $EndSCHEMATC

Commit message: PCB layout
Parts:
- added R1506: 0, Resistor_SMD:R_0603_1608Metric_Pad0.98x0.95mm_HandSolder, symbol Device:R
- renumbered C301 to C1501, C302 to C1502, C303 to C1503, C304 to C1504, C305 to C1505, C306 to C1506, C307 to C1507, C308 to C1508, C309 to C1509, C310 to C1510, C311 to C1511, C312 to C1512, C313 to C1513, C314 to C1514, C315 to C1515, C316 to C1516, C317 to C1517, C318 to C1518, C319 to C1519, C320 to C1520, C321 to C1521, C322 to C1522, C323 to C1523, C324 to C1524, C325 to C1525, R301 to R1501, R302 to R1502, R303 to R1503, R304 to R1504, R305 to R1505, R306 to R1507, R307 to R1508, R308 to R1509, R309 to R1510, R310 to R1511, R311 to R1512, R312 to R1513, R313 to R1514, R314 to R1515, R315 to R1516, R316 to R1517, U301 to U1501, U302 to U1502, U303 to U1503, U304 to U1504, U305 to U1505, U306 to U1506, U307 to U1507, U308 to U1508
Connections:
- net at U1503.1, U1505.2 (-), U1505.6: now also R1506.1
- net at U1502.10, U1502.15, U1502.3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: now also R1506.2
