File: hardware/project/ETH3CDAQ1_MEASURE/Connector1.sch (KiCad schematic (older format))
At the start: 2 parts, among them J1001 Conn_02x02_Odd_Even, J1002 Conn_02x04_Odd_Even

Commit message: PCB layout
Parts:
- renumbered J1001 to J701, J1002 to J702
Changed lines of the file:
@@
 $EndDescr
 $Comp
-L Connector_Generic:Conn_02x02_Odd_Even J1001
+L Connector_Generic:Conn_02x02_Odd_Even J701
 U 1 1 5FC8AAE4
 P 5200 3350
-F 0 "J1001" H 5250 3567 50  0000 C CNN
+F 0 "J701" H 5250 3567 50  0000 C CNN
 F 1 "Conn_02x02_Odd_Even" H 5250 3476 50  0000 C CNN
 F 2 "Connector_PinSocket_2.54mm:PinSocket_2x02_P2.54mm_Vertical" H 5200 3350 50  0001 C CNN
@@
 $EndComp
 $Comp
-L Connector_Generic:Conn_02x04_Odd_Even J1002
+L Connector_Generic:Conn_02x04_Odd_Even J702
 U 1 1 5FC8B9F5
 P 6650 3450
-F 0 "J1002" H 6700 3767 50  0000 C CNN
+F 0 "J702" H 6700 3767 50  0000 C CNN
 F 1 "Conn_02x04_Odd_Even" H 6700 3676 50  0000 C CNN
 F 2 "Connector_PinSocket_2.54mm:PinSocket_2x04_P2.54mm_Vertical" H 6650 3450 50  0001 C CNN
@@
 $EndComp
 $Comp
-L power:Earth #PWR01003
+L power:Earth #PWR0703
 U 1 1 5FB875C1
 P 6450 3350
-F 0 "#PWR01003" H 6450 3100 50  0001 C CNN
+F 0 "#PWR0703" H 6450 3100 50  0001 C CNN
 F 1 "Earth" H 6450 3200 50  0001 C CNN
 F 2 "" H 6450 3350 50  0001 C CNN
@@
 $EndComp
 $Comp
-L power:Earth #PWR01004
+L power:Earth #PWR0704
 U 1 1 5FB87E11
 P 6450 3650
-F 0 "#PWR01004" H 6450 3400 50  0001 C CNN
+F 0 "#PWR0704" H 6450 3400 50  0001 C CNN
 F 1 "Earth" H 6450 3500 50  0001 C CNN
 F 2 "" H 6450 3650 50  0001 C CNN
@@
 $EndComp
 $Comp
-L power:Earth #PWR01006
+L power:Earth #PWR0706
 U 1 1 5FB880DB
 P 6950 3650
-F 0 "#PWR01006" H 6950 3400 50  0001 C CNN
+F 0 "#PWR0706" H 6950 3400 50  0001 C CNN
 F 1 "Earth" H 6950 3500 50  0001 C CNN
 F 2 "" H 6950 3650 50  0001 C CNN
@@
 $EndComp
 $Comp
-L power:Earth #PWR01005
+L power:Earth #PWR0705
 U 1 1 5FB8868B
 P 6950 3350
-F 0 "#PWR01005" H 6950 3100 50  0001 C CNN
+F 0 "#PWR0705" H 6950 3100 50  0001 C CNN
 F 1 "Earth" H 6950 3200 50  0001 C CNN
 F 2 "" H 6950 3350 50  0001 C CNN
@@
 	5000 3350 4950 3350
 $Comp
-L ETH3CDAQ1:GND_TRIG #PWR01001
+L ETH3CDAQ1:GND_TRIG #PWR0701
 U 1 1 5FB990E0
 P 4950 3450
-F 0 "#PWR01001" H 4950 3200 50  0001 C CNN
+F 0 "#PWR0701" H 4950 3200 50  0001 C CNN
 F 1 "GND_TRIG" V 4955 3322 50  0000 R CNN
 F 2 "" H 4950 3450 50  0001 C CNN
@@
 $EndComp
 $Comp
-L ETH3CDAQ1:GND_TRIG #PWR01002
+L ETH3CDAQ1:GND_TRIG #PWR0702
 U 1 1 5FB992B6
 P 5550 3450
-F 0 "#PWR01002" H 5550 3200 50  0001 C CNN
+F 0 "#PWR0702" H 5550 3200 50  0001 C CNN
 F 1 "GND_TRIG" V 5555 3322 50  0000 R CNN
 F 2 "" H 5550 3450 50  0001 C CNN
