File: hardware/project/ETH3CDAQ1_MEASURE/Trigger.sch (KiCad schematic (older format))
At the start: 22 parts, among them U401 TXB0104PW, U402 ADuM5402, U403 74AC125

Commit message: PCB layout
Parts:
- renumbered C401 to C301, C402 to C302, C403 to C303, C404 to C304, C405 to C305, C406 to C306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
