File: hardware/project/ETH3CDAQ1_MEASURE/MCU.sch (KiCad schematic (older format))
At the start: 51 parts, among them J201 20021111-00010T4LF, J202 Conn_02x01, U201 HDC1080, U202 SN74LVC1T45DBV, U203 SN74LVC1T45DBV, U204 SN74LVC1T45DBV, U205 STM32H743ZI, U206 24LC08B-E/MS, Y201 NX3225GD-8MHZ

Commit message: Measurement module development.
Connections:
- net MCU_MOSI: now reaches U205.113 (PC12,TRACED3,SPI3_MOSI,I2S3_SD,USART3_CK,UART5_TX,SDMMC1_CK,DCMI_D9,EVENTOUT)
- net MCU_CNV renamed MCU_~CS
- net MCU_~CS1: no longer names the net of U205.116 (PD2,TRACED2,TIM3_ETR,UART5_RX,SDMMC1_CMD,DCMI_D11,EVENTOUT)
- net MCU_~CS2: no longer names the net of U205.117 (PD3,DFSDM1_CKOUT,SPI2_SCK,I2S2_CK,DFSDM1_DATIN0,USART2_CTS,FMC_CLK,DCMI_D5,LCD_G7,EVENTOUT)
- net MCU_~CS3: no longer names the net of U205.118 (PD4,DFSDM1_CKIN0,USART2_RTS,FMC_NOE,EVENTOUT)
- no-connect marks 46 -> 48
Changed lines of the file:
@@
 $Descr A3 16535 11693
 encoding utf-8
-Sheet 2 10
+Sheet 2 15
 Title "MCU"
 Date "2020-03-07"
@@
 Text HLabel 3350 6050 0    50   Input ~ 0
 MCU_MISO
-NoConn ~ 3400 6150
 Text HLabel 3350 4750 0    50   Output ~ 0
-MCU_CNV
+MCU_~CS
 Wire Wire Line
 	3350 4750 3400 4750
-Text HLabel 14850 3150 2    50   Output ~ 0
-MCU_~CS1
-Text HLabel 14850 3250 2    50   Output ~ 0
-MCU_~CS2
-Text HLabel 14850 3350 2    50   Output ~ 0
-MCU_~CS3
-Wire Wire Line
-	14800 3150 14850 3150
-Wire Wire Line
-	14850 3250 14800 3250
-Wire Wire Line
-	14800 3350 14850 3350
+Text HLabel 3350 6150 0    50   Output ~ 0
+MCU_MOSI
+Wire Wire Line
+	3350 6150 3400 6150
+NoConn ~ 14800 3150
+NoConn ~ 14800 3250
+NoConn ~ 14800 3350
 Wire Bus Line
 	1400 3500 1400 4800

Commit message: PCB layout
Connections:
- net MCU_SR_CLK: now also U205.3 (PE4,TRACED1,SPI4_NSS,SAI1_FS_A,DFSDM1_DATIN3,FMC_A20,DCMI_D4,LCD_B0,EVENTOUT); no longer U205.97 (PC7,TIM3_CH2,TIM8_CH2,I2S3_MCK,DFSDM1_DATIN3,USART6_RX,FMC_NE1,SDMMC2_D7,SDMMC1_D7,DCMI_D1,LCD_G6,EVENTOUT)
- net MCU_SR_DAT: now also U205.1 (PE2,TRACECLK,SPI4_SCK,SAI1_MCLK_A,QUADSPI_BK1_IO2,ETH_MII_TXD3,FMC_A23,EVENTOUT); no longer U205.96 (PC6,TIM3_CH1,TIM8_CH1,I2S2_MCK,DFSDM1_CKIN3,USART6_TX,FMC_NWAIT,SDMMC2_D6,SDMMC1_D6,DCMI_D0,LCD_HSYNC,EVENTOUT)
- net MCU_SR_LAT: now also U205.2 (PE3,TRACED0,SAI1_SD_B,FMC_A19,EVENTOUT); no longer U205.98 (PC8,TRACED1,TIM3_CH3,TIM8_CH3,UART5_RTS,USART6_CK,FMC_NE2,FMC_NCE,SDMMC1_D0,DCMI_D2,EVENTOUT)
- net TRIG_EN: now also U205.40 (PA4,SPI1_NSS,I2S1_WS,SPI3_NSS,I2S3_WS,USART2_CK,SPI6_NSS,OTG_HS_SOF,DCMI_HSYNC,LCD_VSYNC,EVENTOUT,ADC1_IN4,ADC2_IN4,DAC_OUT1); no longer U205.73 (PB12,TIM1_BKIN,I2C2_SMBA,SPI2_NSS,I2S2_WS,DFSDM1_DATIN1,USART3_CK,UART5_RX,CAN2_RX,OTG_HS_ULPI_D5,ETH_MII_TXD0,ETH_RMII_TXD0,OTG_HS_ID,EVENTOUT)
- net TRIG_IN: now also U205.42 (PA6,TIM1_BKIN,TIM3_CH1,TIM8_BKIN,SPI1_MISO,SPI6_MISO,TIM13_CH1,MDIOS_MDC,DCMI_PIXCLK,LCD_G2,EVENTOUT,ADC1_IN6,ADC2_IN6); no longer U205.69 (PB10,TIM2_CH3,I2C2_SCL,SPI2_SCK,I2S2_CK,DFSDM1_DATIN7,USART3_TX,QUADSPI_BK1_NCS,OTG_HS_ULPI_D3,ETH_MII_RX_ER,LCD_G4,EVENTOUT)
- net TRIG_OUT: now also U205.41 (PA5,TIM2_CH1,TIM2_ETR,TIM8_CH1N,SPI1_SCK,I2S1_CK,SPI6_SCK,OTG_HS_ULPI_CK,LCD_R4,EVENTOUT,ADC1_IN5,ADC2_IN5,DAC_OUT2); no longer U205.70 (PB11,TIM2_CH4,I2C2_SDA,DFSDM1_CKIN7,USART3_RX,OTG_HS_ULPI_D4,ETH_MII_TX_EN,ETH_RMII_TX_EN,_DSI_TE,LCD_G5,EVENTOUT)
- net at U205.7 (PC13,EVENTOUT,RTC_TAMP2,RTC_TS,WKUP5): no longer R203.1
- net at U205.8 (PC14,EVENTOUT,OSC32_IN): no longer R204.1
- net at U205.87 (PG2,FMC_A12,EVENTOUT): now also R204.1
- net at U205.9 (PC15,EVENTOUT,OSC32_OUT): no longer R205.1
- net at U205.91 (PG6,FMC_NE3,DCMI_D12,LCD_R7,EVENTOUT): now also R205.1
- new net: R203.1, U205.73 (PB12,TIM1_BKIN,I2C2_SMBA,SPI2_NSS,I2S2_WS,DFSDM1_DATIN1,USART3_CK,UART5_RX,CAN2_RX,OTG_HS_ULPI_D5,ETH_MII_TXD0,ETH_RMII_TXD0,OTG_HS_ID,EVENTOUT)
Other:
- moved on the sheet: D201, D202, D203, R203, R204, R205
Changed lines of the file:
@@
 Text HLabel 15750 8350 2    50   BiDi ~ 0
 NRST
-Text HLabel 14850 7550 2    50   Output ~ 0
+Text HLabel 3350 3650 0    50   Output ~ 0
 TRIG_EN
-Text HLabel 14850 7450 2    50   Output ~ 0
+Text HLabel 3350 3750 0    50   Output ~ 0
 TRIG_OUT
-Text HLabel 14850 7350 2    50   Input ~ 0
+Text HLabel 3350 3850 0    50   Input ~ 0
 TRIG_IN
 Wire Wire Line
-	14850 7350 14800 7350
-Wire Wire Line
-	14850 7450 14800 7450
-Wire Wire Line
-	14800 7550 14850 7550
+	3350 3850 3400 3850
+Wire Wire Line
+	3350 3750 3400 3750
+Wire Wire Line
+	3400 3650 3350 3650
 NoConn ~ 3400 3550
-NoConn ~ 3400 3650
-NoConn ~ 3400 3850
 NoConn ~ 3400 5250
 NoConn ~ 14800 2450
@@
 L Device:R R203
 U 1 1 5E648C3B
-P 3050 6600
-F 0 "R203" V 2843 6600 50  0000 C CNN
-F 1 "680" V 2934 6600 50  0000 C CNN
-F 2 "Resistor_SMD:R_0603_1608Metric_Pad0.98x0.95mm_HandSolder" V 2980 6600 50  0001 C CNN
-F 3 "~" H 3050 6600 50  0001 C CNN
-	1    3050 6600
-	0    1    1    0
+P 15000 7550
+F 0 "R203" V 14793 7550 50  0000 C CNN
+F 1 "680" V 14884 7550 50  0000 C CNN
+F 2 "Resistor_SMD:R_0603_1608Metric_Pad0.98x0.95mm_HandSolder" V 14930 7550 50  0001 C CNN
+F 3 "~" H 15000 7550 50  0001 C CNN
+	1    15000 7550
+	0    -1   1    0
 $EndComp
 $Comp
 L Device:R R204
 U 1 1 5E64A32E
-P 3050 7000
-F 0 "R204" V 2843 7000 50  0000 C CNN
-F 1 "560" V 2934 7000 50  0000 C CNN
-F 2 "Resistor_SMD:R_0603_1608Metric_Pad0.98x0.95mm_HandSolder" V 2980 7000 50  0001 C CNN
-F 3 "~" H 3050 7000 50  0001 C CNN
-	1    3050 7000
-	0    1    1    0
+P 15200 1450
+F 0 "R204" V 14993 1450 50  0000 C CNN
+F 1 "560" V 15084 1450 50  0000 C CNN
+F 2 "Resistor_SMD:R_0603_1608Metric_Pad0.98x0.95mm_HandSolder" V 15130 1450 50  0001 C CNN
+F 3 "~" H 15200 1450 50  0001 C CNN
+	1    15200 1450
+	0    -1   1    0
 $EndComp
 $Comp
 L Device:R R205
 U 1 1 5E64A698
-P 3050 7400
-F 0 "R205" V 2843 7400 50  0000 C CNN
-F 1 "680" V 2934 7400 50  0000 C CNN
-F 2 "Resistor_SMD:R_0603_1608Metric_Pad0.98x0.95mm_HandSolder" V 2980 7400 50  0001 C CNN
-F 3 "~" H 3050 7400 50  0001 C CNN
-	1    3050 7400
-	0    1    1    0
+P 15200 1850
+F 0 "R205" V 14993 1850 50  0000 C CNN
+F 1 "680" V 15084 1850 50  0000 C CNN
+F 2 "Resistor_SMD:R_0603_1608Metric_Pad0.98x0.95mm_HandSolder" V 15130 1850 50  0001 C CNN
+F 3 "~" H 15200 1850 50  0001 C CNN
+	1    15200 1850
+	0    -1   1    0
 $EndComp
 $Comp
 L Device:LED D201
 U 1 1 5E66EF29
-P 2750 6600
-F 0 "D201" H 2743 6345 50  0000 C CNN
-F 1 "RED" H 2743 6436 50  0000 C CNN
-F 2 "LED_SMD:LED_0603_1608Metric_Pad1.05x0.95mm_HandSolder" H 2750 6600 50  0001 C CNN
-F 3 "~" H 2750 6600 50  0001 C CNN
-	1    2750 6600
-	-1   0    0    1
+P 15300 7550
+F 0 "D201" H 15293 7295 50  0000 C CNN
+F 1 "RED" H 15293 7386 50  0000 C CNN
+F 2 "LED_SMD:LED_0603_1608Metric_Pad1.05x0.95mm_HandSolder" H 15300 7550 50  0001 C CNN
+F 3 "~" H 15300 7550 50  0001 C CNN
+	1    15300 7550
+	1    0    0    1
 $EndComp
 $Comp
 L Device:LED D202
 U 1 1 5E66FC1B
-P 2750 7000
-F 0 "D202" H 2743 6745 50  0000 C CNN
-F 1 "GREEN" H 2743 6836 50  0000 C CNN
-F 2 "LED_SMD:LED_0603_1608Metric_Pad1.05x0.95mm_HandSolder" H 2750 7000 50  0001 C CNN
-F 3 "~" H 2750 7000 50  0001 C CNN
-	1    2750 7000
-	-1   0    0    1
+P 15500 1450
+F 0 "D202" H 15493 1195 50  0000 C CNN
+F 1 "GREEN" H 15493 1286 50  0000 C CNN
+F 2 "LED_SMD:LED_0603_1608Metric_Pad1.05x0.95mm_HandSolder" H 15500 1450 50  0001 C CNN
+F 3 "~" H 15500 1450 50  0001 C CNN
+	1    15500 1450
+	1    0    0    1
 $EndComp
 $Comp
 L Device:LED D203
 U 1 1 5E69BE69
-P 2750 7400
-F 0 "D203" H 2743 7145 50  0000 C CNN
-F 1 "BLUE" H 2743 7236 50  0000 C CNN
-F 2 "LED_SMD:LED_0603_1608Metric_Pad1.05x0.95mm_HandSolder" H 2750 7400 50  0001 C CNN
-F 3 "~" H 2750 7400 50  0001 C CNN
-	1    2750 7400
-	-1   0    0    1
-$EndComp
-Wire Wire Line
-	2550 7400 2550 7000
-Wire Wire Line
-	2550 6600 2600 6600
-Wire Wire Line
-	2600 7400 2550 7400
-Wire Wire Line
-	2550 7000 2600 7000
-Connection ~ 2550 7000
-Wire Wire Line
-	2550 7000 2550 6600
-Wire Wire Line
-	2500 7000 2550 7000
+P 15500 1850
+F 0 "D203" H 15493 1595 50  0000 C CNN
+F 1 "BLUE" H 15493 1686 50  0000 C CNN
+F 2 "LED_SMD:LED_0603_1608Metric_Pad1.05x0.95mm_HandSolder" H 15500 1850 50  0001 C CNN
+F 3 "~" H 15500 1850 50  0001 C CNN
+	1    15500 1850
+	1    0    0    1
+$EndComp
 $Comp
 L Sensor_Humidity:HDC1080 U201
@@
 A9
 Wire Wire Line
-	15050 1250 14800 1250
-Wire Wire Line
-	15050 1350 14800 1350
-Text Label 15050 1250 2    50   ~ 0
+	14950 1250 14800 1250
+Wire Wire Line
+	14950 1350 14800 1350
+Text Label 14950 1250 2    50   ~ 0
 A10
-Text Label 15050 1350 2    50   ~ 0
+Text Label 14950 1350 2    50   ~ 0
 A11
 Text HLabel 14850 1650 2    50   BiDi ~ 0
@@
 $EndComp
 Wire Wire Line
-	3200 6600 3250 6600
-Wire Wire Line
-	3250 6600 3250 6250
-Wire Wire Line
-	3200 7000 3300 7000
-Wire Wire Line
-	3300 7000 3300 6350
-Wire Wire Line
-	3350 7400 3350 6450
-Wire Wire Line
-	3200 7400 3350 7400
+	14850 7550 14800 7550
 Wire Wire Line
 	10450 10350 11050 10350
@@
 NoConn ~ 3400 5150
 NoConn ~ 3400 2550
-NoConn ~ 14800 1450
 NoConn ~ 14800 1550
 NoConn ~ 14800 2250
 NoConn ~ 14800 2150
 NoConn ~ 14800 1950
-NoConn ~ 14800 1850
 NoConn ~ 14800 3450
 NoConn ~ 14800 3550
 NoConn ~ 14800 3650
-NoConn ~ 14800 4850
-NoConn ~ 14800 4950
-NoConn ~ 14800 5050
 NoConn ~ 14800 5150
 NoConn ~ 14800 5250
@@
 NoConn ~ 3400 4350
 NoConn ~ 3400 4450
-NoConn ~ 3400 3750
 NoConn ~ 3400 2450
 NoConn ~ 3400 2350
@@
 	0    -1   -1   0
 $EndComp
-$Comp
-L power:+3.3V #PWR0214
-U 1 1 6036A38B
-P 2500 7000
-F 0 "#PWR0214" H 2500 6850 50  0001 C CNN
-F 1 "+3.3V" V 2500 7150 50  0000 L CNN
-F 2 "" H 2500 7000 50  0001 C CNN
-F 3 "" H 2500 7000 50  0001 C CNN
-	1    2500 7000
-	0    -1   -1   0
-$EndComp
 NoConn ~ 14800 7650
 NoConn ~ 14800 7750
@@
 Text Label 2250 6400 2    50   ~ 0
 MCU_SR_DAT
-Wire Wire Line
-	3350 6450 3400 6450
-Wire Wire Line
-	3400 6350 3300 6350
-Wire Wire Line
-	3250 6250 3400 6250
 $Comp
 L Device:C C204
@@
 	900  9400 950  9400
 Wire Wire Line
-	2900 5550 3400 5550
-Text Label 2900 5550 0    50   ~ 0
+	15300 4850 14800 4850
+Text Label 15300 4850 2    50   ~ 0
 MCU_SR_DAT
 Wire Wire Line
-	3400 5650 2900 5650
-Text Label 2900 5650 0    50   ~ 0
+	14800 5050 15300 5050
+Text Label 15300 5050 2    50   ~ 0
 MCU_SR_CLK
 Wire Wire Line
-	3400 5750 2900 5750
-Text Label 2900 5750 0    50   ~ 0
+	14800 4950 15300 4950
+Text Label 15300 4950 2    50   ~ 0
 MCU_SR_LAT
 Text HLabel 3350 5950 0    50   Output ~ 0
@@
 NoConn ~ 14800 3250
 NoConn ~ 14800 3350
+NoConn ~ 3400 5550
+NoConn ~ 3400 5650
+NoConn ~ 3400 5750
+NoConn ~ 14800 7350
+NoConn ~ 14800 7450
+$Comp
+L power:+3.3V #PWR0103
+U 1 1 5FEF1852
+P 15450 7550
+F 0 "#PWR0103" H 15450 7400 50  0001 C CNN
+F 1 "+3.3V" V 15450 7800 50  0000 C CNN
+F 2 "" H 15450 7550 50  0001 C CNN
+F 3 "" H 15450 7550 50  0001 C CNN
+	1    15450 7550
+	0    1    1    0
+$EndComp
+NoConn ~ 3400 6250
+$Comp
+L power:+3.3V #PWR0104
+U 1 1 5FF939B2
+P 15650 1450
+F 0 "#PWR0104" H 15650 1300 50  0001 C CNN
+F 1 "+3.3V" V 15650 1700 50  0000 C CNN
+F 2 "" H 15650 1450 50  0001 C CNN
+F 3 "" H 15650 1450 50  0001 C CNN
+	1    15650 1450
+	0    1    1    0
+$EndComp
+NoConn ~ 3400 6350
+NoConn ~ 3400 6450
+Wire Wire Line
+	15050 1850 14800 1850
+Wire Wire Line
+	14800 1450 15050 1450
+$Comp
+L power:+3.3V #PWR0105
+U 1 1 601108C9
+P 15650 1850
+F 0 "#PWR0105" H 15650 1700 50  0001 C CNN
+F 1 "+3.3V" V 15650 2100 50  0000 C CNN
+F 2 "" H 15650 1850 50  0001 C CNN
+F 3 "" H 15650 1850 50  0001 C CNN
+	1    15650 1850
+	0    1    1    0
+$EndComp
 Wire Bus Line
 	1400 3500 1400 4800

Commit message: PCB layout
Parts:
- added C228: 100n, Capacitor_SMD:C_0603_1608Metric_Pad1.08x0.95mm_HandSolder, symbol Device:C
- added R203, R204: 4k7, Resistor_SMD:R_0603_1608Metric_Pad0.98x0.95mm_HandSolder, symbol Device:R
- added U205: PCA9517, Package_SO:TSSOP-8_3x3mm_P0.65mm, symbol ETH3CDAQ1:PCA9517
- renumbered C206 to C204, C207 to C205, C212 to C206, C214 to C207, C216 to C208, C218 to C209, C220 to C210, C222 to C211, C224 to C212, C226 to C213, C227 to C214, C204 to C215, C205 to C216, C211 to C217, C213 to C218, C208 to C219, C209 to C220, C215 to C221, C210 to C222, C217 to C223, C219 to C224, C221 to C225, C223 to C226, C225 to C227, C228 to C229, R206 to R205, R207 to R206, R208 to R207, R203 to R208, R204 to R209, R205 to R210, R209 to R211, R210 to R212, U202 to U201, U203 to U202, U204 to U203, U201 to U204, U205 to U207
Connections:
- net +3V3: now also C228.1, R203.1, R204.1, U205.1 (VCCA), U205.5 (EN), U205.8 (VCCB)
- net EEPROM_SCL: now also U205.6 (SDAB)
- net EEPROM_SDA: now also U205.7 (SCLB)
- net GND: now also C228.2, U205.4 (GND)
- net DAC_~SYNC: now reaches U207.18 (PF6,TIM10_CH1,SPI5_NSS,SAI1_SD_B,UART7_RX,QUADSPI_BK1_IO3,EVENTOUT,ADC3_IN4)
- net DAC_SCLK: now reaches U207.19 (PF7,TIM11_CH1,SPI5_SCK,SAI1_MCLK_B,UART7_TX,QUADSPI_BK1_IO2,EVENTOUT,ADC3_IN5)
- net DAC_DIN: now reaches U207.21 (PF9,SPI5_MOSI,SAI1_FS_B,UART7_CTS,TIM14_CH1,QUADSPI_BK1_IO1,EVENTOUT,ADC3_IN7)
- net DAC_LDAC: now reaches U207.22 (PF10,QUADSPI_CLK,DCMI_D11,LCD_DE,EVENTOUT,ADC3_IN8)
- new net I2C_SCL: R203.2, U205.2 (SCLA)
- new net I2C_SDA: R204.2, U205.3 (SDAA)
- no-connect marks 48 -> 44
Other:
- moved on the sheet: C201, C202, C203, C204, C205, C206, C207, C208, C209, C210, C211, C212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

Commit message: Started development of first current measurement module. Added CAN to the DAQ module.
Parts:
- added C223: 100n, Capacitor_SMD:C_0603_1608Metric_Pad1.08x0.95mm_HandSolder, symbol Device:C
- added R203: 120, Resistor_SMD:R_0603_1608Metric_Pad0.98x0.95mm_HandSolder, symbol Device:R
- added R204: R, Resistor_SMD:R_0603_1608Metric_Pad0.98x0.95mm_HandSolder, symbol Device:R
- added U205: MCP2551-I-SN, Package_SO:SOIC-8_3.9x4.9mm_P1.27mm, symbol Interface_CAN_LIN:MCP2551-I-SN
- renumbered C223 to C224, C224 to C225, C225 to C226, C226 to C227, C227 to C228, C228 to C229, C229 to C230, R203 to R205, R204 to R206, R205 to R207, R206 to R208, R207 to R209, R208 to R210, R209 to R211, R210 to R212, R211 to R213, R212 to R214, U207 to U206, U205 to U207, U206 to U208
Connections:
- net +5V: now also C223.1, U205.3 (VDD)
- net GND: now also C223.2, R204.2, U205.2 (VSS)
- net CAN_RX: now reaches U206.103 (PA11,TIM1_CH4,SPI2_NSS,I2S2_WS,UART4_RX,USART1_CTS,CAN1_RX,OTG_FS_DM,LCD_R4,EVENTOUT)
- net CAN_RX: now also U205.4 (RXD)
- net CAN_TX: now reaches U206.104 (PA12,TIM1_ETR,SPI2_SCK,I2S2_CK,UART4_TX,USART1_RTS,SAI2_FS_B,CAN1_TX,OTG_FS_DP,LCD_R5,EVENTOUT)
- net CAN_TX: now also U205.1 (TXD)
- new net: R204.1, U205.8 (Rs)
- new net CANH: R203.1, U205.7 (CANH)
- new net CANL: R203.2, U205.6 (CANL)
- no-connect marks 44 -> 43
Other:
- moved on the sheet: C224, C225, C226, C227, C228, C229, J201, R205, R206, R207, R208, U207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

Commit message: Modification in PCBs. Created BOM files.
Parts:
- R204: value R -> 1k
Connections:
- net at R211.1: now also U206.88 (PG3,FMC_A13,EVENTOUT); no longer U206.87 (PG2,FMC_A12,EVENTOUT)
- new net A12: U206.87 (PG2,FMC_A12,EVENTOUT)
- no-connect marks 43 -> 42
Other:
- moved on the sheet: C215, C216, C219, C220, C222, C230, D201, D202, D203, J202, R209, R210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

Commit message: Changed 24LC08 to 24LC024. Added fixes to ethernetif.c to solve the problem with D Cache and RX deadlock. The fixes are also in ethernetif_fix.c, because code generator will overwrite ethernetif.c.
Parts:
- U208: value 24LC08B-E/MS -> 24LC024T-I/MS
Changed lines of the file:
@@
 P 15300 15200
 F 0 "U208" H 15650 15550 50  0000 C CNN
-F 1 "24LC08B-E/MS" H 15650 15450 50  0000 C CNN
+F 1 "24LC024T-I/MS" H 15650 15450 50  0000 C CNN
 F 2 "Package_SO:MSOP-8_3x3mm_P0.65mm" H 15300 15200 50  0001 C CNN
 F 3 "http://ww1.microchip.com/downloads/en/DeviceDoc/21710J.pdf" H 15300 15200 50  0001 C CNN

Commit message: PCB and software development.
Connections:
- net EEPROM_SCL: now also U207.7 (SCLB); no longer U207.6 (SDAB)
- net EEPROM_SDA: now also U207.6 (SDAB); no longer U207.7 (SCLB)
Changed lines of the file:
@@
 Wire Wire Line
 	15800 13350 15800 13300
+Text Label 16300 13550 2    50   ~ 0
+EEPROM_SDA
 Text Label 16300 13450 2    50   ~ 0
-EEPROM_SDA
-Text Label 16300 13550 2    50   ~ 0
 EEPROM_SCL
 Wire Wire Line
+	16300 13550 15700 13550
+Wire Wire Line
 	16300 13450 15700 13450
-Wire Wire Line
-	16300 13550 15700 13550
 Text HLabel 13700 13450 0    50   BiDi ~ 0
 I2C_SCL
