File: hardware/project/ETH3CDAQ1_CURRENT_ISO_T2/ETH3CDAQ1_CURRENT_ISO_T2.kicad_pcb (KiCad board)
At the start: 2 copper layers, 80 x 30 mm, 80 parts, among them J1 GMSTB2,5/2-GF-7,62, J2 Conn_02x10_Odd_Even, K1 G5Q-1, U1 DG211, U10 74LVC1GU04DRL, U11 74LVC1GU04DRL, U12 74LVC1GU04DRL, U13 24LC08B-E/MS, U14 TXB0104PW, U15 PCA9557PW, U17 LM3480-12, U18 FODM214, U2 DG419xY, U3 LT3032, U4 OPA140, U5 ISO124, U6 ADuM5410, U7 DCP020515DU, U8 OPA237_SOT23, U9 LT3032-15

Commit message: PCB layout
Parts:
- added R1: 100k, Resistor_SMD:R_0603_1608Metric_Pad0.98x0.95mm_HandSolder, B.Cu at (104.4, 54.7)
- added R2: 316, Resistor_SMD:R_0603_1608Metric_Pad0.98x0.95mm_HandSolder, B.Cu at (104.4, 51.3)
- added U16: OPA132, Package_SO:SOIC-8_3.9x4.9mm_P1.27mm, B.Cu at (108.3, 53.1)
- U3: moved to B.Cu
- moved U3 133.2 mm to (119.4, 48.4), turned to 90 degrees
- moved U8 132.3 mm to (140.0, 60.6)
- moved U9 125.2 mm to (140.0, 67.3)
- moved R10 7.62 mm to (132.6, 56.3)
- moved U18 7.62 mm to (126.4, 56.9)
- moved R3 3.33 mm to (102.2, 65.5)
- moved U15 2.38 mm to (140.0, 55.1)
- moved U1 2.22 mm to (140.0, 49.3)
- moved R5 0.64 mm to (109.0, 59.8)
- moved D1 0.40 mm to (102.4, 44.2)
- moved U17 0.40 mm to (102.4, 47.4)
- moved D2 0.36 mm to (93.2, 49.3)
- moved K1 0.36 mm to (98.4, 44.2)
- moved R4 0.18 mm to (102.5, 67.9)
- moved U2 0.13 mm to (114.2, 57.5)
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
Commit message: Modifications in PCBs.
Parts:
- C1, C10, C14, C18, C19, C23, C30, C31, C4, C5, C7, C9, FB2, FB3, R14, R15, R16, R17, R18, R19, R20, R21, R22, R23, R24, R26, R6, R7, R8, R9, U11: moved to B.Cu
- moved C7 182.8 mm to (111.6, 56.9), turned to 270 degrees
- moved R16 176.0 mm to (113.2, 62.4)
- moved C17 171.2 mm to (118.2, 55.4), turned to 180 degrees
- moved U12 167.3 mm to (133.3, 56.1), turned to 180 degrees
- moved C14 166.0 mm to (109.6, 44.7)
- moved U11 165.6 mm to (133.3, 56.1), turned to 180 degrees
- moved C23 165.5 mm to (136.0, 66.3), turned to 270 degrees
- moved U10 165.1 mm to (133.3, 58.4), turned to 180 degrees
- moved R18 162.4 mm to (118.2, 56.9)
- moved C10 162.2 mm to (111.6, 48.6), turned to 270 degrees
- moved C31 159.9 mm to (107.2, 54.1)
- moved C4 159.4 mm to (120.0, 46.0), turned to 180 degrees
- moved R9 158.8 mm to (122.8, 47.0), turned to 90 degrees
- moved R20 156.1 mm to (141.6, 60.7)
- moved R14 154.5 mm to (115.6, 65.3)
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Routing:
- net (no net): track 0.00 -> 71.1 mm
Other:
- copper layers 2 -> 4
- board text added: "1"
- board text added: "2"
- board text added: "3"
- board text added: "4"

Commit message: PCB design
Parts:
- added C32: 10u, Capacitor_SMD:C_0603_1608Metric_Pad1.08x0.95mm_HandSolder, B.Cu at (133.5, 46.0)
- added C33: 100n, Capacitor_SMD:C_0603_1608Metric_Pad1.08x0.95mm_HandSolder, B.Cu at (133.5, 48.3)
- C11, C12, C13, C2, C20, C21, C27, C28, C29, C3, C6, C8, R25: moved to B.Cu
- C14: value 100n -> 10u
- C15: value 100n -> 10u; moved to B.Cu
- moved C15 161.5 mm to (121.8, 68.5)
- moved C8 159.0 mm to (115.6, 64.1)
- moved C25 155.4 mm to (139.4, 63.6), turned to 180 degrees
- moved C24 155.3 mm to (139.4, 70.1), turned to 180 degrees
- moved C27 154.2 mm to (142.9, 63.5), turned to 90 degrees
- moved C16 152.6 mm to (118.2, 58.4)
- moved C12 149.4 mm to (115.8, 43.3), turned to 180 degrees
- moved C13 148.4 mm to (121.8, 43.3)
- moved C6 147.6 mm to (109.5, 45.0)
- moved C28 146.6 mm to (130.0, 51.8), turned to 90 degrees
- moved C2 133.9 mm to (111.9, 68.2), turned to 180 degrees
- moved C29 130.3 mm to (130.0, 59.4), turned to 90 degrees
- moved C3 128.1 mm to (111.8, 48.6), turned to 270 degrees
- moved R25 127.8 mm to (138.8, 54.7), turned to 90 degrees
- moved C26 127.3 mm to (142.9, 63.5), turned to 90 degrees
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Routing:
- added copper zone on In1.Cu, net GND

Commit message: PCB design.
Parts:
- moved C22 0.38 mm to (143.3, 67.8)
- moved C26 0.38 mm to (143.3, 63.5)
- moved C10 0.25 mm to (116.2, 70.7)
- moved C14 0.25 mm to (116.2, 68.5)
Routing:
- net AGNDF: track 0.00 -> 108.6 mm, vias 0 -> 25
- net -15VF: track 0.00 -> 43.2 mm, vias 0 -> 11
- net Net-(D2-Pad1): track 0.00 -> 37.0 mm
- net Net-(D2-Pad3): track 0.00 -> 33.8 mm
- net +5VF: track 0.00 -> 29.1 mm, vias 0 -> 5
- net /RLY: track 0.00 -> 28.7 mm
- net Net-(R15-Pad1): track 0.00 -> 24.8 mm, vias 0 -> 3
- net /G1: track 0.00 -> 19.3 mm, vias 0 -> 2
- net /A0: track 0.00 -> 18.0 mm
- net Net-(U1-Pad11): track 0.00 -> 17.4 mm
- net +15VF: track 0.00 -> 16.6 mm, vias 0 -> 12
- net /AZ: track 0.00 -> 15.4 mm
- net /G10: track 0.00 -> 14.3 mm, vias 0 -> 2
- net Net-(K1-Pad4): track 0.00 -> 12.7 mm
- net /A1: track 0.00 -> 12.2 mm
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- added copper zone on B.Cu, net +15V
- added copper zone on F.Cu, net +15V
- added copper zone on B.Cu, net +15VF
- added copper zone on F.Cu, net +15VF
- added copper zone on In2.Cu, net +15VF
- added copper zone on B.Cu, net +18V
- added copper zone on F.Cu, net +18V
- added copper zone on In2.Cu, net +5VF
- added copper zone on B.Cu, net -15V
- added copper zone on F.Cu, net -15V
- added copper zone on B.Cu, net -15VF
- added copper zone on F.Cu, net -15VF
- added copper zone on In2.Cu, net -15VF
- added copper zone on B.Cu, net -18V
- added copper zone on F.Cu, net -18V
- added copper zone on B.Cu, net AGNDF
- added copper zone on F.Cu, net AGNDF
- added copper zone on In1.Cu, net AGNDF
- added copper zone on B.Cu, net GND
- added copper zone on F.Cu, net GND
- added copper zone on B.Cu, net VCC
- added copper zone on F.Cu, net VCC
- added copper zone on B.Cu, net VDD
- added copper zone on F.Cu, net VDD
Other:
- net class Default: clearance 0.2 -> 0.127; trace_width 0.25 -> 0.127; via_dia 0.8 -> 0.5; via_drill 0.4 -> 0.2
- rule trace_clearance: 0.2 -> 0.127
- rule trace_min: 0.2 -> 0.127
- rule via_min_drill: 0.3 -> 0.2

Commit message: PCB design
Parts:
- moved C2 1.81 mm to (113.3, 69.3), turned to 270 degrees
- moved C32 1.02 mm to (132.6, 46.5)
- moved C33 1.02 mm to (132.6, 48.8)
- moved C20 0.13 mm to (135.8, 70.1)
- moved U18 0.10 mm to (126.5, 55.9)
Routing:
- net +3V3: track 0.00 -> 23.8 mm, vias 0 -> 5
- net /AOUT: track 0.00 -> 22.6 mm
- net Net-(K1-Pad3): track 2.78 -> 22.9 mm
- net Net-(R20-Pad2): track 0.00 -> 18.9 mm, vias 0 -> 2
- net AGNDF: track 108.6 -> 126.8 mm
- net -15V: track 6.82 -> 23.1 mm, vias 7 -> 8
- net /SCL: track 11.7 -> 25.3 mm
- net GND: track 7.82 -> 19.3 mm, vias 7 -> 18
- net +15VF: track 16.6 -> 27.5 mm
- net +5V: track 2.99 -> 13.4 mm, vias 2 -> 9
- net +15V: track 3.45 -> 10.8 mm
- net /SDA: track 10.2 -> 17.1 mm
- net /WP: track 0.00 -> 6.45 mm
- net Net-(C19-Pad1): track 0.00 -> 5.06 mm, vias 0 -> 1
- net -15VF: track 43.2 -> 39.0 mm
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- added copper zone on In2.Cu, net +18V
- added copper zone on In2.Cu, net +3V3
- added copper zone on B.Cu, net +5V
- added copper zone on F.Cu, net +5V
- added copper zone on In2.Cu, net +5V
