File: hardware/project/ETH3CDAQ1_CURRENT_ISO_T1/ETH3CDAQ1_CURRENT_ISO_T1.sch (KiCad schematic (older format))
At the start: 25 parts, among them J1 PC 5/2-G-7.62, J2 Conn_02x10_Odd_Even, U1 L78L15_SOT89, U2 L79L15_SOT89, U3 T60404-N4646-X400, U4 STM32F042K6Tx, U5 MCP2551-I-SN, U6 24LC08B-E/MS, U7 PCA9557PW

Commit message: Voltage front-end development
Parts:
- added R?: 120, symbol Device:R
Connections:
- net labels added: +5V, CANH, CANL
- wire segments 98 -> 109
- no-connect marks 3 -> 2
Changed lines of the file:
@@
 Wire Wire Line
 	9750 3700 9900 3700
-Text Label 9750 3800 0    50   ~ 0
-A2
-Wire Wire Line
-	9750 3800 9900 3800
 Text Label 8650 1300 2    50   ~ 0
 EEPROM_WP
@@
 	0    1    1    0
 $EndComp
-$Comp
-L power:GND #PWR019
-U 1 1 5FC3CF72
-P 10400 3800
-F 0 "#PWR019" H 10400 3550 50  0001 C CNN
-F 1 "GND" V 10400 3650 50  0000 R CNN
-F 2 "" H 10400 3800 50  0001 C CNN
-F 3 "" H 10400 3800 50  0001 C CNN
-	1    10400 3800
-	0    -1   -1   0
-$EndComp
 Wire Wire Line
 	10400 3600 10700 3600
@@
 	10050 5400 10050 5350
 Connection ~ 10050 5350
-NoConn ~ 10400 4400
 $Comp
 L ETH3CDAQ1:-18V #PWR014
@@
 L Interface_CAN_LIN:MCP2551-I-SN U5
 U 1 1 5FCB9237
-P 7600 5550
-F 0 "U5" H 7600 6131 50  0000 C CNN
-F 1 "MCP2551-I-SN" H 7600 6040 50  0000 C CNN
-F 2 "Package_SO:SOIC-8_3.9x4.9mm_P1.27mm" H 7600 5050 50  0001 C CIN
-F 3 "http://ww1.microchip.com/downloads/en/devicedoc/21667d.pdf" H 7600 5550 50  0001 C CNN
-	1    7600 5550
+P 8400 5400
+F 0 "U5" H 8700 5850 50  0000 C CNN
+F 1 "MCP2551-I-SN" H 8750 5750 50  0000 C CNN
+F 2 "Package_SO:SOIC-8_3.9x4.9mm_P1.27mm" H 8400 4900 50  0001 C CIN
+F 3 "http://ww1.microchip.com/downloads/en/devicedoc/21667d.pdf" H 8400 5400 50  0001 C CNN
+	1    8400 5400
 	1    0    0    -1
 $EndComp
@@
 	1    0    0    -1
 $EndComp
+$Comp
+L power:+5V #PWR?
+U 1 1 5FC1802D
+P 10400 4400
+F 0 "#PWR?" H 10400 4250 50  0001 C CNN
+F 1 "+5V" V 10400 4550 50  0000 L CNN
+F 2 "" H 10400 4400 50  0001 C CNN
+F 3 "" H 10400 4400 50  0001 C CNN
+	1    10400 4400
+	0    1    1    0
+$EndComp
+Wire Wire Line
+	10400 3800 10700 3800
+Text Label 10700 3800 2    50   ~ 0
+CANL
+Wire Wire Line
+	9900 3800 9600 3800
+Text Label 9600 3800 0    50   ~ 0
+CANH
+Wire Wire Line
+	9100 5200 9400 5200
+Text Label 9400 5200 2    50   ~ 0
+CANH
+$Comp
+L Device:R R?
+U 1 1 5FC28721
+P 9100 5400
+F 0 "R?" H 9170 5446 50  0000 L CNN
+F 1 "120" H 9170 5355 50  0000 L CNN
+F 2 "" V 9030 5400 50  0001 C CNN
+F 3 "~" H 9100 5400 50  0001 C CNN
+	1    9100 5400
+	1    0    0    -1
+$EndComp
+Wire Wire Line
+	8900 5300 8950 5300
+Wire Wire Line
+	8950 5300 8950 5200
+Wire Wire Line
+	8950 5200 9100 5200
+Wire Wire Line
+	9100 5200 9100 5250
+Wire Wire Line
+	8900 5500 8950 5500
+Wire Wire Line
+	8950 5500 8950 5600
+Wire Wire Line
+	8950 5600 9100 5600
+Wire Wire Line
+	9100 5600 9100 5550
+Connection ~ 9100 5200
+Wire Wire Line
+	9100 5600 9400 5600
+Text Label 9400 5600 2    50   ~ 0
+CANL
+$Comp
+L power:+5V #PWR?
+U 1 1 5FC39469
+P 8400 5000
+F 0 "#PWR?" H 8400 4850 50  0001 C CNN
+F 1 "+5V" H 8415 5173 50  0000 C CNN
+F 2 "" H 8400 5000 50  0001 C CNN
+F 3 "" H 8400 5000 50  0001 C CNN
+	1    8400 5000
+	1    0    0    -1
+$EndComp
+$Comp
+L power:GND #PWR?
+U 1 1 5FC39C9E
+P 8400 5800
+F 0 "#PWR?" H 8400 5550 50  0001 C CNN
+F 1 "GND" H 8405 5627 50  0000 C CNN
+F 2 "" H 8400 5800 50  0001 C CNN
+F 3 "" H 8400 5800 50  0001 C CNN
+	1    8400 5800
+	1    0    0    -1
+$EndComp
+Connection ~ 9100 5600
 $EndSCHEMATC

Commit message: PCB design
Parts:
- removed C1, C2, C3, C4: 10u/35V, symbol Device:C
- removed FB1, FB2: Ferrite_Bead, symbol Device:Ferrite_Bead
- removed R?: 120, symbol Device:R
- removed U1: L78L15_SOT89, Package_TO_SOT_SMD:SOT-89-3, symbol Regulator_Linear:L78L15_SOT89
- removed U2: L79L15_SOT89, Package_TO_SOT_SMD:SOT-89-3, symbol Regulator_Linear:L79L15_SOT89
- removed U4: STM32F042K6Tx, Package_QFP:LQFP-32_7x7mm_P0.8mm, symbol MCU_ST_STM32F0:STM32F042K6Tx
- removed U5: MCP2551-I-SN, Package_SO:SOIC-8_3.9x4.9mm_P1.27mm, symbol Interface_CAN_LIN:MCP2551-I-SN
Connections:
- wire segments 109 -> 65

Commit message: Current module development
Parts:
- removed C5: C, symbol Device:C
- added C? (x2): 100n, symbol Device:C
- added C? (x2): 10u, symbol Device:C
- added C? (x2): 2u2, symbol Device:C
- added R5: 18k, symbol Device:R
- added R6: 2k, symbol Device:R
- added R?: 0, symbol Device:R
- added R? (x2): 10k, symbol Device:R
- added U1: DG419xY, Package_SO:SOIC-8_3.9x4.9mm_P1.27mm, symbol Analog_Switch:DG419xY
- added U2: DG211, symbol ETH3CDAQ1:DG211
- added U4: OPA140, symbol ETH3CDAQ1:OPA140
- added U5: LT3032-15, Package_DFN_QFN:Linear_DE14MA, symbol Regulator_Linear:LT3032-15
- added U? (x3): 74LVC1GU04DRL, Package_TO_SOT_SMD:SOT-553, symbol 74xGxx:74LVC1GU04DRL
- added U?: TXB0104PW, Package_SO:TSSOP-14_4.4x5mm_P0.65mm, symbol Logic_LevelTranslator:TXB0104PW
- R1: value 22 -> 100
- R2: value R -> 180k
- R3: value 0 -> 100k
Connections:
- net A2 is gone; now on net GND: U6.3 (A2), U7.5 (A2)
- net +15V: now also C?.1, C?.1, U1.4 (V+), U2.13 (V+), U4.7 (V+), U5.1 (OUTP)
- net +18V: now also C?.1, U5.12 (~SHDNP), U5.14 (INP)
- net +3V3: now also R?.1, U?.1 (VCCA)
- net +5V: now also R?.2, U1.5 (VL), U2.12 (VL), U?.14 (VCCB), U?.5 (VCC), U?.5 (VCC), U?.5 (VCC)
- net -15V: now also C?.1, C?.1, U1.7 (V-), U2.4 (V-), U4.4 (V-), U5.7 (OUTN)
- net -18V: now also C?.1, U5.10 (~SHDNN), U5.6 (INN), U5.9 (INN)
- net A0: no longer U6.1 (A0)
- net A1: no longer U6.2 (A1)
- net ANALOG_OUT: now also R2.1, U2.3, U4.6
- net GND: now also C?.2, C?.2, C?.2, C?.2, R6.2, U1.3 (GND), U1.8, U2.5 (GND), U5.4 (GND), U5.5 (GND), U?.3 (GND), U?.3 (GND), U?.3 (GND), U?.7 (GND)
- net at R2.2: now also R5.1, U2.6
- net IO3: now reaches U7.10 (IO3)
- net IO3: now also U?.4 (A3)
- net IO4: now reaches U7.11 (IO4)
- net IO4: now also U?.3 (A2)
- net IO5: now reaches U7.12 (IO5)
- net IO5: now also U?.2 (A1)
- net IO2: now reaches U7.9 (IO2)
- net IO2: now also U?.5 (A4)
- net EEPROM_WP renamed WP
- net Is: no longer names the net of C6.1, R1.1, R3.2, U3.7 (Is)
- net Vs1: no longer names the net of R3.1
- net Vs1: now also U1.2
- new net: C?.2, U5.3 (BYPP)
- new net: C?.2, U5.11 (BYPN)
- new net: U1.1, U4.3 (+)
- new net: U2.11, U2.2, U2.7, U4.2 (-)
- new net: U2.14, U2.15
- new net: R?.1, U2.16
- new net: R5.2, R6.1, U2.10
- new net: R?.1, U?.13 (B1), U?.2
- new net: U?.12 (B2), U?.2
- new net: U?.11 (B3), U?.2
- new net: R?.2, U?.8 (OE)
- new net AZ: U1.6, U?.10 (B4)
- new net G1: R?.2, U2.1, U?.4
- new net G10: U2.8, U?.4
- new net G100: U2.9, U?.4
- no-connect marks 2 -> 4
Other:
- note removed: "OPTION A"
- moved on the sheet: C6, C7, H1, H2, J1, J2, R1, R3, R4, RV1, U3, U6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

Commit message: PCB design
Parts:
- added R10, R11: 4k7, Resistor_SMD:R_0603_1608Metric_Pad0.98x0.95mm_HandSolder, symbol Device:R
- C1, C2, C3, C4, C5, C8: renamed from C?; footprint (none) -> Capacitor_SMD:C_0603_1608Metric_Pad1.08x0.95mm_HandSolder
- C6, C7: footprint (none) -> Capacitor_SMD:C_0603_1608Metric_Pad1.08x0.95mm_HandSolder
- J1: footprint (none) -> ETH3CDAQ1:PC5_2-G-7_62
- R2: value 180k -> 180k/0.05%; footprint (none) -> Resistor_SMD:R_0603_1608Metric_Pad0.98x0.95mm_HandSolder
- R3, R4: footprint (none) -> Resistor_SMD:R_0603_1608Metric_Pad0.98x0.95mm_HandSolder
- R5: value 18k -> 18k/0.05%; footprint (none) -> Resistor_SMD:R_0603_1608Metric_Pad0.98x0.95mm_HandSolder
- R6: value 2k -> 2k/0.05%; footprint (none) -> Resistor_SMD:R_0603_1608Metric_Pad0.98x0.95mm_HandSolder
- R7, R8, R9: renamed from R?; footprint (none) -> Resistor_SMD:R_0603_1608Metric_Pad0.98x0.95mm_HandSolder
- RV1: footprint (none) -> ETH3CDAQ1:4032
- U2, U7: footprint (none) -> Package_SO:TSSOP-16_4.4x5mm_P0.65mm
- U3: footprint (none) -> ETH3CDAQ1:T60404-N4646-X400
- U4: footprint (none) -> Package_SO:SOIC-8_3.9x4.9mm_P1.27mm
- U6: footprint (none) -> Package_SO:MSOP-8_3x3mm_P0.65mm
- gave numbers to parts that had none: 4
Connections:
- net +3V3: now also R10.1, R11.1
- net A0: now also U6.1 (A0)
- net A1: now also U6.2 (A1)
- net I2C_SCL: now also R11.2
- net I2C_SDA: now also R10.2
- net at RV1.1, U3.1 (Ip), U3.2 (Ip)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: now also J1.2 (Pin_2); no longer J1.1 (Pin_1)
- net at RV1.2, U3.4 (Ip), U3.5 (Ip)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: now also J1.1 (Pin_1); no longer J1.2 (Pin_2)
Other:
- moved on the sheet: U6

Commit message: PCB design
Parts:
- added C10, C11, C12, C13, C14, C15, C16, C17, C18, C19, C20, C21, C22, C9: 100n, Capacitor_SMD:C_0603_1608Metric_Pad1.08x0.95mm_HandSolder, symbol Device:C
- C6: footprint Capacitor_SMD:C_0603_1608Metric_Pad1.08x0.95mm_HandSolder -> Capacitor_SMD:C_1206_3216Metric_Pad1.33x1.80mm_HandSolder
- R1: footprint (none) -> Resistor_SMD:R_1206_3216Metric_Pad1.30x1.75mm_HandSolder
Connections:
- net +15V: now also C10.1, C11.1, C12.1, C9.1
- net +3V3: now also C20.1, C21.1, C22.1
- net +5V: now also C17.1, C18.1, C19.1
- net -15V: now also C13.1, C14.1, C15.1, C16.1
- net GND: now also C10.2, C11.2, C12.2, C13.2, C14.2, C15.2, C16.2, C17.2, C18.2, C19.2, C20.2, C21.2, C22.2, C9.2
Other:
- note added: "URG3216L-101-L-T05"
- moved on the sheet: C1, C2, C3, C4, C5, C6, C7, C8, H1, H2, J1, J2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

Commit message: PCB design
Parts:
- added FB1, FB2: Ferrite_Bead_Small, Resistor_SMD:R_0603_1608Metric_Pad0.98x0.95mm_HandSolder, symbol Device:Ferrite_Bead_Small
Connections:
- net +15V: now also FB1.2
- net +18V: now also FB1.1
- net -15V: now also FB2.2
- net -18V: now also FB2.1
Changed lines of the file:
@@
 Text Notes 4650 3100 0    50   ~ 0
 URG3216L-101-L-T05
+$Comp
+L Device:Ferrite_Bead_Small FB2
+U 1 1 5FCB1998
+P 9350 9550
+F 0 "FB2" V 9113 9550 50  0000 C CNN
+F 1 "Ferrite_Bead_Small" V 9204 9550 50  0000 C CNN
+F 2 "Resistor_SMD:R_0603_1608Metric_Pad0.98x0.95mm_HandSolder" V 9280 9550 50  0001 C CNN
+F 3 "~" H 9350 9550 50  0001 C CNN
+	1    9350 9550
+	0    1    1    0
+$EndComp
+$Comp
+L Device:Ferrite_Bead_Small FB1
+U 1 1 5FCB2CF0
+P 9350 9100
+F 0 "FB1" V 9113 9100 50  0000 C CNN
+F 1 "Ferrite_Bead_Small" V 9204 9100 50  0000 C CNN
+F 2 "Resistor_SMD:R_0603_1608Metric_Pad0.98x0.95mm_HandSolder" V 9280 9100 50  0001 C CNN
+F 3 "~" H 9350 9100 50  0001 C CNN
+	1    9350 9100
+	0    1    1    0
+$EndComp
+$Comp
+L ETH3CDAQ1:+18V #PWR0130
+U 1 1 5FCB31FE
+P 9450 9100
+F 0 "#PWR0130" H 9450 8950 50  0001 C CNN
+F 1 "+18V" V 9450 9350 50  0000 C CNN
+F 2 "" H 9450 9100 50  0001 C CNN
+F 3 "" H 9450 9100 50  0001 C CNN
+	1    9450 9100
+	0    1    1    0
+$EndComp
+$Comp
+L power:+15V #PWR0131
+U 1 1 5FCB3CDC
+P 9250 9100
+F 0 "#PWR0131" H 9250 8950 50  0001 C CNN
+F 1 "+15V" V 9250 9350 50  0000 C CNN
+F 2 "" H 9250 9100 50  0001 C CNN
+F 3 "" H 9250 9100 50  0001 C CNN
+	1    9250 9100
+	0    -1   -1   0
+$EndComp
+$Comp
+L ETH3CDAQ1:-18V #PWR0132
+U 1 1 5FCB4ECB
+P 9450 9550
+F 0 "#PWR0132" H 9450 9400 50  0001 C CNN
+F 1 "-18V" V 9450 9800 50  0000 C CNN
+F 2 "" H 9450 9550 50  0001 C CNN
+F 3 "" H 9450 9550 50  0001 C CNN
+	1    9450 9550
+	0    1    1    0
+$EndComp
+$Comp
+L power:-15V #PWR0133
+U 1 1 5FCB6FB5
+P 9250 9550
+F 0 "#PWR0133" H 9250 9650 50  0001 C CNN
+F 1 "-15V" V 9250 9800 50  0000 C CNN
+F 2 "" H 9250 9550 50  0001 C CNN
+F 3 "" H 9250 9550 50  0001 C CNN
+	1    9250 9550
+	0    -1   -1   0
+$EndComp
 $EndSCHEMATC

Commit message: PCB design
Connections:
- net ANALOG_OUT: no longer J2.7 (Pin_7), J2.8 (Pin_8)
- net GND: now also J2.7 (Pin_7), J2.8 (Pin_8)
Changed lines of the file:
@@
 	14300 8600 14250 8600
 Wire Wire Line
-	14250 8600 14250 8500
-Wire Wire Line
-	14250 8400 14300 8400
+	14250 8600 14250 8550
 Wire Wire Line
 	14300 8500 14250 8500
-Connection ~ 14250 8500
-Wire Wire Line
-	14250 8500 14250 8400
-Text Label 13750 8500 0    50   ~ 0
+Text Label 13750 8550 0    50   ~ 0
 ANALOG_OUT
 Wire Wire Line
-	14250 8500 13750 8500
+	14250 8550 13750 8550
 Wire Wire Line
 	14800 8600 14850 8600
 Wire Wire Line
-	14850 8600 14850 8500
-Wire Wire Line
-	14850 8400 14800 8400
+	14850 8600 14850 8550
 Wire Wire Line
 	14800 8500 14850 8500
-Connection ~ 14850 8500
-Wire Wire Line
-	14850 8500 14850 8400
-Text Label 15350 8500 2    50   ~ 0
+Text Label 15350 8550 2    50   ~ 0
 ANALOG_OUT
 Wire Wire Line
-	14850 8500 15350 8500
+	14850 8550 15350 8550
 NoConn ~ 14300 8900
 $Comp
@@
 	0    -1   -1   0
 $EndComp
+$Comp
+L power:GND #PWR?
+U 1 1 5FCC1D19
+P 14300 8400
+F 0 "#PWR?" H 14300 8150 50  0001 C CNN
+F 1 "GND" V 14300 8250 50  0000 R CNN
+F 2 "" H 14300 8400 50  0001 C CNN
+F 3 "" H 14300 8400 50  0001 C CNN
+	1    14300 8400
+	0    1    1    0
+$EndComp
+$Comp
+L power:GND #PWR?
+U 1 1 5FCC253E
+P 14800 8400
+F 0 "#PWR?" H 14800 8150 50  0001 C CNN
+F 1 "GND" V 14800 8250 50  0000 R CNN
+F 2 "" H 14800 8400 50  0001 C CNN
+F 3 "" H 14800 8400 50  0001 C CNN
+	1    14800 8400
+	0    -1   -1   0
+$EndComp
+Connection ~ 14250 8550
+Wire Wire Line
+	14250 8550 14250 8500
+Connection ~ 14850 8550
+Wire Wire Line
+	14850 8550 14850 8500
 $EndSCHEMATC

Commit message: Modification in PCBs. Created BOM files.
Parts:
- R1: value 100 -> URG3216L-101-L-T05
Connections:
- net CANH: no longer names the net of J2.5 (Pin_5)
- net CANL: no longer names the net of J2.6 (Pin_6)
- no-connect marks 4 -> 8
Other:
- note removed: "URG3216L-101-L-T05"
Changed lines of the file:
@@
 P 5100 2500
 F 0 "R1" H 5170 2546 50  0000 L CNN
-F 1 "100" H 5170 2455 50  0000 L CNN
+F 1 "URG3216L-101-L-T05 " H 4650 2800 50  0000 L CNN
 F 2 "Resistor_SMD:R_1206_3216Metric_Pad1.30x1.75mm_HandSolder" V 5030 2500 50  0001 C CNN
 F 3 "~" H 5100 2500 50  0001 C CNN
@@
 	0    1    1    0
 $EndComp
-Wire Wire Line
-	14800 8300 15100 8300
-Text Label 15100 8300 2    50   ~ 0
-CANL
-Wire Wire Line
-	14300 8300 14000 8300
-Text Label 14000 8300 0    50   ~ 0
-CANH
 $Comp
 L power:GND #PWR01
@@
 	1    0    0    -1
 $EndComp
-Text Notes 4650 3100 0    50   ~ 0
-URG3216L-101-L-T05
 $Comp
 L Device:Ferrite_Bead_Small FB2
@@
 $EndComp
 $Comp
-L power:GND #PWR?
+L power:GND #PWR0134
 U 1 1 5FCC1D19
 P 14300 8400
-F 0 "#PWR?" H 14300 8150 50  0001 C CNN
+F 0 "#PWR0134" H 14300 8150 50  0001 C CNN
 F 1 "GND" V 14300 8250 50  0000 R CNN
 F 2 "" H 14300 8400 50  0001 C CNN
@@
 $EndComp
 $Comp
-L power:GND #PWR?
+L power:GND #PWR0135
 U 1 1 5FCC253E
 P 14800 8400
-F 0 "#PWR?" H 14800 8150 50  0001 C CNN
+F 0 "#PWR0135" H 14800 8150 50  0001 C CNN
 F 1 "GND" V 14800 8250 50  0000 R CNN
 F 2 "" H 14800 8400 50  0001 C CNN
@@
 Wire Wire Line
 	14850 8550 14850 8500
+NoConn ~ 14300 8300
+NoConn ~ 14800 8300
+NoConn ~ 13750 2000
+NoConn ~ 13750 2100
+$Comp
+L power:PWR_FLAG #FLG0101
+U 1 1 5FF00015
+P 11900 9550
+F 0 "#FLG0101" H 11900 9625 50  0001 C CNN
+F 1 "PWR_FLAG" H 11900 9723 50  0000 C CNN
+F 2 "" H 11900 9550 50  0001 C CNN
+F 3 "~" H 11900 9550 50  0001 C CNN
+	1    11900 9550
+	-1   0    0    1
+$EndComp
+$Comp
+L power:+3.3V #PWR0136
+U 1 1 5FF0071D
+P 11900 9550
+F 0 "#PWR0136" H 11900 9400 50  0001 C CNN
+F 1 "+3.3V" H 11915 9723 50  0000 C CNN
+F 2 "" H 11900 9550 50  0001 C CNN
+F 3 "" H 11900 9550 50  0001 C CNN
+	1    11900 9550
+	1    0    0    -1
+$EndComp
+$Comp
+L power:PWR_FLAG #FLG0102
+U 1 1 5FF00F4D
+P 12350 9550
+F 0 "#FLG0102" H 12350 9625 50  0001 C CNN
+F 1 "PWR_FLAG" H 12350 9723 50  0000 C CNN
+F 2 "" H 12350 9550 50  0001 C CNN
+F 3 "~" H 12350 9550 50  0001 C CNN
+	1    12350 9550
+	-1   0    0    1
+$EndComp
+$Comp
+L power:+5V #PWR0137
+U 1 1 5FF019AA
+P 12350 9550
+F 0 "#PWR0137" H 12350 9400 50  0001 C CNN
+F 1 "+5V" H 12365 9723 50  0000 C CNN
+F 2 "" H 12350 9550 50  0001 C CNN
+F 3 "" H 12350 9550 50  0001 C CNN
+	1    12350 9550
+	1    0    0    -1
+$EndComp
+$Comp
+L power:PWR_FLAG #FLG0103
+U 1 1 5FF031D9
+P 12800 9550
+F 0 "#FLG0103" H 12800 9625 50  0001 C CNN
+F 1 "PWR_FLAG" H 12800 9723 50  0000 C CNN
+F 2 "" H 12800 9550 50  0001 C CNN
+F 3 "~" H 12800 9550 50  0001 C CNN
+	1    12800 9550
+	-1   0    0    1
+$EndComp
+$Comp
+L ETH3CDAQ1:+18V #PWR0138
+U 1 1 5FF03FA8
+P 12800 9550
+F 0 "#PWR0138" H 12800 9400 50  0001 C CNN
+F 1 "+18V" H 12815 9723 50  0000 C CNN
+F 2 "" H 12800 9550 50  0001 C CNN
+F 3 "" H 12800 9550 50  0001 C CNN
+	1    12800 9550
+	1    0    0    -1
+$EndComp
+$Comp
+L power:GND #PWR0139
+U 1 1 5FF07847
+P 13700 9550
+F 0 "#PWR0139" H 13700 9300 50  0001 C CNN
+F 1 "GND" H 13705 9377 50  0000 C CNN
+F 2 "" H 13700 9550 50  0001 C CNN
+F 3 "" H 13700 9550 50  0001 C CNN
+	1    13700 9550
+	1    0    0    -1
+$EndComp
+$Comp
+L power:PWR_FLAG #FLG0104
+U 1 1 5FF08AEB
+P 13700 9550
+F 0 "#FLG0104" H 13700 9625 50  0001 C CNN
+F 1 "PWR_FLAG" H 13700 9723 50  0000 C CNN
+F 2 "" H 13700 9550 50  0001 C CNN
+F 3 "~" H 13700 9550 50  0001 C CNN
+	1    13700 9550
+	1    0    0    -1
+$EndComp
+$Comp
+L ETH3CDAQ1:-18V #PWR0140
+U 1 1 5FF314D3
+P 13250 9550
+F 0 "#PWR0140" H 13250 9400 50  0001 C CNN
+F 1 "-18V" H 13265 9723 50  0000 C CNN
+F 2 "" H 13250 9550 50  0001 C CNN
+F 3 "" H 13250 9550 50  0001 C CNN
+	1    13250 9550
+	1    0    0    -1
+$EndComp
+$Comp
+L power:PWR_FLAG #FLG0105
+U 1 1 5FF484DD
+P 13250 9550
+F 0 "#FLG0105" H 13250 9625 50  0001 C CNN
+F 1 "PWR_FLAG" H 13250 9723 50  0000 C CNN
+F 2 "" H 13250 9550 50  0001 C CNN
+F 3 "~" H 13250 9550 50  0001 C CNN
+	1    13250 9550
+	-1   0    0    1
+$EndComp
 $EndSCHEMATC
