File: hardware/project/ETH3CADC1/FPGA1.sch (KiCad schematic (older format))
At the start: 25 parts, among them J1301 Conn_02x05_Odd_Even, U1301 ICE40UP5K-SG48ITR, U1302 W25Q32JVSS, U1303 AP2127K-1.2, X1301 ASAAIG-40.000MHZ

Commit message: PCB layout
Parts:
- added R1308: 10k, Resistor_SMD:R_0402_1005Metric_Pad0.72x0.64mm_HandSolder, symbol Device:R
- added R1309: NC, Resistor_SMD:R_0402_1005Metric_Pad0.72x0.64mm_HandSolder, symbol Device:R
Connections:
- net +3V3: now also R1308.1, R1309.1
- net FPGA1_UART6_TX: now reaches U1301.25 (IOT_36b)
- net FPGA1_UART6_RX: now reaches U1301.26 (IOT_39a)
- net CODE1: now reaches U1301.2 (IOB_6a)
- net CODE1: now also R1308.2
- net CODE2: now reaches U1301.3 (IOB_9b)
- net CODE2: now also R1309.2
- no-connect marks 24 -> 20
Other:
- moved on the sheet: C1309, C1312, D1301
Changed lines of the file:
@@
 L Device:D D1301
 U 1 1 606867C8
-P 9050 2700
-F 0 "D1301" H 9050 2483 50  0000 C CNN
-F 1 "CDBU0520" H 9050 2574 50  0000 C CNN
-F 2 "Diode_SMD:D_SOD-523" H 9050 2700 50  0001 C CNN
-F 3 "~" H 9050 2700 50  0001 C CNN
-	1    9050 2700
+P 8750 2700
+F 0 "D1301" H 8750 2483 50  0000 C CNN
+F 1 "CDBU0520" H 8750 2574 50  0000 C CNN
+F 2 "Diode_SMD:D_SOD-523" H 8750 2700 50  0001 C CNN
+F 3 "~" H 8750 2700 50  0001 C CNN
+	1    8750 2700
 	-1   0    0    1
 $EndComp
@@
 L Device:C C1309
 U 1 1 606870CE
-P 8650 2950
-F 0 "C1309" H 8765 2996 50  0000 L CNN
-F 1 "100n" H 8765 2905 50  0000 L CNN
-F 2 "Capacitor_SMD:C_0402_1005Metric_Pad0.74x0.62mm_HandSolder" H 8688 2800 50  0001 C CNN
-F 3 "~" H 8650 2950 50  0001 C CNN
-	1    8650 2950
+P 8350 2950
+F 0 "C1309" H 8465 2996 50  0000 L CNN
+F 1 "100n" H 8465 2905 50  0000 L CNN
+F 2 "Capacitor_SMD:C_0402_1005Metric_Pad0.74x0.62mm_HandSolder" H 8388 2800 50  0001 C CNN
+F 3 "~" H 8350 2950 50  0001 C CNN
+	1    8350 2950
 	1    0    0    -1
 $EndComp
@@
 L Device:C C1312
 U 1 1 60687838
-P 9350 2950
-F 0 "C1312" H 9465 2996 50  0000 L CNN
-F 1 "4u7" H 9465 2905 50  0000 L CNN
-F 2 "Capacitor_SMD:C_0603_1608Metric_Pad1.08x0.95mm_HandSolder" H 9388 2800 50  0001 C CNN
-F 3 "~" H 9350 2950 50  0001 C CNN
-	1    9350 2950
-	1    0    0    -1
-$EndComp
-Wire Wire Line
-	8650 2800 8650 2700
-Wire Wire Line
-	8650 2700 8900 2700
-Wire Wire Line
-	9350 2700 9350 2800
+P 9050 2950
+F 0 "C1312" H 9165 2996 50  0000 L CNN
+F 1 "4u7" H 9165 2905 50  0000 L CNN
+F 2 "Capacitor_SMD:C_0603_1608Metric_Pad1.08x0.95mm_HandSolder" H 9088 2800 50  0001 C CNN
+F 3 "~" H 9050 2950 50  0001 C CNN
+	1    9050 2950
+	1    0    0    -1
+$EndComp
+Wire Wire Line
+	8350 2800 8350 2700
+Wire Wire Line
+	8350 2700 8600 2700
+Wire Wire Line
+	9050 2700 9050 2800
 $Comp
 L power:GND #PWR01321
 U 1 1 6068A4C0
-P 9350 3100
-F 0 "#PWR01321" H 9350 2850 50  0001 C CNN
-F 1 "GND" H 9355 2927 50  0000 C CNN
-F 2 "" H 9350 3100 50  0001 C CNN
-F 3 "" H 9350 3100 50  0001 C CNN
-	1    9350 3100
+P 9050 3100
+F 0 "#PWR01321" H 9050 2850 50  0001 C CNN
+F 1 "GND" H 9055 2927 50  0000 C CNN
+F 2 "" H 9050 3100 50  0001 C CNN
+F 3 "" H 9050 3100 50  0001 C CNN
+	1    9050 3100
 	1    0    0    -1
 $EndComp
@@
 L power:GND #PWR01317
 U 1 1 6068A932
-P 8650 3100
-F 0 "#PWR01317" H 8650 2850 50  0001 C CNN
-F 1 "GND" H 8655 2927 50  0000 C CNN
-F 2 "" H 8650 3100 50  0001 C CNN
-F 3 "" H 8650 3100 50  0001 C CNN
-	1    8650 3100
+P 8350 3100
+F 0 "#PWR01317" H 8350 2850 50  0001 C CNN
+F 1 "GND" H 8355 2927 50  0000 C CNN
+F 2 "" H 8350 3100 50  0001 C CNN
+F 3 "" H 8350 3100 50  0001 C CNN
+	1    8350 3100
 	1    0    0    -1
 $EndComp
@@
 L power:+3.3V #PWR01316
 U 1 1 6068CFE8
-P 8650 2650
-F 0 "#PWR01316" H 8650 2500 50  0001 C CNN
-F 1 "+3.3V" H 8665 2823 50  0000 C CNN
-F 2 "" H 8650 2650 50  0001 C CNN
-F 3 "" H 8650 2650 50  0001 C CNN
-	1    8650 2650
-	1    0    0    -1
-$EndComp
-Wire Wire Line
-	8650 2650 8650 2700
-Connection ~ 8650 2700
+P 8350 2650
+F 0 "#PWR01316" H 8350 2500 50  0001 C CNN
+F 1 "+3.3V" H 8365 2823 50  0000 C CNN
+F 2 "" H 8350 2650 50  0001 C CNN
+F 3 "" H 8350 2650 50  0001 C CNN
+	1    8350 2650
+	1    0    0    -1
+$EndComp
+Wire Wire Line
+	8350 2650 8350 2700
+Connection ~ 8350 2700
 $Comp
 L Regulator_Linear:AP2127K-1.2 U1303
@@
 Wire Wire Line
 	9450 1900 9500 1900
-Connection ~ 9350 2700
-Wire Wire Line
-	9350 2700 9450 2700
-Wire Wire Line
-	9200 2700 9350 2700
+Connection ~ 9050 2700
+Wire Wire Line
+	8900 2700 9050 2700
 $Comp
 L power:+3.3V #PWR01305
@@
 Text HLabel 3150 2200 0    50   BiDi ~ 0
 FGPA1_SCLK
-NoConn ~ 5000 3000
 $Comp
 L ETH3CDAQ1:ASAAIG-xxx X1301
@@
 Wire Wire Line
 	1250 6950 1700 6950
-NoConn ~ 5000 2800
 NoConn ~ 5000 2900
 Text HLabel 1550 2800 0    50   Output ~ 0
@@
 Wire Wire Line
 	9500 2700 9450 2700
-Connection ~ 9450 2700
 Connection ~ 9050 1150
 Wire Wire Line
@@
 NoConn ~ 1600 2100
 NoConn ~ 1600 2000
-NoConn ~ 1600 1700
 NoConn ~ 1600 1800
-NoConn ~ 1600 1400
 NoConn ~ 1600 1600
 NoConn ~ 1600 1900
@@
 	4950 2400 5000 2400
 NoConn ~ 1600 2400
+Text Label 4750 2800 0    50   ~ 0
+CODE1
+Wire Wire Line
+	4750 2800 5000 2800
+Text Label 4750 3000 0    50   ~ 0
+CODE2
+Wire Wire Line
+	4750 3000 5000 3000
+Text Label 3500 6850 0    50   ~ 0
+CODE1
+Text Label 3500 6950 0    50   ~ 0
+CODE2
+$Comp
+L Device:R R1308
+U 1 1 60071695
+P 3850 6650
+F 0 "R1308" H 3920 6696 50  0000 L CNN
+F 1 "10k" H 3920 6605 50  0000 L CNN
+F 2 "Resistor_SMD:R_0402_1005Metric_Pad0.72x0.64mm_HandSolder" V 3780 6650 50  0001 C CNN
+F 3 "~" H 3850 6650 50  0001 C CNN
+	1    3850 6650
+	1    0    0    -1
+$EndComp
+$Comp
+L Device:R R1309
+U 1 1 60074053
+P 4250 6650
+F 0 "R1309" H 4320 6696 50  0000 L CNN
+F 1 "NC" H 4320 6605 50  0000 L CNN
+F 2 "Resistor_SMD:R_0402_1005Metric_Pad0.72x0.64mm_HandSolder" V 4180 6650 50  0001 C CNN
+F 3 "~" H 4250 6650 50  0001 C CNN
+	1    4250 6650
+	1    0    0    -1
+$EndComp
+Wire Wire Line
+	3850 6850 3850 6800
+Wire Wire Line
+	3500 6850 3850 6850
+Wire Wire Line
+	4250 6950 4250 6800
+Wire Wire Line
+	3500 6950 4250 6950
+Wire Wire Line
+	3850 6500 3850 6450
+Wire Wire Line
+	3850 6450 4050 6450
+Wire Wire Line
+	4250 6450 4250 6500
+$Comp
+L power:+3.3V #PWR01323
+U 1 1 6008422B
+P 4050 6400
+F 0 "#PWR01323" H 4050 6250 50  0001 C CNN
+F 1 "+3.3V" H 4065 6573 50  0000 C CNN
+F 2 "" H 4050 6400 50  0001 C CNN
+F 3 "" H 4050 6400 50  0001 C CNN
+	1    4050 6400
+	1    0    0    -1
+$EndComp
+Wire Wire Line
+	4050 6400 4050 6450
+Connection ~ 4050 6450
+Wire Wire Line
+	4050 6450 4250 6450
+Wire Wire Line
+	9050 2700 9450 2700
+Connection ~ 9450 2700
+Text HLabel 1550 1400 0    50   BiDi ~ 0
+FPGA1_UART6_TX
+Text HLabel 1550 1700 0    50   BiDi ~ 0
+FPGA1_UART6_RX
+Wire Wire Line
+	1600 1700 1550 1700
+Wire Wire Line
+	1600 1400 1550 1400
 $EndSCHEMATC
