File: hardware/project/ETH3CADC1/ETH3CADC1.kicad_pcb (KiCad board)
At the start: 2 copper layers, 73 x 100 mm, 327 parts, among them J1001 Conn_02x10_Odd_Even, J1101 Conn_02x10_Odd_Even, J1201 Conn_02x10_Odd_Even, J1301 Conn_02x02_Odd_Even, J1302 Conn_02x04_Odd_Even, J501 20021111-00010T4LF, J502 Conn_02x01, Q301 MMBTA55, Q302 BC847, U201 DG211B, U202 OPA2192, U203 DG419xY, U204 LT5400-100k-100k, U205 LT5400-5k-1k, U206 OPA177, U207 OPA140, U208 OPA192, U209 LT5400-10k-10k, U210 LM311, U301 LT1021-7, U302 LM399H, U401 DG211B, U402 OPA2192, U403 DG419xY, U404 LT5400-100k-100k, U405 LT5400-5k-1k, U406 OPA177, U407 OPA140, U408 OPA192, U409 LT5400-10k-10k, U410 LM311, U501 SN74LVC1T45DBV, U502 SN74LVC1T45DBV, U503 SN74LVC1T45DBV, U504 HDC1080, U505 MCP2551-I-SN, U506 STM32H743ZI, U507 PCA9517, U508 24LC08B-E/MS, U601 LAN8742A, U602 LC03-3.3, U603 LC03-3.3, U701 TXB0104PW, U702 ADuM5402, U703 74AC125, U801 DG211B, U802 OPA2192, U803 DG419xY, U804 LT5400-100k-100k, U805 LT5400-5k-1k, U806 OPA177, U807 OPA140, U808 OPA192, U809 LT5400-10k-10k, U810 LM311, U901 AP2127K-1.2, U902 SN74LVC1T45DBV, U903 SN74LVC1T45DBV, U904 ICE40UP5K-SG48ITR, U905 SN74LVC1T45DBV, U906 SN74LVC1T45DBV, U907 SN74LVC1T45DBV, U908 SN74LVC1T45DBV, U909 W25Q32JVSS, Y501 NX3225GD-8MHZ, Y601 NX5032GA-25.000M-LN-CD-1

Commit message: PCB layout
Parts:
- removed R903, R904, R905, R906, R907: 150, Resistor_SMD:R_0402_1005Metric_Pad0.72x0.64mm_HandSolder
- added C1401: 100n, Capacitor_SMD:C_0402_1005Metric_Pad0.74x0.62mm_HandSolder, B.Cu at (192.5, 75.2)
- added C1402: 100n, Capacitor_SMD:C_0402_1005Metric_Pad0.74x0.62mm_HandSolder, B.Cu at (190.6, 59.1)
- added C1403: 100n, Capacitor_SMD:C_0402_1005Metric_Pad0.74x0.62mm_HandSolder, B.Cu at (188.7, 59.1)
- added C1404: 100n, Capacitor_SMD:C_0402_1005Metric_Pad0.74x0.62mm_HandSolder, B.Cu at (209.6, 59.1)
- added C1405: 100n, Capacitor_SMD:C_0402_1005Metric_Pad0.74x0.62mm_HandSolder, B.Cu at (195.3, 59.1)
- added C1406: 100n, Capacitor_SMD:C_0402_1005Metric_Pad0.74x0.62mm_HandSolder, B.Cu at (199.3, 59.1)
- added C1407: 100n, Capacitor_SMD:C_0402_1005Metric_Pad0.74x0.62mm_HandSolder, B.Cu at (197.4, 75.2)
- added C1501: 10u/50V, Capacitor_SMD:C_0805_2012Metric_Pad1.18x1.45mm_HandSolder, F.Cu at (220.1, 127.4)
- added C1502: 4u7/50V, Capacitor_SMD:C_0805_2012Metric_Pad1.18x1.45mm_HandSolder, F.Cu at (220.1, 130.3)
- added C1503: 4u7/50V, Capacitor_SMD:C_0805_2012Metric_Pad1.18x1.45mm_HandSolder, F.Cu at (220.1, 134.2)
- added C302: 100n, Capacitor_SMD:C_0402_1005Metric_Pad0.74x0.62mm_HandSolder, B.Cu at (191.0, 132.3)
- added R1501: 1k23, Resistor_SMD:R_0402_1005Metric_Pad0.72x0.64mm_HandSolder, B.Cu at (213.9, 131.1)
- added R1502: 120, Resistor_SMD:R_0402_1005Metric_Pad0.72x0.64mm_HandSolder, B.Cu at (212.0, 131.1)
- added R201: 10M, Resistor_SMD:R_0603_1608Metric_Pad0.98x0.95mm_HandSolder, B.Cu at (160.8, 56.8)
- added R214: 10k, Resistor_SMD:R_0402_1005Metric_Pad0.72x0.64mm_HandSolder, B.Cu at (158.0, 64.9)
- added R215: 10k, Resistor_SMD:R_0402_1005Metric_Pad0.72x0.64mm_HandSolder, B.Cu at (163.7, 64.3)
- added R216: 10k, Resistor_SMD:R_0402_1005Metric_Pad0.72x0.64mm_HandSolder, F.Cu at (125.3, 36.2)
- added R310: 6k95/.05%, Resistor_SMD:R_0603_1608Metric_Pad0.98x0.95mm_HandSolder, B.Cu at (194.4, 127.8)
- added R311: 3k01/.1%, Resistor_SMD:R_0603_1608Metric_Pad0.98x0.95mm_HandSolder, B.Cu at (194.4, 132.5)
- added R312: 3k01/.1%, Resistor_SMD:R_0603_1608Metric_Pad0.98x0.95mm_HandSolder, B.Cu at (194.4, 130.0)
- added R313: 0, Resistor_SMD:R_0603_1608Metric_Pad0.98x0.95mm_HandSolder, F.Cu at (194.4, 127.5)
- added U1401: MT48LC16M16A2P-6A, ETH3CDAQ1:TSSOP-54, B.Cu at (199.3, 67.2)
- added U1501: LM337_SOT223, Package_TO_SOT_SMD:SOT-223-3_TabPin2, F.Cu at (214.4, 130.8)
- added U201: DG211, Package_SO:TSSOP-16_4.4x5mm_P0.65mm, F.Cu at (160.8, 62.6)
- added U205: OPA140, Package_SO:SOIC-8_3.9x4.9mm_P1.27mm, F.Cu at (160.8, 56.1)
- added U303: OPA177, Package_SO:SOIC-8_3.9x4.9mm_P1.27mm, F.Cu at (194.4, 131.1)
- C205, C501, C502, C503, C504, C505, C506, C508, C509, C510, C511, C512, C513, C515, C516, C524, C525, C526, C528, C529, C530, C601, C602, C604, C605, C608, C609, C610, C611, C612, C613, C614, C701, C703, C704, C706, C708, C902, C904, C905, C907, C908, C910, C911, C913, C914, C916, C917, C919, C920, C921, C922, C923, D202, D301, D901, R305, R502, R504, R507, R508, R509, R510, R511, R512, R513, R606, R607, R608, R609, R611, R612, R613, R614, R615, R616, R617, R618, R619, R701, R901, R902, R908, R909, R911, R912, Y501: moved to B.Cu
- C210: renamed from C207; moved to B.Cu
- C221: renamed from C220; moved to B.Cu
- C514, C607: footprint Capacitor_SMD:C_0603_1608Metric_Pad1.08x0.95mm_HandSolder -> Capacitor_SMD:C_0402_1005Metric_Pad0.74x0.62mm_HandSolder
- C518, C519, C521, C606, C702, C705, C707: footprint Capacitor_SMD:C_0603_1608Metric_Pad1.08x0.95mm_HandSolder -> Capacitor_SMD:C_0402_1005Metric_Pad0.74x0.62mm_HandSolder; moved to B.Cu
- C709: footprint Capacitor_SMD:C_0402_1005Metric_Pad0.74x0.62mm_HandSolder -> Capacitor_SMD:C_0603_1608Metric_Pad1.08x0.95mm_HandSolder
- R202: renamed from R201; moved to B.Cu
- R203: renamed from R202; moved to B.Cu
- R204: renamed from R203; moved to B.Cu
- R205: renamed from R204; moved to B.Cu
- R206: renamed from R205; moved to B.Cu
- R207: renamed from R206; moved to B.Cu
- R208: renamed from R207; moved to B.Cu
- R209: renamed from R208; moved to B.Cu
- R210: renamed from R209; moved to B.Cu
- R211: renamed from R210; moved to B.Cu
- R212: renamed from R211; moved to B.Cu
- R213: renamed from R212; moved to B.Cu
- R620, R621, R702, R703, R704, R705, R706: footprint Resistor_SMD:R_0402_1005Metric_Pad0.72x0.64mm_HandSolder -> Resistor_SMD:R_0603_1608Metric_Pad0.98x0.95mm_HandSolder; moved to B.Cu
- U207: renamed from U205; moved to B.Cu
- U208: renamed from U206; moved to B.Cu
- moved Q302 250.4 mm to (201.2, 130.2), turned to 90 degrees
- moved U302 247.3 mm to (193.0, 142.0), turned to 180 degrees
- moved U301 247.0 mm to (206.0, 142.0), turned to 90 degrees
- moved Q301 236.6 mm to (210.6, 142.0), turned to 90 degrees
- moved D302 235.8 mm to (206.6, 129.7)
- moved D301 229.9 mm to (206.0, 144.0)
- moved C602 208.2 mm to (191.5, 90.9), turned to 90 degrees
- moved R615 203.4 mm to (203.1, 94.5), turned to 90 degrees
- moved R617 199.5 mm to (196.7, 94.5), turned to 90 degrees
- moved C609 198.4 mm to (193.3, 91.8), turned to 180 degrees
- moved R621 198.1 mm to (201.8, 104.8), turned to 270 degrees
- moved R606 198.0 mm to (198.6, 83.3), turned to 270 degrees
- moved R611 196.6 mm to (205.5, 92.8)
- moved R603 196.1 mm to (196.8, 83.3), turned to 90 degrees
- moved R609 196.0 mm to (193.3, 86.2)
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- renumbered C208 to C207, C209 to C208, C210 to C209, C214 to C213, C216 to C214, C217 to C215, C213 to C216, C215 to C217, C221 to C220, U201 to U202, U202 to U203, U203 to U204, U204 to U206, U207 to U209, U208 to U210, U209 to U211, U210 to U212
Connections:
- net /VREF/VREF_N7V renamed Net-(R307-Pad1)
- C501 pad 2: GND -> AGNDF
- C502 pad 2: GND -> AGNDF
- C503 pad 2: GND -> AGNDF
- C504 pad 2: GND -> AGNDF
- C505 pad 2: GND -> AGNDF
- C506 pad 2: GND -> AGNDF
- C507 pad 2: GND -> AGNDF
- C508 pad 2: GND -> AGNDF
- C509 pad 2: GND -> AGNDF
- C510 pad 2: GND -> AGNDF
- C511 pad 2: GND -> AGNDF
- C512 pad 2: GND -> AGNDF
- C513 pad 2: GND -> AGNDF
- C514 pad 2: GND -> AGNDF
- C515 pad 2: GND -> AGNDF
- C516 pad 2: GND -> AGNDF
- C517 pad 2: GND -> AGNDF
- C518 pad 2: GND -> AGNDF
- C519 pad 2: GND -> AGNDF
- C520 pad 2: GND -> AGNDF
- C521 pad 2: GND -> AGNDF
- C522 pad 2: GND -> AGNDF
- C523 pad 2: GND -> AGNDF
- C524 pad 2: GND -> AGNDF
- C525 pad 2: GND -> AGNDF
- C526 pad 2: GND -> AGNDF
- C527 pad 2: GND -> AGNDF
- C528 pad 2: GND -> AGNDF
- C529 pad 2: GND -> AGNDF
- C530 pad 1: /MCU/NRST -> /Ethernet/NRST
- C530 pad 2: GND -> AGNDF
- C601 pad 2: GND -> AGNDF
- C602 pad 2: GND -> AGNDF
- C603 pad 2: GND -> AGNDF
- C604 pad 2: GND -> AGNDF
- C605 pad 2: GND -> AGNDF
- C606 pad 2: GND -> AGNDF
- C607 pad 2: GND -> AGNDF
- C608 pad 2: GND -> AGNDF
- C609 pad 2: GND -> AGNDF
- C610 pad 2: GND -> AGNDF
- C611 pad 2: GND -> AGNDF
- C612 pad 2: GND -> AGNDF
- C613 pad 2: GND -> AGNDF
- C701 pad 2: GND -> AGNDF
- C702 pad 2: GND -> AGNDF
- C703 pad 2: GND -> AGNDF
- C704 pad 2: GND -> AGNDF
- C705 pad 2: GND -> AGNDF
- C709 pad 1: /Trigger/EXT_TRIG -> /Connector/EXT_TRIG
- C901 pad 2: GND -> AGNDF
- C902 pad 2: GND -> AGNDF
- C903 pad 2: GND -> AGNDF
- C904 pad 2: GND -> AGNDF
- C905 pad 2: GND -> AGNDF
- C906 pad 2: GND -> AGNDF
- C907 pad 2: GND -> AGNDF
- C908 pad 2: GND -> AGNDF
- C909 pad 2: GND -> AGNDF
- C910 pad 2: GND -> AGNDF
- C911 pad 2: GND -> AGNDF
- C912 pad 2: GND -> AGNDF
- C913 pad 2: GND -> AGNDF
- C914 pad 2: GND -> AGNDF
- C915 pad 2: GND -> AGNDF
- C916 pad 2: GND -> AGNDF
- C917 pad 2: GND -> AGNDF
- C918 pad 2: GND -> AGNDF
- C919 pad 2: GND -> AGNDF
- C920 pad 2: GND -> AGNDF
- C921 pad 2: GND -> AGNDF
- C922 pad 2: GND -> AGNDF
- C923 pad 2: GND -> AGNDF
- D703 pad 1: /Trigger/EXT_TRIG -> /Connector/EXT_TRIG
- J1001 pad 1: (no net) -> AGNDF
- J1001 pad 10: (no net) -> /ADC 1/ADIN1
- J1001 pad 11: (no net) -> /ADC 1/ADIN1
- J1001 pad 12: (no net) -> /ADC 1/ADIN1
- J1001 pad 13: (no net) -> AGNDF
- J1001 pad 14: (no net) -> AGNDF
- J1001 pad 15: (no net) -> +3V3
- J1001 pad 16: (no net) -> +3V3
- J1001 pad 18: (no net) -> +5V
- J1001 pad 19: (no net) -> -18VF
- J1001 pad 20: (no net) -> +18VF
- J1001 pad 3: (no net) -> AGNDF
- J1001 pad 7: (no net) -> AGNDF
- J1001 pad 8: (no net) -> AGNDF
- J1001 pad 9: (no net) -> /ADC 1/ADIN1
- J1301 pad 1: (no net) -> /Connector/EXT_TRIG
- J1301 pad 2: (no net) -> /Connector/EXT_TRIG
- J1301 pad 3: (no net) -> GND_TRIG
- J1301 pad 4: (no net) -> GND_TRIG
- J1302 pad 1: (no net) -> Earth
- J1302 pad 2: (no net) -> Earth
- J1302 pad 3: (no net) -> /Connector/RX+
- J1302 pad 4: (no net) -> /Connector/TX+
- J1302 pad 5: (no net) -> /Connector/RX-
- J1302 pad 6: (no net) -> /Connector/TX-
- J1302 pad 7: (no net) -> Earth
- J1302 pad 8: (no net) -> Earth
- J501 pad 10: /MCU/NRST -> /Ethernet/NRST
- J501 pad 3: GND -> AGNDF
- J501 pad 5: GND -> AGNDF
- J502 pad 2: GND -> AGNDF
- L701 pad 1: /Trigger/EXT_TRIG -> /Connector/EXT_TRIG
- R503 pad 2: GND -> AGNDF
- R509 pad 2: GND -> AGNDF
- R513 pad 2: /MCU/NRST -> /Ethernet/NRST
- R601 pad 2: (no net) -> /Ethernet/RMII_RXD0
- R602 pad 2: (no net) -> /Ethernet/RMII_RXD1
- R603 pad 2: GND -> AGNDF
- R604 pad 2: (no net) -> /Ethernet/RMII_CRS_DV
- R605 pad 2: (no net) -> /Ethernet/REF_CLK
- R611 pad 2: GND -> AGNDF
- R612 pad 1: GND -> AGNDF
- R613 pad 2: GND -> AGNDF
- R614 pad 2: GND -> AGNDF
- R619 pad 2: GND -> AGNDF
- U206 pad 8: (no net) -> Net-(U205-Pad2)
- U302 pad 4: (no net) -> -18VF
- U501 pad 2: GND -> AGNDF
- U501 pad 5: GND -> AGNDF
- U502 pad 2: GND -> AGNDF
- U502 pad 5: GND -> AGNDF
- U503 pad 2: GND -> AGNDF
- U503 pad 5: GND -> AGNDF
- U504 pad 2: GND -> AGNDF
- U505 pad 2: GND -> AGNDF
- U506 pad 10: (no net) -> /MCU/A0
- U506 pad 107: GND -> AGNDF
- U506 pad 11: (no net) -> /MCU/A1
- U506 pad 114: (no net) -> /MCU/D2
- U506 pad 115: (no net) -> /MCU/D3
- U506 pad 12: (no net) -> /MCU/A2
- U506 pad 120: GND -> AGNDF
- U506 pad 126: (no net) -> /Ethernet/RMII_TXEN
- U506 pad 128: (no net) -> /Ethernet/RMII_TXD0
- U506 pad 129: (no net) -> /Ethernet/RMII_TXD1
- U506 pad 13: (no net) -> /MCU/A3
- U506 pad 130: GND -> AGNDF
- U506 pad 132: (no net) -> /MCU/~CAS
- U506 pad 135: (no net) -> /MCU/CKE
- U506 pad 136: (no net) -> /MCU/~CS
- U506 pad 14: (no net) -> /MCU/A4
- U506 pad 141: (no net) -> /MCU/LDQM
- U506 pad 142: (no net) -> /MCU/UDQM
- U506 pad 15: (no net) -> /MCU/A5
- U506 pad 16: GND -> AGNDF
- U506 pad 25: /MCU/NRST -> /Ethernet/NRST
- U506 pad 26: (no net) -> /MCU/~WE
- U506 pad 27: (no net) -> /Ethernet/RMII_MDC
- U506 pad 31: GND -> AGNDF
- U506 pad 35: (no net) -> /Ethernet/REF_CLK
- U506 pad 36: (no net) -> /Ethernet/RMII_MDIO
- U506 pad 38: GND -> AGNDF
- U506 pad 40: (no net) -> /MCU/TRIG_EN
- U506 pad 41: (no net) -> /MCU/TRIG_OUT
- U506 pad 42: (no net) -> /MCU/TRIG_IN
- U506 pad 43: (no net) -> /Ethernet/RMII_CRS_DV
- U506 pad 44: (no net) -> /Ethernet/RMII_RXD0
- U506 pad 45: (no net) -> /Ethernet/RMII_RXD1
- U506 pad 49: (no net) -> /MCU/~RAS
- U506 pad 50: (no net) -> /MCU/A6
- U506 pad 51: GND -> AGNDF
- U506 pad 53: (no net) -> /MCU/A7
- U506 pad 54: (no net) -> /MCU/A8
- U506 pad 55: (no net) -> /MCU/A9
- U506 pad 56: (no net) -> /MCU/A10
- U506 pad 57: (no net) -> /MCU/A11
- U506 pad 58: (no net) -> /MCU/D4
- U506 pad 59: (no net) -> /MCU/D5
- U506 pad 60: (no net) -> /MCU/D6
- U506 pad 61: GND -> AGNDF
- U506 pad 63: (no net) -> /MCU/D7
- U506 pad 64: (no net) -> /MCU/D8
- U506 pad 65: (no net) -> /MCU/D9
- U506 pad 66: (no net) -> /MCU/D10
- U506 pad 67: (no net) -> /MCU/D11
- U506 pad 68: (no net) -> /MCU/D12
- U506 pad 77: (no net) -> /MCU/D13
- U506 pad 78: (no net) -> /MCU/D14
- U506 pad 79: (no net) -> /MCU/D15
- U506 pad 83: GND -> AGNDF
- U506 pad 85: (no net) -> /MCU/D0
- U506 pad 86: (no net) -> /MCU/D1
- U506 pad 87: (no net) -> /MCU/A12
- U506 pad 89: (no net) -> /MCU/BA0
- U506 pad 90: (no net) -> /MCU/BA1
- U506 pad 93: (no net) -> /MCU/CLK
- U506 pad 94: GND -> AGNDF
- U507 pad 4: GND -> AGNDF
- U508 pad 1: GND -> AGNDF
- U508 pad 2: GND -> AGNDF
- U508 pad 3: GND -> AGNDF
- U508 pad 4: GND -> AGNDF
- U601 pad 13: (no net) -> /Ethernet/RMII_MDC
- U601 pad 15: (no net) -> /Ethernet/NRST
- U601 pad 16: (no net) -> /Ethernet/RMII_TXEN
- U601 pad 17: (no net) -> /Ethernet/RMII_TXD0
- U601 pad 18: (no net) -> /Ethernet/RMII_TXD1
- U601 pad 25: GND -> AGNDF
- U602 pad 5: (no net) -> /Connector/TX-
- U602 pad 8: (no net) -> /Connector/TX+
- U603 pad 5: (no net) -> /Connector/RX-
- U603 pad 8: (no net) -> /Connector/RX+
- U701 pad 2: (no net) -> /MCU/TRIG_EN
- U701 pad 3: (no net) -> /MCU/TRIG_OUT
- U701 pad 4: (no net) -> /MCU/TRIG_IN
- U701 pad 7: GND -> AGNDF
- U702 pad 2: GND -> AGNDF
- U702 pad 8: GND -> AGNDF
- U901 pad 2: GND -> AGNDF
- U902 pad 2: GND -> AGNDF
- U902 pad 4: /FPGA 1/AD_IIN -> (no net)
- U902 pad 5: GND -> AGNDF
- U903 pad 2: GND -> AGNDF
- U903 pad 4: /FPGA 1/AD_IRN -> (no net)
- U903 pad 5: GND -> AGNDF
- U904 pad 49: GND -> AGNDF
- U905 pad 2: GND -> AGNDF
- U905 pad 4: /FPGA 1/AD_ID -> (no net)
- U905 pad 5: GND -> AGNDF
- U906 pad 2: GND -> AGNDF
- U906 pad 4: /FPGA 1/AD_IRP -> (no net)
- U906 pad 5: GND -> AGNDF
- U907 pad 2: GND -> AGNDF
- U907 pad 4: /FPGA 1/AD_VRH -> (no net)
- U907 pad 5: GND -> AGNDF
- U908 pad 2: GND -> AGNDF
- U909 pad 4: GND -> AGNDF
Other:
- board size 73 x 100 mm -> 72.5 x 100 mm

Commit message: PCB modifications
Parts:
- removed C217: DNP, Capacitor_SMD:C_0402_1005Metric_Pad0.74x0.62mm_HandSolder
- C202, C204, C216, C514, C520, C901, R216, R501, R503, R505, R506, R514: moved to B.Cu
- FB501: footprint Inductor_SMD:L_0805_2012Metric_Pad1.15x1.40mm_HandSolder -> Inductor_SMD:L_0603_1608Metric_Pad1.05x0.95mm_HandSolder; moved to B.Cu
- FB601: footprint Inductor_SMD:L_0805_2012Metric_Pad1.15x1.40mm_HandSolder -> Inductor_SMD:L_0603_1608Metric_Pad1.05x0.95mm_HandSolder
- moved R501 93.8 mm to (187.2, 87.0), turned to 180 degrees
- moved C520 70.8 mm to (187.2, 82.4)
- moved C207 65.4 mm to (136.8, 57.7)
- moved C215 65.4 mm to (136.8, 61.6)
- moved C203 65.4 mm to (140.0, 57.7)
- moved C206 65.4 mm to (140.0, 55.7)
- moved C212 65.4 mm to (133.6, 57.7)
- moved C214 65.4 mm to (140.0, 61.6)
- moved C218 65.4 mm to (143.2, 59.6)
- moved C219 65.4 mm to (146.4, 57.7)
- moved C220 65.4 mm to (146.4, 59.6)
- moved R503 60.4 mm to (189.1, 85.0), turned to 90 degrees
- moved C216 53.5 mm to (163.2, 78.7)
- moved C211 52.3 mm to (169.0, 73.0), turned to 0 degrees
- moved C202 51.4 mm to (164.7, 69.2), turned to 270 degrees
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Connections:
- U210 pad 1: Net-(C217-Pad1) -> (no net)
- U210 pad 8: Net-(C217-Pad2) -> (no net)

Commit message: PCB modifications
Parts:
- removed the C517 at (257.2, 57.4)
- removed the C520 at (187.2, 82.4)
- removed the C522 at (257.2, 52.8)
- removed the C523 at (257.2, 55.1)
- removed C527, C528: 100n, Capacitor_SMD:C_0402_1005Metric_Pad0.74x0.62mm_HandSolder
- removed the U501 at (252.5, 51.7)
- removed the U502 at (258.4, 46.9)
- removed the U503 at (247.9, 58.0)
- C203, C206, C207, C212, C214, C507: moved to B.Cu
- C216: renamed from C215; moved to B.Cu
- C217: renamed from C218; moved to B.Cu
- C218: renamed from C219; moved to B.Cu
- C219: renamed from C220; moved to B.Cu
- moved C507 48.8 mm to (208.5, 54.4), turned to 90 degrees
- moved C212 38.2 mm to (171.7, 60.7), turned to 270 degrees
- moved C216 36.8 mm to (173.4, 57.5), turned to 90 degrees
- moved C206 36.4 mm to (172.1, 72.9), turned to 270 degrees
- moved C214 33.9 mm to (173.4, 55.2), turned to 270 degrees
- moved C207 27.3 mm to (164.0, 60.8), turned to 90 degrees
- moved C219 26.9 mm to (169.2, 73.9), turned to 180 degrees
- moved C217 25.9 mm to (166.2, 71.5), turned to 90 degrees
- moved C203 23.8 mm to (163.6, 54.2), turned to 90 degrees
- moved C218 15.7 mm to (161.0, 63.4), turned to 180 degrees
- moved C202 12.8 mm to (163.6, 56.5)
- moved U207 12.7 mm to (169.2, 67.2), turned to 180 degrees
- moved U211 12.7 mm to (169.2, 67.2), turned to 0 degrees
- moved U204 10.8 mm to (169.0, 55.5)
- moved U208 10.8 mm to (169.0, 55.5)
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- renumbered C210 to C209, C209 to C210, C216 to C215, C221 to C220, C524 to C517, C521 to C520, C525 to C521, C526 to C522, C529 to C523, C530 to C524, R214 to R201, R215 to R202, R216 to R203, R201 to R204, R202 to R205, R203 to R206, R204 to R207, R205 to R208, R206 to R209, R207 to R210, R208 to R211, R209 to R212, R210 to R213, R211 to R214, R212 to R215, R213 to R216, R908 to R903, R909 to R904, R910 to R905, R911 to R906, R912 to R907, U504 to U501, U505 to U502, U506 to U503, U507 to U504, U508 to U505
Connections:
- U503 pad 1: /MCU/MCU_SR_DAT -> (no net)
- U503 pad 2: /MCU/MCU_SR_LAT -> (no net)
- U503 pad 3: /MCU/MCU_SR_CLK -> (no net)
Other:
- net class Default: clearance 0.2 -> 0.127; trace_width 0.25 -> 0.127; via_dia 0.8 -> 0.5; via_drill 0.4 -> 0.2
- rule trace_clearance: 0.2 -> 0.127
- rule trace_min: 0.2 -> 0.127
- rule via_min_drill: 0.3 -> 0.2
- rule via_min_size: 0.4 -> 0.5

Commit message: SDRAM works, thanks to the website https://medium.com/@pjinwoo123/stm32h7-external-sdram-evaluation-board-cc72444898d8 . Modified the code to work with SDRAM BANK2. SCPI library works.
Parts:
- removed the C401 at (200.2, 30.7)
- removed the C402 at (197.0, 32.6)
- removed the C403 at (203.4, 26.7)
- removed the C404 at (200.2, 28.7)
- removed the C405 at (197.0, 30.7)
- removed the C406 at (200.2, 26.7)
- removed the C407 at (197.0, 28.7)
- removed the C408 at (282.7, -13.3)
- removed the C409 at (197.0, 26.7)
- removed the C410 at (206.6, 26.7)
- removed the C411 at (203.4, 28.7)
- removed the C412 at (200.2, 32.6)
- removed the C413 at (183.1, 8.00)
- removed the C414 at (203.4, 30.7)
- removed the C415 at (179.9, 8.00)
- removed the C416 at (206.6, 28.7)
- removed the C417 at (209.8, 26.7)
- removed the C418 at (203.4, 32.6)
- removed the C419 at (206.6, 30.7)
- removed the C420 at (209.8, 28.7)
- removed the C421 at (206.6, 32.6)
- removed C801, C802, C803, C804, C805, C806, C807, C809, C810, C811, C812, C814, C816, C817, C818, C819, C820, C821, C908, C910, C911, C913, C914, C916, C917, C919, C920, C921, C922, C923: 100n, Capacitor_SMD:C_0402_1005Metric_Pad0.74x0.62mm_HandSolder
- removed C808: 2n2/SMD, Capacitor_SMD:C_0603_1608Metric_Pad1.08x0.95mm_HandSolder
- removed C813: 33p, Capacitor_SMD:C_0402_1005Metric_Pad0.74x0.62mm_HandSolder
- removed C815: DNP, Capacitor_SMD:C_0402_1005Metric_Pad0.74x0.62mm_HandSolder
- removed the D401 at (328.3, 16.2)
- removed the D402 at (318.7, 24.6)
- removed D801, D802: BAV21W, Diode_SMD:D_SOD-123
- removed the R401 at (193.5, 3.25)
- removed the R402 at (189.2, 5.76)
- removed the R403 at (193.5, 0.74)
- removed the R404 at (189.2, 3.25)
- removed the R405 at (184.8, 5.76)
- removed the R406 at (193.5, 5.76)
- removed the R407 at (180.5, 0.74)
- removed the R408 at (184.8, 0.74)
- removed the R409 at (180.5, 3.25)
- removed the R410 at (180.5, 5.76)
- removed the R411 at (184.8, 3.25)
- removed the R412 at (189.2, 0.74)
- removed R801, R802, R804, R805, R809: 10, Resistor_SMD:R_0402_1005Metric_Pad0.72x0.64mm_HandSolder
- removed R803: 12k/.05%, Resistor_SMD:R_0603_1608Metric_Pad0.98x0.95mm_HandSolder
- removed R806: 62k, Resistor_SMD:R_0402_1005Metric_Pad0.72x0.64mm_HandSolder
- removed R807: 620/.05%, Resistor_SMD:R_0603_1608Metric_Pad0.98x0.95mm_HandSolder
- removed R808, R812: 3k9/.05%, Resistor_SMD:R_0603_1608Metric_Pad0.98x0.95mm_HandSolder
- removed R810: 62/.1%, Resistor_SMD:R_0603_1608Metric_Pad0.98x0.95mm_HandSolder
- removed R811: 39k/.05%, Resistor_SMD:R_0603_1608Metric_Pad0.98x0.95mm_HandSolder
- removed R902: 1k, Resistor_SMD:R_0402_1005Metric_Pad0.72x0.64mm_HandSolder
- removed the U401 at (304.3, 9.28)
- removed the U402 at (312.8, 19.7)
- removed the U403 at (329.7, 6.78)
- removed the U404 at (329.1, 12.3)
- removed the U405 at (337.6, 5.83)
- removed U406, U806: OPA177, Package_SO:SOIC-8_3.9x4.9mm_P1.27mm
- removed U407, U807: OPA140, Package_SO:SOIC-8_3.9x4.9mm_P1.27mm
- removed U408, U808: OPA192, Package_SO:SOIC-8_3.9x4.9mm_P1.27mm
- removed U409, U809: LT5400-10k-10k, Package_SO:MSOP-8-1EP_3x3mm_P0.65mm_EP1.73x1.85mm_ThermalVias
- removed U410, U810: LM311, Package_SO:SOIC-8_3.9x4.9mm_P1.27mm
- removed U801: DG211B, Package_SO:TSSOP-16_4.4x5mm_P0.65mm
- removed U802: OPA2192, Package_SO:SOIC-8_3.9x4.9mm_P1.27mm
- removed U803: DG419xY, Package_SO:SOIC-8_3.9x4.9mm_P1.27mm
- removed U804: LT5400-100k-100k, Package_SO:MSOP-8-1EP_3x3mm_P0.65mm_EP1.73x1.85mm_ThermalVias
- removed U805: LT5400-5k-1k, Package_SO:MSOP-8-1EP_3x3mm_P0.65mm_EP1.73x1.85mm_ThermalVias
- removed U902, U903, U905, U906, U907, U908: SN74LVC1T45DBV, Package_TO_SOT_SMD:SOT-23-6
- added C1312: 100n, Capacitor_SMD:C_0402_1005Metric_Pad0.74x0.62mm_HandSolder, B.Cu at (174.9, 56.6)
- added J1301: Conn_02x05_Odd_Even, Connector_PinHeader_1.27mm:PinHeader_2x05_P1.27mm_Vertical, F.Cu at (175.6, 79.9)
- added R1303: 22, Resistor_SMD:R_0402_1005Metric_Pad0.72x0.64mm_HandSolder, F.Cu at (174.4, 58.7)
- added RN401: R_Pack04, Resistor_SMD:R_Array_Concave_4x0402, F.Cu at (186.2, 62.4)
- added RN402: R_Pack04, Resistor_SMD:R_Array_Concave_4x0402, F.Cu at (186.2, 59.3)
- added X1301: ASAAIG-40.000MHZ, ETH3CDAQ1:ASAAIG, F.Cu at (174.9, 56.1)
- C1301: renamed from C901; moved to F.Cu
- C1304: renamed from C904; moved to F.Cu
- C1307: renamed from C907; moved to F.Cu
- C214: moved to F.Cu
- D1301: renamed from D901; moved to F.Cu
- D501: renamed from D601; value YELLOW -> GREEN
- D502: renamed from D602; value GREEN -> YELLOW
- R1301: renamed from R901; moved to F.Cu
- R1305: renamed from R905; moved to B.Cu
- U1301: renamed from U901; moved to F.Cu
- U204: value DG419xY -> DG419DY
- U404: renamed from U504; footprint Package_SO:TSSOP-8_3x3mm_P0.65mm -> Package_SO:MSOP-8_3x3mm_P0.65mm
- moved C420 18.1 mm to (194.1, 75.2)
- moved R1306 17.9 mm to (176.9, 73.3)
- moved C401 17.8 mm to (212.1, 74.3)
- moved R1305 17.3 mm to (177.5, 77.5), turned to 0 degrees
- moved U1303 17.0 mm to (178.2, 72.6)
- moved C1311 17.0 mm to (179.6, 70.5)
- moved R1302 17.0 mm to (176.9, 70.5)
- moved R1304 17.0 mm to (179.6, 73.7)
- moved R1307 16.4 mm to (179.6, 71.8)
- moved C1302 7.69 mm to (178.4, 55.6), turned to 180 degrees
- moved C1307 6.99 mm to (182.2, 56.5), turned to 0 degrees
- moved C1310 6.48 mm to (175.6, 66.7), turned to 90 degrees
- moved R1002 6.25 mm to (214.5, 125.3)
- moved C1308 5.88 mm to (181.9, 63.2)
- moved Q302 5.85 mm to (199.9, 124.5)
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- renumbered C1501 to C1001, C1502 to C1002, C1503 to C1003, C902 to C1302, C903 to C1303, C905 to C1305, C906 to C1306, C909 to C1308, C912 to C1309, C915 to C1310, C918 to C1311, C501 to C401, C502 to C402, C503 to C403, C504 to C404, C505 to C405, C506 to C406, C507 to C407, C508 to C408, C509 to C409, C510 to C410, C511 to C411, C512 to C412, C513 to C413, C514 to C414, C515 to C415, C516 to C416, C517 to C417, C518 to C418, C519 to C419, C520 to C420, C521 to C421, C522 to C422, C523 to C423, C524 to C424, C601 to C501, C602 to C502, C603 to C503, C604 to C504, C605 to C505, C606 to C506, C607 to C507, C608 to C508, C609 to C509, C610 to C510, C611 to C511, C612 to C512, C613 to C513, C614 to C514, C701 to C601, C702 to C602, C703 to C603, C704 to C604, C705 to C605, C706 to C606, C707 to C607, C708 to C608, C709 to C609, C1401 to C901, C1402 to C902, C1403 to C903, C1404 to C904, C1405 to C905, C1406 to C906, C1407 to C907, D501 to D401, D502 to D402, D503 to D403, D701 to D601, D702 to D602, D703 to D603, FB501 to FB401, FB601 to FB501, J1201 to J1101, J1101 to J1201, J501 to J401, J502 to J402, J1001 to J701, J1301 to J801, J1302 to J802, L601 to L501, L701 to L601, R1501 to R1001, R1502 to R1002, R903 to R1302, R904 to R1304, R906 to R1306, R907 to R1307, R501 to R401, R502 to R402, R503 to R403, R504 to R404, R505 to R405, R506 to R406, R507 to R407, R508 to R408, R509 to R409, R510 to R410, R511 to R411, R512 to R412, R513 to R413, R514 to R414, R601 to R501, R602 to R502, R603 to R503, R604 to R504, R605 to R505, R606 to R506, R607 to R507, R608 to R508, R609 to R509, R610 to R510, R611 to R511, R612 to R512, R613 to R513, R614 to R514, R615 to R515, R616 to R516, R617 to R517, R618 to R518, R619 to R519, R620 to R520, R621 to R521, R701 to R601, R702 to R602, R703 to R603, R704 to R604, R705 to R605, R706 to R606, U1501 to U1001, U904 to U1302, U909 to U1303, U211 to U210, U210 to U211, U501 to U401, U502 to U402, U503 to U403, U505 to U405, U601 to U501, U602 to U502, U603 to U503, U701 to U601, U702 to U602, U703 to U603, U1401 to U901, Y501 to Y401, Y601 to Y501
Connections:
- net /FPGA 1/FLASH_MISO renamed /FPGA 1/iCE_MISO
- net /FPGA 1/FLASH_MOSI renamed /FPGA 1/iCE_MOSI
- net /FPGA 1/FT_SCL renamed /FPGA 1/iCE_SCK
- net /FPGA 1/FT_SSn renamed /FPGA 1/iCE_SSn
- net /FPGA 1/~CRESET renamed /FPGA 1/iCE_CRESET
- J1101 pad 1: (no net) -> AGNDF
- J1101 pad 10: (no net) -> /CH3 Connector/ADIN3
- J1101 pad 11: (no net) -> /CH3 Connector/ADIN3
- J1101 pad 12: (no net) -> /CH3 Connector/ADIN3
- J1101 pad 13: (no net) -> AGNDF
- J1101 pad 14: (no net) -> AGNDF
- J1101 pad 15: (no net) -> +3V3
- J1101 pad 16: (no net) -> +3V3
- J1101 pad 18: (no net) -> +5V
- J1101 pad 19: (no net) -> -18VF
- J1101 pad 2: (no net) -> /CH1 Connector/I2C_SCL
- J1101 pad 20: (no net) -> +18VF
- J1101 pad 3: (no net) -> AGNDF
- J1101 pad 4: (no net) -> /CH1 Connector/I2C_SDA
- J1101 pad 5: (no net) -> /CH1 Connector/CANH
- J1101 pad 6: (no net) -> /CH1 Connector/CANL
- J1101 pad 7: (no net) -> AGNDF
- J1101 pad 8: (no net) -> AGNDF
- J1101 pad 9: (no net) -> /CH3 Connector/ADIN3
- J1201 pad 1: (no net) -> AGNDF
- J1201 pad 10: (no net) -> /CH2 Connector/ADIN2
- J1201 pad 11: (no net) -> /CH2 Connector/ADIN2
- J1201 pad 12: (no net) -> /CH2 Connector/ADIN2
- J1201 pad 13: (no net) -> AGNDF
- J1201 pad 14: (no net) -> AGNDF
- J1201 pad 15: (no net) -> +3V3
- J1201 pad 16: (no net) -> +3V3
- J1201 pad 18: (no net) -> +5V
- J1201 pad 19: (no net) -> -18VF
- J1201 pad 2: (no net) -> /CH1 Connector/I2C_SCL
- J1201 pad 20: (no net) -> +18VF
- J1201 pad 3: (no net) -> AGNDF
- J1201 pad 4: (no net) -> /CH1 Connector/I2C_SDA
- J1201 pad 5: (no net) -> /CH1 Connector/CANH
- J1201 pad 6: (no net) -> /CH1 Connector/CANL
- J1201 pad 7: (no net) -> AGNDF
- J1201 pad 8: (no net) -> AGNDF
- J1201 pad 9: (no net) -> /CH2 Connector/ADIN2
- J701 pad 2: (no net) -> /CH1 Connector/I2C_SCL
- J701 pad 4: (no net) -> /CH1 Connector/I2C_SDA
- J701 pad 5: (no net) -> /CH1 Connector/CANH
- J701 pad 6: (no net) -> /CH1 Connector/CANL
- R202 pad 2: (no net) -> +10VRF
- R216 pad 2: /ADC 1/AD_COMP1 -> /FPGA 1/ADC_COMP1
- R302 pad 2: (no net) -> /MCU/MCU_AD_RFS
- R313 pad 1: (no net) -> +10VRF
- R401 pad 1: /MCU/CANH -> /CH1 Connector/CANH
- R401 pad 2: /MCU/CANL -> /CH1 Connector/CANL
- R405 pad 2: /MCU/I2C_SCL -> /CH1 Connector/I2C_SCL
- R406 pad 2: /MCU/I2C_SDA -> /CH1 Connector/I2C_SDA
- U1302 pad 20: (no net) -> /FPGA 1/FPGA_CLK
- U1302 pad 23: (no net) -> /ADC 1/FGPA1_AD_ID
- U1302 pad 25: (no net) -> /FPGA 1/FGPA1_AD_VRH
- U1302 pad 26: (no net) -> /ADC 1/FGPA1_AD_IIN
- U1302 pad 27: (no net) -> /ADC 1/FGPA1_AD_IRP
- U1302 pad 28: (no net) -> /ADC 1/FGPA1_AD_IRN
- U1302 pad 31: (no net) -> /FPGA 1/ADC_COMP1
- U1302 pad 32: (no net) -> /ADC 1/FPGA1_MUX_ADIN
- U1302 pad 34: (no net) -> /ADC 1/FPGA1_MUX_10V
- U1302 pad 37: (no net) -> /ADC 1/FPGA1_MUX_GND
- U1302 pad 44: (no net) -> /FPGA 1/FGPA1_nSS
- U1302 pad 46: (no net) -> /FPGA 1/FGPA1_MISO
- U1302 pad 47: (no net) -> /FPGA 1/FGPA1_MOSI
- U1302 pad 48: (no net) -> /FPGA 1/FGPA1_SCLK
- U1302 pad 7: (no net) -> /FPGA 1/iCE_CDONE
- U201 pad 1: (no net) -> /ADC 1/FPGA1_MUX_ADIN
- U201 pad 12: +5VF -> +3.3VF
- U201 pad 8: (no net) -> /ADC 1/FPGA1_MUX_GND
- U201 pad 9: (no net) -> /ADC 1/FPGA1_MUX_10V
- U202 pad 1: (no net) -> /ADC 1/FGPA1_AD_IIN
- U202 pad 12: +5VF -> +3.3VF
- U202 pad 16: (no net) -> /ADC 1/FGPA1_AD_ID
- U202 pad 8: (no net) -> /ADC 1/FGPA1_AD_IRN
- U202 pad 9: (no net) -> /ADC 1/FGPA1_AD_IRP
- U204 pad 5: +5VF -> +3.3VF
- U204 pad 6: (no net) -> /FPGA 1/FGPA1_AD_VRH
- U212 pad 7: /ADC 1/AD_COMP1 -> /FPGA 1/ADC_COMP1
- U402 pad 6: /MCU/CANL -> /CH1 Connector/CANL
- U402 pad 7: /MCU/CANH -> /CH1 Connector/CANH
- U403 pad 110: (no net) -> /FPGA 1/FGPA1_nSS
- U403 pad 111: (no net) -> /FPGA 1/FGPA1_SCLK
- U403 pad 112: (no net) -> /MCU/MCU_MISO
- U403 pad 113: (no net) -> /MCU/MCU_MOSI
- U403 pad 40: /MCU/TRIG_EN -> (no net)
- U403 pad 41: /MCU/TRIG_OUT -> (no net)
- U403 pad 42: /MCU/TRIG_IN -> (no net)
- U403 pad 7: (no net) -> /MCU/TRIG_EN
- U403 pad 8: (no net) -> /MCU/TRIG_OUT
- U403 pad 9: (no net) -> /MCU/TRIG_IN
- U403 pad 98: (no net) -> /MCU/MCU_AD_RFS
- U404 pad 2: /MCU/I2C_SCL -> /CH1 Connector/I2C_SCL
- U404 pad 3: /MCU/I2C_SDA -> /CH1 Connector/I2C_SDA
Other:
- board size 72.5 x 100 mm -> 73 x 100 mm
