File: hardware/project/ETH3CADC1/ETH3CADC1.kicad_pcb (KiCad board)
At the start: 6 copper layers, 73 x 100 mm, 238 parts, among them J1101 Conn_02x10_Odd_Even, J1201 Conn_02x10_Odd_Even, J1301 Conn_02x05_Odd_Even, J401 20021111-00010T4LF, J402 Conn_02x01, J701 Conn_02x10_Odd_Even, J801 Conn_02x02_Odd_Even, J802 Conn_02x04_Odd_Even, Q301 MMBTA55, Q302 BC847, U1001 LM337_SOT223, U1301 ICE40UP5K-SG48ITR, U1302 W25Q32JVSS, U1303 AP2127K-1.2, U201 DG211, U202 DG211B, U203 OPA2192, U204 DG419DY, U205 OPA140, U206 LT5400-100k-100k, U207 LT5400-5k-1k, U208 OPA177, U209 OPA140, U210 LT5400-10k-10k, U211 OPA192, U212 LM311, U301 LT1021-7, U302 LM399H, U303 OPA177, U401 HDC1080, U402 MCP2551-I-SN, U403 STM32H743ZI, U404 PCA9517, U405 24LC08B-E/MS, U501 LAN8742A, U502 LC03-3.3, U503 LC03-3.3, U601 TXB0104PW, U602 ADuM5402, U603 74AC125, U901 MT48LC16M16A2P-6A, X1301 ASAAIG-40.000MHZ, Y401 NX3225GD-8MHZ, Y501 NX5032GA-25.000M-LN-CD-1

Commit message: Development
Parts:
- removed the C207 at (163.7, 60.2)
- removed the C213 at (160.8, 57.3)
- removed the C216 at (170.7, 58.2)
- removed the C218 at (174.1, 58.0)
- removed the R209 at (166.0, 73.9)
- removed the R219 at (158.2, 54.9)
- added C1201: 100n, Capacitor_SMD:C_0402_1005Metric_Pad0.74x0.62mm_HandSolder, B.Cu at (174.2, 66.7)
- added C1202: 100n, Capacitor_SMD:C_0402_1005Metric_Pad0.74x0.62mm_HandSolder, B.Cu at (175.9, 60.6)
- added C1203: 100n, Capacitor_SMD:C_0402_1005Metric_Pad0.74x0.62mm_HandSolder, B.Cu at (182.5, 63.4)
- added C1204: 100n, Capacitor_SMD:C_0402_1005Metric_Pad0.74x0.62mm_HandSolder, B.Cu at (179.3, 70.6)
- added C1206: 4u7, Capacitor_SMD:C_0603_1608Metric_Pad1.08x0.95mm_HandSolder, F.Cu at (182.0, 53.6)
- added C1207: 4u7, Capacitor_SMD:C_0603_1608Metric_Pad1.08x0.95mm_HandSolder, B.Cu at (182.0, 55.9)
- added C1208: 100n, Capacitor_SMD:C_0402_1005Metric_Pad0.74x0.62mm_HandSolder, B.Cu at (182.4, 58.4)
- added C1212: 4u7, Capacitor_SMD:C_0603_1608Metric_Pad1.08x0.95mm_HandSolder, F.Cu at (182.0, 55.9)
- added C1305: 100n, Capacitor_SMD:C_0402_1005Metric_Pad0.74x0.62mm_HandSolder, B.Cu at (174.6, 89.0)
- added C1308: 100n, Capacitor_SMD:C_0402_1005Metric_Pad0.74x0.62mm_HandSolder, B.Cu at (182.4, 91.4)
- added C1310: 4u7, Capacitor_SMD:C_0603_1608Metric_Pad1.08x0.95mm_HandSolder, B.Cu at (179.3, 93.7)
- added C1311: 100n, Capacitor_SMD:C_0402_1005Metric_Pad0.74x0.62mm_HandSolder, F.Cu at (179.1, 91.1)
- added C1401: 100n, Capacitor_SMD:C_0402_1005Metric_Pad0.74x0.62mm_HandSolder, F.Cu at (139.8, 36.6)
- added C1402: 100n, Capacitor_SMD:C_0402_1005Metric_Pad0.74x0.62mm_HandSolder, F.Cu at (143.0, 38.6)
- added C1403: 100n, Capacitor_SMD:C_0402_1005Metric_Pad0.74x0.62mm_HandSolder, F.Cu at (136.7, 44.5)
- added C1404: 100n, Capacitor_SMD:C_0402_1005Metric_Pad0.74x0.62mm_HandSolder, F.Cu at (133.5, 40.5)
- added C1405: 100n, Capacitor_SMD:C_0402_1005Metric_Pad0.74x0.62mm_HandSolder, F.Cu at (136.6, 38.6)
- added C1406: 100n, Capacitor_SMD:C_0402_1005Metric_Pad0.74x0.62mm_HandSolder, F.Cu at (147.0, 27.6)
- added C1407: 100n, Capacitor_SMD:C_0402_1005Metric_Pad0.74x0.62mm_HandSolder, F.Cu at (142.4, 32.1)
- added C1408: 100n, Capacitor_SMD:C_0402_1005Metric_Pad0.74x0.62mm_HandSolder, F.Cu at (133.5, 42.5)
- added C1409: 100n, Capacitor_SMD:C_0402_1005Metric_Pad0.74x0.62mm_HandSolder, F.Cu at (147.0, 29.6)
- added C1410: 2n2/SMD, Capacitor_SMD:C_0603_1608Metric_Pad1.08x0.95mm_HandSolder, F.Cu at (134.3, 32.4)
- added C1411: 100n, Capacitor_SMD:C_0402_1005Metric_Pad0.74x0.62mm_HandSolder, F.Cu at (143.1, 34.1)
- added C1412: 100n, Capacitor_SMD:C_0402_1005Metric_Pad0.74x0.62mm_HandSolder, F.Cu at (136.7, 40.5)
- added C1413: 100n, Capacitor_SMD:C_0402_1005Metric_Pad0.74x0.62mm_HandSolder, F.Cu at (145.6, 32.1)
- added C1414: 100n, Capacitor_SMD:C_0402_1005Metric_Pad0.74x0.62mm_HandSolder, F.Cu at (174.6, 86.4)
- added C1415: 100n, Capacitor_SMD:C_0402_1005Metric_Pad0.74x0.62mm_HandSolder, F.Cu at (139.8, 38.6)
- added C1416: 33p, Capacitor_SMD:C_0402_1005Metric_Pad0.74x0.62mm_HandSolder, F.Cu at (133.5, 44.5)
- added C1417: 100n, Capacitor_SMD:C_0402_1005Metric_Pad0.74x0.62mm_HandSolder, F.Cu at (136.7, 42.5)
- added C1418: 100n, Capacitor_SMD:C_0402_1005Metric_Pad0.74x0.62mm_HandSolder, F.Cu at (143.1, 36.1)
- added C1419: 100n, Capacitor_SMD:C_0402_1005Metric_Pad0.74x0.62mm_HandSolder, F.Cu at (146.3, 34.1)
- added C1420: 100n, Capacitor_SMD:C_0402_1005Metric_Pad0.74x0.62mm_HandSolder, F.Cu at (139.9, 40.5)
- added C1421: 100n, Capacitor_SMD:C_0402_1005Metric_Pad0.74x0.62mm_HandSolder, F.Cu at (148.8, 31.6)
- added C1601: 100n, Capacitor_SMD:C_0402_1005Metric_Pad0.74x0.62mm_HandSolder, F.Cu at (123.4, 132.9)
- added C1602: 100n, Capacitor_SMD:C_0402_1005Metric_Pad0.74x0.62mm_HandSolder, F.Cu at (118.7, 138.1)
- added C1603: 100n, Capacitor_SMD:C_0402_1005Metric_Pad0.74x0.62mm_HandSolder, F.Cu at (126.7, 130.8)
- added C1604: 100n, Capacitor_SMD:C_0402_1005Metric_Pad0.74x0.62mm_HandSolder, F.Cu at (122.7, 135.4)
- added C1605: 100n, Capacitor_SMD:C_0402_1005Metric_Pad0.74x0.62mm_HandSolder, F.Cu at (126.6, 132.9)
- added C1606: 4u7, Capacitor_SMD:C_0603_1608Metric_Pad1.08x0.95mm_HandSolder, F.Cu at (182.0, 119.6)
- added C1607: 4u7, Capacitor_SMD:C_0603_1608Metric_Pad1.08x0.95mm_HandSolder, F.Cu at (112.5, 135.5)
- added C1608: 100n, Capacitor_SMD:C_0402_1005Metric_Pad0.74x0.62mm_HandSolder, F.Cu at (121.9, 138.1)
- added C1609: 100n, Capacitor_SMD:C_0402_1005Metric_Pad0.74x0.62mm_HandSolder, F.Cu at (125.9, 134.9)
- added C1610: 4u7, Capacitor_SMD:C_0603_1608Metric_Pad1.08x0.95mm_HandSolder, F.Cu at (119.0, 129.2)
- added C1611: 100n, Capacitor_SMD:C_0402_1005Metric_Pad0.74x0.62mm_HandSolder, F.Cu at (119.5, 136.1)
- added C1612: 4u7, Capacitor_SMD:C_0603_1608Metric_Pad1.08x0.95mm_HandSolder, F.Cu at (112.5, 133.0)
- added C1701: 100n, Capacitor_SMD:C_0402_1005Metric_Pad0.74x0.62mm_HandSolder, F.Cu at (90.8, 135.9)
- added C1702: 100n, Capacitor_SMD:C_0402_1005Metric_Pad0.74x0.62mm_HandSolder, F.Cu at (91.9, 126.0)
- added C1703: 100n, Capacitor_SMD:C_0402_1005Metric_Pad0.74x0.62mm_HandSolder, F.Cu at (91.9, 128.0)
- added C1704: 100n, Capacitor_SMD:C_0402_1005Metric_Pad0.74x0.62mm_HandSolder, F.Cu at (76.1, 143.6)
- added C1705: 100n, Capacitor_SMD:C_0402_1005Metric_Pad0.74x0.62mm_HandSolder, F.Cu at (84.4, 137.0)
- added C1706: 100n, Capacitor_SMD:C_0402_1005Metric_Pad0.74x0.62mm_HandSolder, F.Cu at (79.3, 141.6)
- added C1707: 100n, Capacitor_SMD:C_0402_1005Metric_Pad0.74x0.62mm_HandSolder, F.Cu at (88.7, 131.4)
- added C1708: 100n, Capacitor_SMD:C_0402_1005Metric_Pad0.74x0.62mm_HandSolder, F.Cu at (83.3, 139.0)
- added C1709: 100n, Capacitor_SMD:C_0402_1005Metric_Pad0.74x0.62mm_HandSolder, F.Cu at (88.7, 133.3)
- added C1710: 2n2/SMD, Capacitor_SMD:C_0603_1608Metric_Pad1.08x0.95mm_HandSolder, F.Cu at (81.7, 132.8)
- added C1711: 100n, Capacitor_SMD:C_0402_1005Metric_Pad0.74x0.62mm_HandSolder, F.Cu at (91.9, 130.0)
- added C1712: 100n, Capacitor_SMD:C_0402_1005Metric_Pad0.74x0.62mm_HandSolder, F.Cu at (76.1, 145.5)
- added C1713: 100n, Capacitor_SMD:C_0402_1005Metric_Pad0.74x0.62mm_HandSolder, F.Cu at (82.5, 144.9)
- added C1714: 100n, Capacitor_SMD:C_0402_1005Metric_Pad0.74x0.62mm_HandSolder, F.Cu at (91.9, 133.9)
- added C1715: 100n, Capacitor_SMD:C_0402_1005Metric_Pad0.74x0.62mm_HandSolder, F.Cu at (82.5, 143.0)
- added C1716: 33p, Capacitor_SMD:C_0402_1005Metric_Pad0.74x0.62mm_HandSolder, F.Cu at (79.3, 145.5)
- added C1717: 100n, Capacitor_SMD:C_0402_1005Metric_Pad0.74x0.62mm_HandSolder, F.Cu at (86.5, 139.0)
- added C1718: 100n, Capacitor_SMD:C_0402_1005Metric_Pad0.74x0.62mm_HandSolder, F.Cu at (83.3, 141.0)
- added C1719: 100n, Capacitor_SMD:C_0402_1005Metric_Pad0.74x0.62mm_HandSolder, F.Cu at (91.9, 131.9)
- added C1720: 100n, Capacitor_SMD:C_0402_1005Metric_Pad0.74x0.62mm_HandSolder, F.Cu at (87.6, 137.0)
- added C1721: 100n, Capacitor_SMD:C_0402_1005Metric_Pad0.74x0.62mm_HandSolder, F.Cu at (79.3, 143.6)
- added C204: 100n, Capacitor_SMD:C_0402_1005Metric_Pad0.74x0.62mm_HandSolder, B.Cu at (173.1, 54.9)
- added C212: 100n, Capacitor_SMD:C_0402_1005Metric_Pad0.74x0.62mm_HandSolder, B.Cu at (158.0, 60.3)
- added C215: 100n, Capacitor_SMD:C_0402_1005Metric_Pad0.74x0.62mm_HandSolder, B.Cu at (160.7, 57.3)
- added C217: 100n, Capacitor_SMD:C_0402_1005Metric_Pad0.74x0.62mm_HandSolder, B.Cu at (170.7, 58.2)
- added C220: 100n, Capacitor_SMD:C_0402_1005Metric_Pad0.74x0.62mm_HandSolder, B.Cu at (160.8, 62.2)
- added D1301: CDBU0520, Diode_SMD:D_SOD-523, F.Cu at (182.4, 91.4)
- added D1401: BAV21W, Diode_SMD:D_SOD-123, F.Cu at (143.4, 23.0)
- added D1402: BAV21W, Diode_SMD:D_SOD-123, F.Cu at (135.0, 29.4)
- added D1601: CDBU0520, Diode_SMD:D_SOD-523, F.Cu at (112.1, 138.0)
- added D1701: BAV21W, Diode_SMD:D_SOD-123, F.Cu at (87.1, 122.2)
- added D1702: BAV21W, Diode_SMD:D_SOD-123, F.Cu at (67.3, 141.9)
- added J1201: Conn_02x05_Odd_Even, Connector_PinHeader_1.27mm:PinHeader_2x05_P1.27mm_Vertical, F.Cu at (175.3, 79.2)
- added J1601: Conn_02x05_Odd_Even, Connector_PinHeader_1.27mm:PinHeader_2x05_P1.27mm_Vertical, F.Cu at (175.4, 145.3)
- added R1201: 22, Resistor_SMD:R_0402_1005Metric_Pad0.72x0.64mm_HandSolder, F.Cu at (174.1, 57.9)
- added R1203: 10k, Resistor_SMD:R_0402_1005Metric_Pad0.72x0.64mm_HandSolder, B.Cu at (176.7, 70.6)
- added R1207: 10k, Resistor_SMD:R_0402_1005Metric_Pad0.72x0.64mm_HandSolder, B.Cu at (177.3, 80.5)
- added R1302: 10k, Resistor_SMD:R_0402_1005Metric_Pad0.72x0.64mm_HandSolder, B.Cu at (177.3, 109.7)
- added R1304: NC, Resistor_SMD:R_0402_1005Metric_Pad0.72x0.64mm_HandSolder, B.Cu at (173.1, 102.6)
- added R1305: 10k, Resistor_SMD:R_0402_1005Metric_Pad0.72x0.64mm_HandSolder, B.Cu at (179.3, 106.8)
- added R1306: 10k, Resistor_SMD:R_0402_1005Metric_Pad0.72x0.64mm_HandSolder, B.Cu at (174.2, 102.6)
- added R1307: 10k, Resistor_SMD:R_0402_1005Metric_Pad0.72x0.64mm_HandSolder, B.Cu at (177.3, 113.5)
- added R1308: 10k, Resistor_SMD:R_0402_1005Metric_Pad0.72x0.64mm_HandSolder, B.Cu at (176.7, 106.4)
- added R1309: 10k, Resistor_SMD:R_0402_1005Metric_Pad0.72x0.64mm_HandSolder, B.Cu at (179.3, 104.9)
- added R1310: 100, Resistor_SMD:R_0402_1005Metric_Pad0.72x0.64mm_HandSolder, F.Cu at (176.5, 91.1)
- added R1401: 10k, Resistor_SMD:R_0402_1005Metric_Pad0.72x0.64mm_HandSolder, F.Cu at (146.5, 25.6)
- added R1402: 10k, Resistor_SMD:R_0402_1005Metric_Pad0.72x0.64mm_HandSolder, F.Cu at (143.8, 28.2)
- added R1403: 10k, Resistor_SMD:R_0402_1005Metric_Pad0.72x0.64mm_HandSolder, F.Cu at (125.0, 39.7)
- added R1404: 10k, Resistor_SMD:R_0402_1005Metric_Pad0.72x0.64mm_HandSolder, F.Cu at (130.2, 41.7)
- added R1405: 10M, Resistor_SMD:R_0603_1608Metric_Pad0.98x0.95mm_HandSolder, F.Cu at (123.2, 42.2)
- added R1406: 0, Resistor_SMD:R_0402_1005Metric_Pad0.72x0.64mm_HandSolder, F.Cu at (130.2, 43.7)
- added R1407: 10k, Resistor_SMD:R_0402_1005Metric_Pad0.72x0.64mm_HandSolder, F.Cu at (143.8, 30.1)
- added R1408: 62/.1%, Resistor_SMD:R_0603_1608Metric_Pad0.98x0.95mm_HandSolder, F.Cu at (123.2, 44.7)
- added R1409: 10, Resistor_SMD:R_0402_1005Metric_Pad0.72x0.64mm_HandSolder, F.Cu at (127.0, 43.7)
- added R1410: 10, Resistor_SMD:R_0402_1005Metric_Pad0.72x0.64mm_HandSolder, F.Cu at (136.6, 36.6)
- added R1411: 12k/.05%, Resistor_SMD:R_0603_1608Metric_Pad0.98x0.95mm_HandSolder, F.Cu at (132.8, 38.0)
- added R1412: 10, Resistor_SMD:R_0402_1005Metric_Pad0.72x0.64mm_HandSolder, F.Cu at (139.9, 34.6)
- added R1413: 10, Resistor_SMD:R_0402_1005Metric_Pad0.72x0.64mm_HandSolder, F.Cu at (136.6, 34.6)
- added R1414: 62k, Resistor_SMD:R_0402_1005Metric_Pad0.72x0.64mm_HandSolder, F.Cu at (127.0, 41.7)
- added R1415: 620/.05%, Resistor_SMD:R_0603_1608Metric_Pad0.98x0.95mm_HandSolder, F.Cu at (140.0, 29.0)
- added R1416: 3k9/.05%, Resistor_SMD:R_0603_1608Metric_Pad0.98x0.95mm_HandSolder, F.Cu at (142.7, 25.9)
- added R1417: 10, Resistor_SMD:R_0402_1005Metric_Pad0.72x0.64mm_HandSolder, F.Cu at (128.2, 39.7)
- added R1418: 62/.1%, Resistor_SMD:R_0603_1608Metric_Pad0.98x0.95mm_HandSolder, F.Cu at (148.5, 22.6)
- added R1419: 39k/.05%, Resistor_SMD:R_0603_1608Metric_Pad0.98x0.95mm_HandSolder, F.Cu at (138.6, 32.4)
- added R1420: 3k9/.05%, Resistor_SMD:R_0603_1608Metric_Pad0.98x0.95mm_HandSolder, F.Cu at (132.8, 35.5)
- added R1601: 22, Resistor_SMD:R_0402_1005Metric_Pad0.72x0.64mm_HandSolder, F.Cu at (127.7, 124.3)
- added R1602: 10k, Resistor_SMD:R_0402_1005Metric_Pad0.72x0.64mm_HandSolder, F.Cu at (123.3, 126.8)
- added R1603: 10k, Resistor_SMD:R_0402_1005Metric_Pad0.72x0.64mm_HandSolder, F.Cu at (120.2, 133.4)
- added R1604: 10k, Resistor_SMD:R_0402_1005Metric_Pad0.72x0.64mm_HandSolder, F.Cu at (126.6, 126.8)
- added R1605: 10k, Resistor_SMD:R_0402_1005Metric_Pad0.72x0.64mm_HandSolder, F.Cu at (116.3, 136.1)
- added R1606: 10k, Resistor_SMD:R_0402_1005Metric_Pad0.72x0.64mm_HandSolder, F.Cu at (120.2, 131.4)
- added R1607: 10k, Resistor_SMD:R_0402_1005Metric_Pad0.72x0.64mm_HandSolder, F.Cu at (126.1, 128.8)
- added R1608: 10k, Resistor_SMD:R_0402_1005Metric_Pad0.72x0.64mm_HandSolder, F.Cu at (123.4, 130.9)
- added R1609: 10k, Resistor_SMD:R_0402_1005Metric_Pad0.72x0.64mm_HandSolder, F.Cu at (115.5, 138.1)
- added R1610: 100, Resistor_SMD:R_0402_1005Metric_Pad0.72x0.64mm_HandSolder, F.Cu at (122.8, 128.9)
- added R1701: 10k, Resistor_SMD:R_0402_1005Metric_Pad0.72x0.64mm_HandSolder, F.Cu at (76.1, 141.6)
- added R1702: 10k, Resistor_SMD:R_0402_1005Metric_Pad0.72x0.64mm_HandSolder, F.Cu at (85.5, 132.5)
- added R1703: 10k, Resistor_SMD:R_0402_1005Metric_Pad0.72x0.64mm_HandSolder, F.Cu at (88.7, 129.4)
- added R1704: 10k, Resistor_SMD:R_0402_1005Metric_Pad0.72x0.64mm_HandSolder, F.Cu at (81.1, 137.0)
- added R1705: 10M, Resistor_SMD:R_0603_1608Metric_Pad0.98x0.95mm_HandSolder, F.Cu at (86.4, 125.2)
- added R1706: 0, Resistor_SMD:R_0402_1005Metric_Pad0.72x0.64mm_HandSolder, F.Cu at (81.1, 135.1)
- added R1707: 10k, Resistor_SMD:R_0402_1005Metric_Pad0.72x0.64mm_HandSolder, F.Cu at (88.7, 127.4)
- added R1708: 62/.1%, Resistor_SMD:R_0603_1608Metric_Pad0.98x0.95mm_HandSolder, F.Cu at (84.9, 128.3)
- added R1709: 10, Resistor_SMD:R_0402_1005Metric_Pad0.72x0.64mm_HandSolder, F.Cu at (91.6, 124.1)
- added R1710: 10, Resistor_SMD:R_0402_1005Metric_Pad0.72x0.64mm_HandSolder, F.Cu at (77.1, 132.5)
- added R1711: 12k/.05%, Resistor_SMD:R_0603_1608Metric_Pad0.98x0.95mm_HandSolder, F.Cu at (92.1, 121.8)
- added R1712: 10, Resistor_SMD:R_0402_1005Metric_Pad0.72x0.64mm_HandSolder, F.Cu at (84.4, 130.5)
- added R1713: 10, Resistor_SMD:R_0402_1005Metric_Pad0.72x0.64mm_HandSolder, F.Cu at (76.8, 139.6)
- added R1714: 62k, Resistor_SMD:R_0402_1005Metric_Pad0.72x0.64mm_HandSolder, F.Cu at (84.4, 135.1)
- added R1715: 620/.05%, Resistor_SMD:R_0603_1608Metric_Pad0.98x0.95mm_HandSolder, F.Cu at (72.3, 141.3)
- added R1716: 3k9/.05%, Resistor_SMD:R_0603_1608Metric_Pad0.98x0.95mm_HandSolder, F.Cu at (77.3, 134.8)
- added R1717: 10, Resistor_SMD:R_0402_1005Metric_Pad0.72x0.64mm_HandSolder, F.Cu at (80.0, 139.6)
- added R1718: 62/.1%, Resistor_SMD:R_0603_1608Metric_Pad0.98x0.95mm_HandSolder, F.Cu at (66.6, 144.8)
- added R1719: 39k/.05%, Resistor_SMD:R_0603_1608Metric_Pad0.98x0.95mm_HandSolder, F.Cu at (72.3, 143.8)
- added R1720: 3k9/.05%, Resistor_SMD:R_0603_1608Metric_Pad0.98x0.95mm_HandSolder, F.Cu at (77.3, 137.4)
- added R207: 10k, Resistor_SMD:R_0402_1005Metric_Pad0.72x0.64mm_HandSolder, F.Cu at (164.8, 65.3)
- added R215: 620/.05%, Resistor_SMD:R_0603_1608Metric_Pad0.98x0.95mm_HandSolder, B.Cu at (166.0, 79.5)
- added R220: 3k9/.05%, Resistor_SMD:R_0603_1608Metric_Pad0.98x0.95mm_HandSolder, B.Cu at (169.7, 77.6)
- added U1201: ICE40UP5K-SG48ITR, Package_DFN_QFN:QFN-48-1EP_7x7mm_P0.5mm_EP5.6x5.6mm_ThermalVias, F.Cu at (177.9, 64.3)
- added U1203: AP2127K-1.2, Package_TO_SOT_SMD:SOT-23-5, F.Cu at (178.2, 54.7)
- added U1302: W25Q32JVSS, Package_SO:SOIC-8_5.23x5.23mm_P1.27mm, F.Cu at (177.8, 105.8)
- added U1401: DG211, Package_SO:TSSOP-16_4.4x5mm_P0.65mm, F.Cu at (160.9, 94.4)
- added U1402: DG211B, Package_SO:TSSOP-16_4.4x5mm_P0.65mm, F.Cu at (168.9, 105.0)
- added U1403: OPA2192, Package_SO:SOIC-8_3.9x4.9mm_P1.27mm, F.Cu at (168.9, 94.2)
- added U1404: DG419DY, Package_SO:SOIC-8_3.9x4.9mm_P1.27mm, F.Cu at (168.8, 87.9)
- added U1405: OPA140, Package_SO:SOIC-8_3.9x4.9mm_P1.27mm, F.Cu at (160.9, 87.9)
- added U1406: LT5400-100k-100k, Package_SO:MSOP-8-1EP_3x3mm_P0.65mm_EP1.73x1.85mm_ThermalVias, F.Cu at (160.9, 99.7)
- added U1407: LT5400-5k-1k, Package_SO:MSOP-8-1EP_3x3mm_P0.65mm_EP1.73x1.85mm_ThermalVias, B.Cu at (168.9, 99.6)
- added U1408: OPA177, Package_SO:SOIC-8_3.9x4.9mm_P1.27mm, B.Cu at (168.8, 87.9)
- added U1409: OPA140, Package_SO:SOIC-8_3.9x4.9mm_P1.27mm, F.Cu at (160.9, 105.0)
- added U1410: LT5400-10k-10k, Package_SO:MSOP-8-1EP_3x3mm_P0.65mm_EP1.73x1.85mm_ThermalVias, F.Cu at (168.9, 99.6)
- added U1411: OPA192, Package_SO:SOIC-8_3.9x4.9mm_P1.27mm, F.Cu at (160.9, 111.5)
- added U1412: LM311, Package_SO:SOIC-8_3.9x4.9mm_P1.27mm, F.Cu at (168.8, 111.5)
- added U1601: ICE40UP5K-SG48ITR, Package_DFN_QFN:QFN-48-1EP_7x7mm_P0.5mm_EP5.6x5.6mm_ThermalVias, F.Cu at (177.9, 130.3)
- added U1602: W25Q32JVSS, Package_SO:SOIC-8_5.23x5.23mm_P1.27mm, F.Cu at (177.8, 138.8)
- added U1603: AP2127K-1.2, Package_TO_SOT_SMD:SOT-23-5, F.Cu at (178.2, 120.8)
- added U1701: DG211, Package_SO:TSSOP-16_4.4x5mm_P0.65mm, F.Cu at (62.9, 123.8)
- added U1702: DG211B, Package_SO:TSSOP-16_4.4x5mm_P0.65mm, F.Cu at (54.2, 130.4)
- added U1703: DG211, Package_SO:TSSOP-16_4.4x5mm_P0.65mm, F.Cu at (54.2, 123.8)
- added U1704: OPA2192, Package_SO:SOIC-8_3.9x4.9mm_P1.27mm, F.Cu at (168.8, 120.9)
- added U1705: DG419DY, Package_SO:SOIC-8_3.9x4.9mm_P1.27mm, F.Cu at (160.9, 120.9)
- added U1706: OPA140, Package_SO:SOIC-8_3.9x4.9mm_P1.27mm, F.Cu at (80.0, 123.8)
- added U1707: LT5400-100k-100k, Package_SO:MSOP-8-1EP_3x3mm_P0.65mm_EP1.73x1.85mm_ThermalVias, F.Cu at (53.4, 142.5)
- added U1708: LT5400-5k-1k, Package_SO:MSOP-8-1EP_3x3mm_P0.65mm_EP1.73x1.85mm_ThermalVias, F.Cu at (60.7, 142.5)
- added U1709: OPA177, Package_SO:SOIC-8_3.9x4.9mm_P1.27mm, F.Cu at (70.9, 136.8)
- added U1710: OPA140, Package_SO:SOIC-8_3.9x4.9mm_P1.27mm, F.Cu at (71.2, 130.4)
- added U1711: LT5400-10k-10k, Package_SO:MSOP-8-1EP_3x3mm_P0.65mm_EP1.73x1.85mm_ThermalVias, F.Cu at (79.1, 129.3)
- added U1712: OPA192, Package_SO:SOIC-8_3.9x4.9mm_P1.27mm, F.Cu at (71.5, 123.8)
- added U1713: LM311, Package_SO:SOIC-8_3.9x4.9mm_P1.27mm, F.Cu at (62.5, 137.0)
- added X1201: ASAAIG-40.000MHZ, ETH3CDAQ1:ASAAIG, F.Cu at (174.6, 55.5)
- added X1601: ASAAIG-40.000MHZ, ETH3CDAQ1:ASAAIG, F.Cu at (174.6, 121.5)
- C209: value 2n2/SMD -> 100n; footprint Capacitor_SMD:C_0603_1608Metric_Pad1.08x0.95mm_HandSolder -> Capacitor_SMD:C_0402_1005Metric_Pad0.74x0.62mm_HandSolder
- C210: value 100n -> 2n2/SMD; footprint Capacitor_SMD:C_0402_1005Metric_Pad0.74x0.62mm_HandSolder -> Capacitor_SMD:C_0603_1608Metric_Pad1.08x0.95mm_HandSolder
- R206: value 10k -> 0; moved to B.Cu
- R208: value 10 -> 62/.1%; footprint Resistor_SMD:R_0402_1005Metric_Pad0.72x0.64mm_HandSolder -> Resistor_SMD:R_0603_1608Metric_Pad0.98x0.95mm_HandSolder
- R211: value 10 -> 12k/.05%; footprint Resistor_SMD:R_0402_1005Metric_Pad0.72x0.64mm_HandSolder -> Resistor_SMD:R_0603_1608Metric_Pad0.98x0.95mm_HandSolder
- R212: value 62k -> 10
- R213: value 620/.05% -> 10; footprint Resistor_SMD:R_0603_1608Metric_Pad0.98x0.95mm_HandSolder -> Resistor_SMD:R_0402_1005Metric_Pad0.72x0.64mm_HandSolder
- R214: value 3k9/.05% -> 62k; footprint Resistor_SMD:R_0603_1608Metric_Pad0.98x0.95mm_HandSolder -> Resistor_SMD:R_0402_1005Metric_Pad0.72x0.64mm_HandSolder
- R216: value 62/.1% -> 3k9/.05%
- R218: value 3k9/.05% -> 62/.1%
- moved C1301 37.2 mm to (174.2, 99.7), turned to 90 degrees
- moved C1307 34.4 mm to (182.0, 88.9), turned to 0 degrees
- moved C1309 33.2 mm to (176.5, 91.1), turned to 0 degrees
- moved C1302 33.1 mm to (175.9, 93.7)
- moved C1304 33.0 mm to (179.3, 103.6)
- moved R1303 33.0 mm to (176.7, 103.6)
- moved C1306 33.0 mm to (182.0, 86.6)
- moved C1312 33.0 mm to (182.0, 88.9)
- moved U1303 33.0 mm to (178.2, 87.8)
- moved X1301 33.0 mm to (174.6, 88.5)
- moved J1301 33.0 mm to (175.4, 112.3)
- moved R1301 33.0 mm to (174.1, 91.1)
- moved U1301 33.0 mm to (177.9, 97.3)
- moved C1303 30.8 mm to (182.5, 96.4), turned to 270 degrees
- moved C210 14.7 mm to (168.9, 70.1), turned to 0 degrees
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- renumbered C1305 to C1205, C1308 to C1209, C1310 to C1210, C1311 to C1211, C204 to C205, C205 to C206, C206 to C207, C212 to C213, C215 to C216, C217 to C218, C220 to C221, D1301 to D1201, D403 to D401, D401 to D403, J1201 to J1501, R1302 to R1202, R1308 to R1204, R1304 to R1205, R1309 to R1206, R1305 to R1208, R1306 to R1209, R1307 to R1210, R207 to R209, R215 to R217, R217 to R219, R412 to R405, R405 to R406, R406 to R407, R407 to R408, R408 to R409, R409 to R410, R413 to R412, R410 to R413, U1302 to U1202
Connections:
- net /CH2 Connector/ADIN2 renamed /ADC 2/ADIN2
- net /CH3 Connector/ADIN3 renamed /ADC 3/ADIN3
- net /FPGA 1/FPGA_CLK renamed /FPGA 2/FPGA_CLK
- net /FPGA 1/iCE_CDONE renamed /FPGA 2/iCE_CDONE
- C1209 pad 1: Net-(C1308-Pad1) -> Net-(C1209-Pad1)
- C1210 pad 1: Net-(C1308-Pad1) -> Net-(C1209-Pad1)
- C1211 pad 1: Net-(C1307-Pad1) -> Net-(C1207-Pad1)
- C1309 pad 1: +3.3VF -> Net-(C1309-Pad1)
- C208 pad 1: -14VF -> +18VF
- C209 pad 1: Net-(C209-Pad1) -> -14VF
- C209 pad 2: Net-(C209-Pad2) -> AGNDF
- C210 pad 1: -14VF -> Net-(C210-Pad1)
- C210 pad 2: AGNDF -> Net-(C210-Pad2)
- C216 pad 1: Net-(C215-Pad1) -> Net-(C216-Pad1)
- C216 pad 2: Net-(C215-Pad2) -> Net-(C216-Pad2)
- D1201 pad 1: Net-(C1312-Pad1) -> Net-(C1212-Pad1)
- D201 pad 1: Net-(C215-Pad1) -> Net-(C216-Pad1)
- D201 pad 2: Net-(C215-Pad2) -> Net-(C216-Pad2)
- D202 pad 1: Net-(C215-Pad2) -> Net-(C216-Pad2)
- D202 pad 2: Net-(C215-Pad1) -> Net-(C216-Pad1)
- J1301 pad 10: /FPGA 1/iCE_SSn -> /FPGA 2/iCE_SSn
- J1301 pad 6: /FPGA 1/iCE_CRESET -> /FPGA 2/iCE_CRESET
- J1301 pad 7: /FPGA 1/iCE_MOSI -> /FPGA 2/iCE_MOSI
- J1301 pad 8: /FPGA 1/iCE_MISO -> /FPGA 2/iCE_MISO
- J1301 pad 9: /FPGA 1/iCE_SCK -> /FPGA 2/iCE_SCK
- R1210 pad 1: Net-(C1308-Pad1) -> Net-(C1209-Pad1)
- R1210 pad 2: Net-(C1307-Pad1) -> Net-(C1207-Pad1)
- R1303 pad 2: /FPGA 1/iCE_SSn -> /FPGA 2/iCE_SSn
- R206 pad 2: Net-(R206-Pad2) -> Net-(R205-Pad1)
- R208 pad 1: Net-(R208-Pad1) -> Net-(C204-Pad1)
- R208 pad 2: -14VF -> /ADC 1/VREF_N7V_LPF
- R210 pad 1: +18VF -> Net-(R210-Pad1)
- R210 pad 2: Net-(R210-Pad2) -> -14VF
- R211 pad 1: Net-(R211-Pad1) -> Net-(C216-Pad2)
- R211 pad 2: -14VF -> Net-(C210-Pad1)
- R212 pad 1: Net-(C215-Pad1) -> +18VF
- R212 pad 2: Net-(C215-Pad2) -> Net-(R212-Pad2)
- R213 pad 2: AGNDF -> -14VF
- R214 pad 1: Net-(R214-Pad1) -> Net-(C216-Pad1)
- R214 pad 2: Net-(C215-Pad1) -> Net-(C216-Pad2)
- R216 pad 1: +3.3VF -> Net-(R216-Pad1)
- R216 pad 2: Net-(R216-Pad2) -> Net-(C216-Pad1)
- R218 pad 1: Net-(R216-Pad2) -> +3.3VF
- R218 pad 2: /FPGA 1/ADC_COMP1 -> Net-(R218-Pad2)
- R219 pad 1: Net-(R216-Pad2) -> Net-(R218-Pad2)
- U1202 pad 2: /FPGA 1/iCE_MISO -> /FPGA 1/iCE_MOSI
- U1202 pad 5: /FPGA 1/iCE_MOSI -> /FPGA 1/iCE_MISO
- U1301 pad 14: /FPGA 1/iCE_MOSI -> /FPGA 2/iCE_MISO
- U1301 pad 15: /FPGA 1/iCE_SCK -> /FPGA 2/iCE_SCK
- U1301 pad 16: /FPGA 1/iCE_SSn -> /FPGA 2/iCE_SSn
- U1301 pad 17: /FPGA 1/iCE_MISO -> /FPGA 2/iCE_MOSI
- U1301 pad 19: /FPGA 1/FGPA1_MOSI -> /FPGA 1/FGPA1_MISO
- U1301 pad 2: /FPGA 1/CODE1 -> /FPGA 2/CODE1
- U1301 pad 20: /FPGA 1/FGPA1_MISO -> /FPGA 2/FGPA2_MISO
- U1301 pad 25: /FPGA 1/FPGA1_UART6_TX -> /FPGA 2/FPGA2_UART2_TX
- U1301 pad 26: /FPGA 1/FPGA1_UART6_RX -> /FPGA 2/FPGA2_UART2_RX
- U1301 pad 29: Net-(C1308-Pad1) -> Net-(C1309-Pad1)
- U1301 pad 3: /FPGA 1/CODE2 -> /FPGA 2/CODE2
- U1301 pad 37: /FPGA 1/FGPA1_AD_VRH -> /FPGA 2/FGPA2_AD_VRH
- U1301 pad 38: /ADC 1/FPGA1_MUX_ADIN -> /ADC 2/FPGA2_MUX_ADIN
- U1301 pad 39: /ADC 1/FPGA1_MUX_N7V -> /ADC 2/FPGA2_MUX_N7V
- U1301 pad 40: /ADC 1/FPGA1_MUX_P10V -> /ADC 2/FPGA2_MUX_P10V
- U1301 pad 41: /ADC 1/FPGA1_MUX_GND -> /ADC 2/FPGA2_MUX_GND
- U1301 pad 42: /ADC 1/FGPA1_AD_IIN -> /ADC 2/FGPA2_AD_IIN
- U1301 pad 43: /ADC 1/FGPA1_AD_IRN -> /ADC 2/FGPA2_AD_IRN
- U1301 pad 44: /ADC 1/FGPA1_AD_ID -> /ADC 2/FGPA2_AD_ID
- U1301 pad 45: /ADC 1/FGPA1_AD_IRP -> /ADC 2/FGPA2_AD_IRP
- U1301 pad 47: /FPGA 1/ADC_COMP1 -> /FPGA 2/ADC_COMP2
- U1301 pad 8: /FPGA 1/iCE_CRESET -> /FPGA 2/iCE_CRESET
- U202 pad 10: Net-(C209-Pad2) -> Net-(C210-Pad2)
- U202 pad 14: Net-(C209-Pad2) -> Net-(C210-Pad2)
- U202 pad 15: Net-(C209-Pad1) -> Net-(C210-Pad1)
- U202 pad 3: Net-(C209-Pad2) -> Net-(C210-Pad2)
- U202 pad 7: Net-(C209-Pad2) -> Net-(C210-Pad2)
- U205 pad 2: Net-(R206-Pad2) -> Net-(R206-Pad1)
- U205 pad 6: Net-(R206-Pad2) -> Net-(R206-Pad1)
- U206 pad 8: Net-(R206-Pad1) -> Net-(R207-Pad1)
- U208 pad 3: /ADC 1/VREF_N7V_LPF -> Net-(C204-Pad1)
- U209 pad 2: Net-(C209-Pad2) -> Net-(C210-Pad2)
- U209 pad 4: Net-(R208-Pad1) -> Net-(R210-Pad1)
- U209 pad 6: Net-(C209-Pad1) -> Net-(C210-Pad1)
- U211 pad 2: Net-(C215-Pad2) -> Net-(C216-Pad2)
- U211 pad 4: Net-(R211-Pad1) -> Net-(R213-Pad1)
- U211 pad 6: Net-(C215-Pad1) -> Net-(C216-Pad1)
- U211 pad 7: Net-(R210-Pad2) -> Net-(R212-Pad2)
- U212 pad 2: Net-(R214-Pad1) -> Net-(R216-Pad1)
- U212 pad 3: Net-(R213-Pad1) -> Net-(R215-Pad1)
- U403 pad 1: (no net) -> /MCU/MCU_AD_RFS
- U403 pad 112: /FPGA 1/FGPA1_MISO -> /FPGA 3/FGPA3_MISO
- U403 pad 119: (no net) -> /FPGA 2/FPGA2_UART2_TX
- U403 pad 122: (no net) -> /FPGA 2/FPGA2_UART2_RX
- U403 pad 133: (no net) -> /FPGA 3/FPGA3_UART2_RX
- U403 pad 134: (no net) -> /FPGA 3/FPGA3_UART2_TX
- U403 pad 98: /MCU/MCU_AD_RFS -> (no net)
Routing:
- net AGNDF: track 41.0 -> 417.0 mm, vias 19 -> 81
- net (no net): track 184.4 -> 537.0 mm, vias 0 -> 77
- net /CH1 Connector/CANL: track 69.8 -> 1.73 mm
- net /MCU/MCU_AD_RFS: track 0.00 -> 66.5 mm
- net -14VF: track 52.4 -> 107.2 mm, vias 20 -> 30
- net +18VF: track 120.5 -> 156.8 mm, vias 8 -> 20
- net +3.3VF: track 132.2 -> 167.5 mm, vias 52 -> 79
- net /FPGA 3/iCE_MOSI: track 0.00 -> 33.8 mm
- net /FPGA 2/iCE_MOSI: track 0.00 -> 33.8 mm
- net /ADC 3/VREF-: track 0.00 -> 31.0 mm, vias 0 -> 3
- net Net-(C1410-Pad2): track 0.00 -> 27.6 mm, vias 0 -> 3
- net Net-(C210-Pad2): track 0.00 -> 27.6 mm, vias 0 -> 3
- net Net-(C209-Pad2): track 26.9 -> 0.00 mm, vias 3 -> 0
- net Net-(U1404-Pad8): track 0.00 -> 24.8 mm, vias 0 -> 2
- net /FPGA 2/iCE_SSn: track 0.00 -> 24.0 mm, vias 0 -> 3
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- added copper zone on F.Cu, net (none)
- added copper zone on In3.Cu, net +5V_TRIG
- added copper zone on F.Cu, net /ADC 1/ADIN1
- added copper zone on F.Cu, net /ADC 2/ADIN2
- added copper zone on In4.Cu, net GND_TRIG
- added copper zone on F.Cu, net Net-(C1207-Pad1)
- added copper zone on F.Cu, net Net-(C1607-Pad1)
- removed copper zone on B.Cu, net AGNDF
- removed copper zone on F.Cu, net AGNDF
