File: hardware/project/ETH3CADC1/CH1_CONN.sch (KiCad schematic (older format))
At the start: 1 part, among them J1001 Conn_02x10_Odd_Even

Commit message: PCB layout
Connections:
- net GND: now reaches J1001.1 (Pin_1)
- net GND: now also J1001.13 (Pin_13), J1001.14 (Pin_14), J1001.3 (Pin_3), J1001.7 (Pin_7), J1001.8 (Pin_8)
- net ADIN1: now reaches J1001.10 (Pin_10)
- net ADIN1: now also J1001.11 (Pin_11), J1001.12 (Pin_12), J1001.9 (Pin_9)
- net +3V3: now reaches J1001.15 (Pin_15)
- net +3V3: now also J1001.16 (Pin_16)
- net +5V: now reaches J1001.18 (Pin_18)
- net -18VF: now reaches J1001.19 (Pin_19)
- net +18VF: now reaches J1001.20 (Pin_20)
- no-connect marks 0 -> 1
Changed lines of the file:
@@
 $Descr A4 11693 8268
 encoding utf-8
-Sheet 10 13
+Sheet 10 15
 Title ""
 Date ""
@@
 	1    0    0    -1
 $EndComp
+$Comp
+L power:GND #PWR0103
+U 1 1 602209FD
+P 5350 3050
+F 0 "#PWR0103" H 5350 2800 50  0001 C CNN
+F 1 "GND" V 5355 2922 50  0000 R CNN
+F 2 "" H 5350 3050 50  0001 C CNN
+F 3 "" H 5350 3050 50  0001 C CNN
+	1    5350 3050
+	0    1    1    0
+$EndComp
+$Comp
+L power:GND #PWR0104
+U 1 1 60220E99
+P 5350 3150
+F 0 "#PWR0104" H 5350 2900 50  0001 C CNN
+F 1 "GND" V 5355 3022 50  0000 R CNN
+F 2 "" H 5350 3150 50  0001 C CNN
+F 3 "" H 5350 3150 50  0001 C CNN
+	1    5350 3150
+	0    1    1    0
+$EndComp
+$Comp
+L power:GND #PWR0105
+U 1 1 60222DE0
+P 5350 3350
+F 0 "#PWR0105" H 5350 3100 50  0001 C CNN
+F 1 "GND" V 5355 3222 50  0000 R CNN
+F 2 "" H 5350 3350 50  0001 C CNN
+F 3 "" H 5350 3350 50  0001 C CNN
+	1    5350 3350
+	0    1    1    0
+$EndComp
+$Comp
+L power:GND #PWR0106
+U 1 1 60223109
+P 5850 3350
+F 0 "#PWR0106" H 5850 3100 50  0001 C CNN
+F 1 "GND" V 5855 3222 50  0000 R CNN
+F 2 "" H 5850 3350 50  0001 C CNN
+F 3 "" H 5850 3350 50  0001 C CNN
+	1    5850 3350
+	0    -1   -1   0
+$EndComp
+$Comp
+L power:GND #PWR0107
+U 1 1 60223752
+P 5350 3650
+F 0 "#PWR0107" H 5350 3400 50  0001 C CNN
+F 1 "GND" V 5355 3522 50  0000 R CNN
+F 2 "" H 5350 3650 50  0001 C CNN
+F 3 "" H 5350 3650 50  0001 C CNN
+	1    5350 3650
+	0    1    1    0
+$EndComp
+$Comp
+L power:GND #PWR0108
+U 1 1 60223BA8
+P 5850 3650
+F 0 "#PWR0108" H 5850 3400 50  0001 C CNN
+F 1 "GND" V 5855 3522 50  0000 R CNN
+F 2 "" H 5850 3650 50  0001 C CNN
+F 3 "" H 5850 3650 50  0001 C CNN
+	1    5850 3650
+	0    -1   -1   0
+$EndComp
+$Comp
+L power:+3.3V #PWR0109
+U 1 1 6022456D
+P 5350 3750
+F 0 "#PWR0109" H 5350 3600 50  0001 C CNN
+F 1 "+3.3V" V 5350 3900 50  0000 L CNN
+F 2 "" H 5350 3750 50  0001 C CNN
+F 3 "" H 5350 3750 50  0001 C CNN
+	1    5350 3750
+	0    -1   -1   0
+$EndComp
+$Comp
+L power:+3.3V #PWR0110
+U 1 1 60224CD0
+P 5850 3750
+F 0 "#PWR0110" H 5850 3600 50  0001 C CNN
+F 1 "+3.3V" V 5850 3900 50  0000 L CNN
+F 2 "" H 5850 3750 50  0001 C CNN
+F 3 "" H 5850 3750 50  0001 C CNN
+	1    5850 3750
+	0    1    1    0
+$EndComp
+NoConn ~ 5350 3850
+$Comp
+L power:+5V #PWR0111
+U 1 1 6022B65E
+P 5850 3850
+F 0 "#PWR0111" H 5850 3700 50  0001 C CNN
+F 1 "+5V" V 5850 4000 50  0000 L CNN
+F 2 "" H 5850 3850 50  0001 C CNN
+F 3 "" H 5850 3850 50  0001 C CNN
+	1    5850 3850
+	0    1    1    0
+$EndComp
+Wire Wire Line
+	5850 3450 5900 3450
+Wire Wire Line
+	5900 3450 5900 3550
+Wire Wire Line
+	5900 3550 5850 3550
+Wire Wire Line
+	5350 3550 5300 3550
+Wire Wire Line
+	5300 3550 5300 3450
+Wire Wire Line
+	5300 3450 5350 3450
+Text HLabel 5950 3450 2    50   Output ~ 0
+ADIN1
+Wire Wire Line
+	5950 3450 5900 3450
+Connection ~ 5900 3450
+Text HLabel 5250 3450 0    50   Output ~ 0
+ADIN1
+Wire Wire Line
+	5250 3450 5300 3450
+Connection ~ 5300 3450
+$Comp
+L ETH3CDAQ1:+18VF #PWR0112
+U 1 1 5FE8BDA6
+P 5850 3950
+F 0 "#PWR0112" H 5850 3800 50  0001 C CNN
+F 1 "+18VF" V 5850 4100 50  0000 L CNN
+F 2 "" H 5850 3950 50  0001 C CNN
+F 3 "" H 5850 3950 50  0001 C CNN
+	1    5850 3950
+	0    1    1    0
+$EndComp
+$Comp
+L ETH3CDAQ1:-18VF #PWR0113
+U 1 1 5FE8C7FC
+P 5350 3950
+F 0 "#PWR0113" H 5350 3800 50  0001 C CNN
+F 1 "-18VF" V 5350 4100 50  0000 L CNN
+F 2 "" H 5350 3950 50  0001 C CNN
+F 3 "" H 5350 3950 50  0001 C CNN
+	1    5350 3950
+	0    -1   -1   0
+$EndComp
 $EndSCHEMATC

Commit message: SDRAM works, thanks to the website https://medium.com/@pjinwoo123/stm32h7-external-sdram-evaluation-board-cc72444898d8 . Modified the code to work with SDRAM BANK2. SCPI library works.
Parts:
- renumbered J1001 to J701
Connections:
- net I2C_SCL: now reaches J701.2 (Pin_2)
- net I2C_SDA: now reaches J701.4 (Pin_4)
- net CANH: now reaches J701.5 (Pin_5)
- net CANL: now reaches J701.6 (Pin_6)
Changed lines of the file:
@@
 $Descr A4 11693 8268
 encoding utf-8
-Sheet 10 15
+Sheet 7 13
 Title ""
 Date ""
@@
 $EndDescr
 $Comp
-L Connector_Generic:Conn_02x10_Odd_Even J1001
+L Connector_Generic:Conn_02x10_Odd_Even J701
 U 1 1 60C21FE5
 P 5550 3450
-F 0 "J1001" H 5600 4067 50  0000 C CNN
+F 0 "J701" H 5600 4067 50  0000 C CNN
 F 1 "Conn_02x10_Odd_Even" H 5600 3976 50  0000 C CNN
 F 2 "Connector_PinSocket_2.54mm:PinSocket_2x10_P2.54mm_Vertical" H 5550 3450 50  0001 C CNN
@@
 $EndComp
 $Comp
-L power:GND #PWR01001
+L power:GND #PWR0701
 U 1 1 602209FD
 P 5350 3050
-F 0 "#PWR01001" H 5350 2800 50  0001 C CNN
+F 0 "#PWR0701" H 5350 2800 50  0001 C CNN
 F 1 "GND" V 5355 2922 50  0000 R CNN
 F 2 "" H 5350 3050 50  0001 C CNN
@@
 $EndComp
 $Comp
-L power:GND #PWR01002
+L power:GND #PWR0702
 U 1 1 60220E99
 P 5350 3150
-F 0 "#PWR01002" H 5350 2900 50  0001 C CNN
+F 0 "#PWR0702" H 5350 2900 50  0001 C CNN
 F 1 "GND" V 5355 3022 50  0000 R CNN
 F 2 "" H 5350 3150 50  0001 C CNN
@@
 $EndComp
 $Comp
-L power:GND #PWR01003
+L power:GND #PWR0703
 U 1 1 60222DE0
 P 5350 3350
-F 0 "#PWR01003" H 5350 3100 50  0001 C CNN
+F 0 "#PWR0703" H 5350 3100 50  0001 C CNN
 F 1 "GND" V 5355 3222 50  0000 R CNN
 F 2 "" H 5350 3350 50  0001 C CNN
@@
 $EndComp
 $Comp
-L power:GND #PWR01007
+L power:GND #PWR0707
 U 1 1 60223109
 P 5850 3350
-F 0 "#PWR01007" H 5850 3100 50  0001 C CNN
+F 0 "#PWR0707" H 5850 3100 50  0001 C CNN
 F 1 "GND" V 5855 3222 50  0000 R CNN
 F 2 "" H 5850 3350 50  0001 C CNN
@@
 $EndComp
 $Comp
-L power:GND #PWR01004
+L power:GND #PWR0704
 U 1 1 60223752
 P 5350 3650
-F 0 "#PWR01004" H 5350 3400 50  0001 C CNN
+F 0 "#PWR0704" H 5350 3400 50  0001 C CNN
 F 1 "GND" V 5355 3522 50  0000 R CNN
 F 2 "" H 5350 3650 50  0001 C CNN
@@
 $EndComp
 $Comp
-L power:GND #PWR01008
+L power:GND #PWR0708
 U 1 1 60223BA8
 P 5850 3650
-F 0 "#PWR01008" H 5850 3400 50  0001 C CNN
+F 0 "#PWR0708" H 5850 3400 50  0001 C CNN
 F 1 "GND" V 5855 3522 50  0000 R CNN
 F 2 "" H 5850 3650 50  0001 C CNN
@@
 $EndComp
 $Comp
-L power:+3.3V #PWR01005
+L power:+3.3V #PWR0705
 U 1 1 6022456D
 P 5350 3750
-F 0 "#PWR01005" H 5350 3600 50  0001 C CNN
+F 0 "#PWR0705" H 5350 3600 50  0001 C CNN
 F 1 "+3.3V" V 5350 3900 50  0000 L CNN
 F 2 "" H 5350 3750 50  0001 C CNN
@@
 $EndComp
 $Comp
-L power:+3.3V #PWR01009
+L power:+3.3V #PWR0709
 U 1 1 60224CD0
 P 5850 3750
-F 0 "#PWR01009" H 5850 3600 50  0001 C CNN
+F 0 "#PWR0709" H 5850 3600 50  0001 C CNN
 F 1 "+3.3V" V 5850 3900 50  0000 L CNN
 F 2 "" H 5850 3750 50  0001 C CNN
@@
 NoConn ~ 5350 3850
 $Comp
-L power:+5V #PWR01010
+L power:+5V #PWR0710
 U 1 1 6022B65E
 P 5850 3850
-F 0 "#PWR01010" H 5850 3700 50  0001 C CNN
+F 0 "#PWR0710" H 5850 3700 50  0001 C CNN
 F 1 "+5V" V 5850 4000 50  0000 L CNN
 F 2 "" H 5850 3850 50  0001 C CNN
@@
 Connection ~ 5300 3450
 $Comp
-L ETH3CDAQ1:+18VF #PWR01011
+L ETH3CDAQ1:+18VF #PWR0711
 U 1 1 5FE8BDA6
 P 5850 3950
-F 0 "#PWR01011" H 5850 3800 50  0001 C CNN
+F 0 "#PWR0711" H 5850 3800 50  0001 C CNN
 F 1 "+18VF" V 5850 4100 50  0000 L CNN
 F 2 "" H 5850 3950 50  0001 C CNN
@@
 $EndComp
 $Comp
-L ETH3CDAQ1:-18VF #PWR01006
+L ETH3CDAQ1:-18VF #PWR0706
 U 1 1 5FE8C7FC
 P 5350 3950
-F 0 "#PWR01006" H 5350 3800 50  0001 C CNN
+F 0 "#PWR0706" H 5350 3800 50  0001 C CNN
 F 1 "-18VF" V 5350 4100 50  0000 L CNN
 F 2 "" H 5350 3950 50  0001 C CNN
@@
 	0    -1   -1   0
 $EndComp
+Text HLabel 5350 3250 0    50   BiDi ~ 0
+CANH
+Text HLabel 5850 3250 2    50   BiDi ~ 0
+CANL
+Text HLabel 5850 3050 2    50   BiDi ~ 0
+I2C_SCL
+Text HLabel 5850 3150 2    50   BiDi ~ 0
+I2C_SDA
 $EndSCHEMATC
