File: hardware/project/ETH3CADC1/Connector.sch (KiCad schematic (older format))
At the start: 2 parts, among them J1301 Conn_02x02_Odd_Even, J1302 Conn_02x04_Odd_Even

Commit message: PCB layout
Connections:
- net EXT_TRIG: now reaches J1301.1 (Pin_1)
- net EXT_TRIG: now also J1301.2 (Pin_2)
- net GND_TRIG: now reaches J1301.3 (Pin_3)
- net GND_TRIG: now also J1301.4 (Pin_4)
- net Earth: now reaches J1302.1 (Pin_1)
- net Earth: now also J1302.2 (Pin_2), J1302.7 (Pin_7), J1302.8 (Pin_8)
- net RX+: now reaches J1302.3 (Pin_3)
- net TX+: now reaches J1302.4 (Pin_4)
- net RX-: now reaches J1302.5 (Pin_5)
- net TX-: now reaches J1302.6 (Pin_6)
Other:
- moved on the sheet: J1302
Changed lines of the file:
@@
 $Descr A4 11693 8268
 encoding utf-8
-Sheet 13 13
+Sheet 13 15
 Title ""
 Date ""
@@
 L Connector_Generic:Conn_02x04_Odd_Even J1302
 U 1 1 60F3B522
-P 5450 2250
-F 0 "J1302" H 5500 2567 50  0000 C CNN
-F 1 "Conn_02x04_Odd_Even" H 5500 2476 50  0000 C CNN
-F 2 "Connector_PinSocket_2.54mm:PinSocket_2x04_P2.54mm_Vertical" H 5450 2250 50  0001 C CNN
-F 3 "~" H 5450 2250 50  0001 C CNN
-	1    5450 2250
+P 5650 2250
+F 0 "J1302" H 5700 2567 50  0000 C CNN
+F 1 "Conn_02x04_Odd_Even" H 5700 2476 50  0000 C CNN
+F 2 "Connector_PinSocket_2.54mm:PinSocket_2x04_P2.54mm_Vertical" H 5650 2250 50  0001 C CNN
+F 3 "~" H 5650 2250 50  0001 C CNN
+	1    5650 2250
 	1    0    0    -1
 $EndComp
+Text HLabel 3850 2250 0    50   BiDi ~ 0
+EXT_TRIG
+Text HLabel 4350 2250 2    50   BiDi ~ 0
+EXT_TRIG
+$Comp
+L ETH3CDAQ1:GND_TRIG #PWR0118
+U 1 1 5FDB7CC9
+P 3850 2350
+F 0 "#PWR0118" H 3850 2100 50  0001 C CNN
+F 1 "GND_TRIG" V 3855 2222 50  0000 R CNN
+F 2 "" H 3850 2350 50  0001 C CNN
+F 3 "" H 3850 2350 50  0001 C CNN
+	1    3850 2350
+	0    1    1    0
+$EndComp
+$Comp
+L ETH3CDAQ1:GND_TRIG #PWR0119
+U 1 1 5FDB7FF2
+P 4350 2350
+F 0 "#PWR0119" H 4350 2100 50  0001 C CNN
+F 1 "GND_TRIG" V 4355 2222 50  0000 R CNN
+F 2 "" H 4350 2350 50  0001 C CNN
+F 3 "" H 4350 2350 50  0001 C CNN
+	1    4350 2350
+	0    -1   -1   0
+$EndComp
+$Comp
+L power:Earth #PWR0120
+U 1 1 5FDBA93E
+P 5450 2150
+F 0 "#PWR0120" H 5450 1900 50  0001 C CNN
+F 1 "Earth" H 5450 2000 50  0001 C CNN
+F 2 "" H 5450 2150 50  0001 C CNN
+F 3 "~" H 5450 2150 50  0001 C CNN
+	1    5450 2150
+	0    1    1    0
+$EndComp
+$Comp
+L power:Earth #PWR0121
+U 1 1 5FDBADF8
+P 5450 2450
+F 0 "#PWR0121" H 5450 2200 50  0001 C CNN
+F 1 "Earth" H 5450 2300 50  0001 C CNN
+F 2 "" H 5450 2450 50  0001 C CNN
+F 3 "~" H 5450 2450 50  0001 C CNN
+	1    5450 2450
+	0    1    1    0
+$EndComp
+$Comp
+L power:Earth #PWR0122
+U 1 1 5FDBB1CB
+P 5950 2450
+F 0 "#PWR0122" H 5950 2200 50  0001 C CNN
+F 1 "Earth" H 5950 2300 50  0001 C CNN
+F 2 "" H 5950 2450 50  0001 C CNN
+F 3 "~" H 5950 2450 50  0001 C CNN
+	1    5950 2450
+	0    -1   -1   0
+$EndComp
+$Comp
+L power:Earth #PWR0123
+U 1 1 5FDBB5A5
+P 5950 2150
+F 0 "#PWR0123" H 5950 1900 50  0001 C CNN
+F 1 "Earth" H 5950 2000 50  0001 C CNN
+F 2 "" H 5950 2150 50  0001 C CNN
+F 3 "~" H 5950 2150 50  0001 C CNN
+	1    5950 2150
+	0    -1   -1   0
+$EndComp
+Text HLabel 5950 2250 2    50   BiDi ~ 0
+TX+
+Text HLabel 5950 2350 2    50   BiDi ~ 0
+TX-
+Text HLabel 5450 2250 0    50   BiDi ~ 0
+RX+
+Text HLabel 5450 2350 0    50   BiDi ~ 0
+RX-
 $EndSCHEMATC

Commit message: SDRAM works, thanks to the website https://medium.com/@pjinwoo123/stm32h7-external-sdram-evaluation-board-cc72444898d8 . Modified the code to work with SDRAM BANK2. SCPI library works.
Parts:
- renumbered J1301 to J801, J1302 to J802
Changed lines of the file:
@@
 $Descr A4 11693 8268
 encoding utf-8
-Sheet 13 15
+Sheet 13 13
 Title ""
 Date ""
@@
 $EndDescr
 $Comp
-L Connector_Generic:Conn_02x02_Odd_Even J1301
+L Connector_Generic:Conn_02x02_Odd_Even J801
 U 1 1 60F397AF
 P 4050 2250
-F 0 "J1301" H 4100 2467 50  0000 C CNN
+F 0 "J801" H 4100 2467 50  0000 C CNN
 F 1 "Conn_02x02_Odd_Even" H 4100 2376 50  0000 C CNN
 F 2 "Connector_PinSocket_2.54mm:PinSocket_2x02_P2.54mm_Vertical" H 4050 2250 50  0001 C CNN
@@
 $EndComp
 $Comp
-L Connector_Generic:Conn_02x04_Odd_Even J1302
+L Connector_Generic:Conn_02x04_Odd_Even J802
 U 1 1 60F3B522
 P 5650 2250
-F 0 "J1302" H 5700 2567 50  0000 C CNN
+F 0 "J802" H 5700 2567 50  0000 C CNN
 F 1 "Conn_02x04_Odd_Even" H 5700 2476 50  0000 C CNN
 F 2 "Connector_PinSocket_2.54mm:PinSocket_2x04_P2.54mm_Vertical" H 5650 2250 50  0001 C CNN
@@
 EXT_TRIG
 $Comp
-L ETH3CDAQ1:GND_TRIG #PWR01301
+L ETH3CDAQ1:GND_TRIG #PWR0801
 U 1 1 5FDB7CC9
 P 3850 2350
-F 0 "#PWR01301" H 3850 2100 50  0001 C CNN
+F 0 "#PWR0801" H 3850 2100 50  0001 C CNN
 F 1 "GND_TRIG" V 3855 2222 50  0000 R CNN
 F 2 "" H 3850 2350 50  0001 C CNN
@@
 $EndComp
 $Comp
-L ETH3CDAQ1:GND_TRIG #PWR01302
+L ETH3CDAQ1:GND_TRIG #PWR0802
 U 1 1 5FDB7FF2
 P 4350 2350
-F 0 "#PWR01302" H 4350 2100 50  0001 C CNN
+F 0 "#PWR0802" H 4350 2100 50  0001 C CNN
 F 1 "GND_TRIG" V 4355 2222 50  0000 R CNN
 F 2 "" H 4350 2350 50  0001 C CNN
@@
 $EndComp
 $Comp
-L power:Earth #PWR01303
+L power:Earth #PWR0803
 U 1 1 5FDBA93E
 P 5450 2150
-F 0 "#PWR01303" H 5450 1900 50  0001 C CNN
+F 0 "#PWR0803" H 5450 1900 50  0001 C CNN
 F 1 "Earth" H 5450 2000 50  0001 C CNN
 F 2 "" H 5450 2150 50  0001 C CNN
@@
 $EndComp
 $Comp
-L power:Earth #PWR01304
+L power:Earth #PWR0804
 U 1 1 5FDBADF8
 P 5450 2450
-F 0 "#PWR01304" H 5450 2200 50  0001 C CNN
+F 0 "#PWR0804" H 5450 2200 50  0001 C CNN
 F 1 "Earth" H 5450 2300 50  0001 C CNN
 F 2 "" H 5450 2450 50  0001 C CNN
@@
 $EndComp
 $Comp
-L power:Earth #PWR01306
+L power:Earth #PWR0806
 U 1 1 5FDBB1CB
 P 5950 2450
-F 0 "#PWR01306" H 5950 2200 50  0001 C CNN
+F 0 "#PWR0806" H 5950 2200 50  0001 C CNN
 F 1 "Earth" H 5950 2300 50  0001 C CNN
 F 2 "" H 5950 2450 50  0001 C CNN
@@
 $EndComp
 $Comp
-L power:Earth #PWR01305
+L power:Earth #PWR0805
 U 1 1 5FDBB5A5
 P 5950 2150
-F 0 "#PWR01305" H 5950 1900 50  0001 C CNN
+F 0 "#PWR0805" H 5950 1900 50  0001 C CNN
 F 1 "Earth" H 5950 2000 50  0001 C CNN
 F 2 "" H 5950 2150 50  0001 C CNN
