File: hardware/project/ETH3CADC1/FPGA2.sch (KiCad schematic (older format))
At the start: 28 parts, among them J1201 Conn_02x05_Odd_Even, U1201 ICE40UP5K-SG48ITR, U1202 W25Q32JVSS, U1203 AP2127K-1.2, X1201 ASAAIG-40.000MHZ

Commit message: Development
Parts:
- removed C1201, C1202, C1203, C1204, C1205, C1208, C1209, C1211: 100n, Capacitor_SMD:C_0402_1005Metric_Pad0.74x0.62mm_HandSolder, symbol Device:C
- removed C1206, C1207, C1210, C1212: 4u7, Capacitor_SMD:C_0603_1608Metric_Pad1.08x0.95mm_HandSolder, symbol Device:C
- removed D1201: CDBU0520, Diode_SMD:D_SOD-523, symbol Device:D
- removed J1201: Conn_02x05_Odd_Even, Connector_PinHeader_1.27mm:PinHeader_2x05_P1.27mm_Vertical, symbol Connector_Generic:Conn_02x05_Odd_Even
- removed R1201: 22, Resistor_SMD:R_0402_1005Metric_Pad0.72x0.64mm_HandSolder, symbol Device:R
- removed R1202, R1203, R1204, R1205, R1207, R1208, R1209: 10k, Resistor_SMD:R_0402_1005Metric_Pad0.72x0.64mm_HandSolder, symbol Device:R
- removed R1206: NC, Resistor_SMD:R_0402_1005Metric_Pad0.72x0.64mm_HandSolder, symbol Device:R
- removed R1210: 100, Resistor_SMD:R_0402_1005Metric_Pad0.72x0.64mm_HandSolder, symbol Device:R
- removed U1201: ICE40UP5K-SG48ITR, Package_DFN_QFN:QFN-48-1EP_7x7mm_P0.5mm_EP5.6x5.6mm_ThermalVias, symbol FPGA_Lattice:ICE40UP5K-SG48ITR
- removed U1202: W25Q32JVSS, Package_SO:SOIC-8_5.23x5.23mm_P1.27mm, symbol Memory_Flash:W25Q32JVSS
- removed U1203: AP2127K-1.2, Package_TO_SOT_SMD:SOT-23-5, symbol Regulator_Linear:AP2127K-1.2
- removed X1201: ASAAIG-40.000MHZ, ETH3CDAQ1:ASAAIG, symbol ETH3CDAQ1:ASAAIG-xxx
- added C1301, C1302, C1303, C1304, C1305, C1308, C1309, C1311: 100n, Capacitor_SMD:C_0402_1005Metric_Pad0.74x0.62mm_HandSolder, symbol Device:C
- added C1306, C1307, C1310, C1312: 4u7, Capacitor_SMD:C_0603_1608Metric_Pad1.08x0.95mm_HandSolder, symbol Device:C
- added D1301: CDBU0520, Diode_SMD:D_SOD-523, symbol Device:D
- added J1301: Conn_02x05_Odd_Even, Connector_PinHeader_1.27mm:PinHeader_2x05_P1.27mm_Vertical, symbol Connector_Generic:Conn_02x05_Odd_Even
- added R1301: 22, Resistor_SMD:R_0402_1005Metric_Pad0.72x0.64mm_HandSolder, symbol Device:R
- added R1302, R1303, R1305, R1306, R1307, R1308, R1309: 10k, Resistor_SMD:R_0402_1005Metric_Pad0.72x0.64mm_HandSolder, symbol Device:R
- added R1304: NC, Resistor_SMD:R_0402_1005Metric_Pad0.72x0.64mm_HandSolder, symbol Device:R
- added R1310: 100, Resistor_SMD:R_0402_1005Metric_Pad0.72x0.64mm_HandSolder, symbol Device:R
- added U1301: ICE40UP5K-SG48ITR, Package_DFN_QFN:QFN-48-1EP_7x7mm_P0.5mm_EP5.6x5.6mm_ThermalVias, symbol FPGA_Lattice:ICE40UP5K-SG48ITR
- added U1302: W25Q32JVSS, Package_SO:SOIC-8_5.23x5.23mm_P1.27mm, symbol Memory_Flash:W25Q32JVSS
- added U1303: AP2127K-1.2, Package_TO_SOT_SMD:SOT-23-5, symbol Regulator_Linear:AP2127K-1.2
- added X1301: ASAAIG-40.000MHZ, ETH3CDAQ1:ASAAIG, symbol ETH3CDAQ1:ASAAIG-xxx
Connections:
- net +3V3: now also C1301.1, C1302.1, C1303.1, C1304.1, C1305.1, C1306.1, C1308.1, D1301.2 (A), R1302.1, R1303.1, R1304.1, R1305.1, R1306.1, R1307.1, R1308.1, R1309.1, U1301.1 (VCCIO_2), U1301.22 (SPI_VCCIO1), U1301.33 (VCCIO_0), U1302.8 (VCC), U1303.1 (VIN), U1303.3 (EN), X1301.4 (VDD)
- net CODE1: now also R1304.2, U1301.2 (IOB_6a)
- net CODE2: now also R1306.2, U1301.3 (IOB_9b)
- net FPGA_CLK: now also R1301.1, U1301.35 (IOT_46b_G0)
- net GND: now also C1301.2, C1302.2, C1303.2, C1304.2, C1305.2, C1306.2, C1307.2, C1308.2, C1309.2, C1310.2, C1311.2, C1312.2, J1301.2 (Pin_2), U1301.49 (GND), U1302.4 (GND), U1303.2 (GND), X1301.2 (GND)
- net iCE_CDONE: now also J1301.5 (Pin_5), R1307.2, U1301.7 (CDONE)
- net iCE_CRESET: now also J1301.6 (Pin_6), R1302.2, U1301.8 (~CRESET)
- net iCE_MISO: now also J1301.8 (Pin_8), U1301.14 (IOB_32a_SPI_SO), U1302.5 (DI(IO0))
- net iCE_MOSI: now also J1301.7 (Pin_7), U1301.17 (IOB_33b_SPI_SI), U1302.2 (DO(IO1))
- net iCE_SCK: now also J1301.9 (Pin_9), R1305.2, U1301.15 (IOB_34a_SPI_SCK), U1302.6 (CLK)
- net iCE_SSn: now also J1301.10 (Pin_10), R1303.2, U1301.16 (IOB_35b_SPI_SS), U1302.1 (~CS)
- new net: C1312.1, D1301.1 (K), U1301.24 (VPP_2V5)
- new net: C1309.1, C1310.1, R1310.1, U1301.29 (VCCPLL)
- new net: C1307.1, C1311.1, R1310.2, U1301.30 (VCC), U1301.5 (VCC), U1303.5 (VOUT)
- new net: R1301.2, X1301.3 (OUT)
- new net: R1308.2, U1302.3 (IO2)
- new net: R1309.2, U1302.7 (IO3)
- new net ADC_COMP2: U1301.47 (IOB_2a)
- new net FGPA2_AD_ID: U1301.44 (IOB_3b_G6)
- new net FGPA2_AD_IRN: U1301.43 (IOT_49a)
- new net FGPA2_AD_IRP: U1301.45 (IOB_5b)
- new net FGPA2_AD_VRH: U1301.37 (IOT_45a_G1)
- new net FGPA2_MISO: U1301.20 (IOB_25b_G3)
- new net FGPA2_MOSI: U1301.19 (IOB_29b)
- new net FGPA2_SCLK: U1301.21 (IOB_23b)
- new net FGPA2_nSS: U1301.23 (IOT_37a)
- new net FPGA2_AD_IIN: U1301.42 (IOT_51a)
- new net FPGA2_MUX_ADIN: U1301.38 (IOT_50b)
- new net FPGA2_MUX_GND: U1301.41 (RGB2)
- new net FPGA2_MUX_N7V: U1301.39 (RGB0)
- new net FPGA2_MUX_P10V: U1301.40 (RGB1)
- new net FPGA2_UART2_RX: U1301.26 (IOT_39a)
- new net FPGA2_UART2_TX: U1301.25 (IOT_36b)

Commit message: Software development.
Connections:
- net FPGA2_CONV_STR: now reaches U1301.12 (IOB_22b)
- no-connect marks 20 -> 19
Changed lines of the file:
@@
 $Descr A4 11693 8268
 encoding utf-8
-Sheet 14 17
-Title ""
-Date ""
+Sheet 13 17
+Title "FPGA 2"
+Date "2021-01-31"
 Rev ""
 Comp ""
@@
 NoConn ~ 3200 2600
 NoConn ~ 3200 2300
-NoConn ~ 3200 2100
 NoConn ~ 3200 1800
 NoConn ~ 3200 1700
@@
 NoConn ~ 3200 1900
 NoConn ~ 3200 2000
+Text HLabel 3150 2100 0    50   BiDi ~ 0
+FPGA2_CONV_STR
+Wire Wire Line
+	3150 2100 3200 2100
 $EndSCHEMATC
