File: hardware/project/ETH3CADC1/FPGA3.sch (KiCad schematic (older format))
At the start: 28 parts, among them J1201 Conn_02x05_Odd_Even, U1201 ICE40UP5K-SG48ITR, U1202 W25Q32JVSS, U1203 AP2127K-1.2, X1201 ASAAIG-40.000MHZ

Commit message: Development
Parts:
- removed C1201, C1202, C1203, C1204, C1205, C1208, C1209, C1211: 100n, Capacitor_SMD:C_0402_1005Metric_Pad0.74x0.62mm_HandSolder, symbol Device:C
- removed C1206, C1207, C1210, C1212: 4u7, Capacitor_SMD:C_0603_1608Metric_Pad1.08x0.95mm_HandSolder, symbol Device:C
- removed D1201: CDBU0520, Diode_SMD:D_SOD-523, symbol Device:D
- removed J1201: Conn_02x05_Odd_Even, Connector_PinHeader_1.27mm:PinHeader_2x05_P1.27mm_Vertical, symbol Connector_Generic:Conn_02x05_Odd_Even
- removed R1201: 22, Resistor_SMD:R_0402_1005Metric_Pad0.72x0.64mm_HandSolder, symbol Device:R
- removed R1202, R1203, R1204, R1205, R1207, R1208, R1209: 10k, Resistor_SMD:R_0402_1005Metric_Pad0.72x0.64mm_HandSolder, symbol Device:R
- removed R1206: NC, Resistor_SMD:R_0402_1005Metric_Pad0.72x0.64mm_HandSolder, symbol Device:R
- removed R1210: 100, Resistor_SMD:R_0402_1005Metric_Pad0.72x0.64mm_HandSolder, symbol Device:R
- removed U1201: ICE40UP5K-SG48ITR, Package_DFN_QFN:QFN-48-1EP_7x7mm_P0.5mm_EP5.6x5.6mm_ThermalVias, symbol FPGA_Lattice:ICE40UP5K-SG48ITR
- removed U1202: W25Q32JVSS, Package_SO:SOIC-8_5.23x5.23mm_P1.27mm, symbol Memory_Flash:W25Q32JVSS
- removed U1203: AP2127K-1.2, Package_TO_SOT_SMD:SOT-23-5, symbol Regulator_Linear:AP2127K-1.2
- removed X1201: ASAAIG-40.000MHZ, ETH3CDAQ1:ASAAIG, symbol ETH3CDAQ1:ASAAIG-xxx
- added C1601, C1602, C1603, C1604, C1605, C1608, C1609, C1611: 100n, Capacitor_SMD:C_0402_1005Metric_Pad0.74x0.62mm_HandSolder, symbol Device:C
- added C1606, C1607, C1610, C1612: 4u7, Capacitor_SMD:C_0603_1608Metric_Pad1.08x0.95mm_HandSolder, symbol Device:C
- added D1601: CDBU0520, Diode_SMD:D_SOD-523, symbol Device:D
- added J1601: Conn_02x05_Odd_Even, Connector_PinHeader_1.27mm:PinHeader_2x05_P1.27mm_Vertical, symbol Connector_Generic:Conn_02x05_Odd_Even
- added R1601: 22, Resistor_SMD:R_0402_1005Metric_Pad0.72x0.64mm_HandSolder, symbol Device:R
- added R1602, R1603, R1604, R1605, R1606, R1607, R1608, R1609: 10k, Resistor_SMD:R_0402_1005Metric_Pad0.72x0.64mm_HandSolder, symbol Device:R
- added R1610: 100, Resistor_SMD:R_0402_1005Metric_Pad0.72x0.64mm_HandSolder, symbol Device:R
- added U1601: ICE40UP5K-SG48ITR, Package_DFN_QFN:QFN-48-1EP_7x7mm_P0.5mm_EP5.6x5.6mm_ThermalVias, symbol FPGA_Lattice:ICE40UP5K-SG48ITR
- added U1602: W25Q32JVSS, Package_SO:SOIC-8_5.23x5.23mm_P1.27mm, symbol Memory_Flash:W25Q32JVSS
- added U1603: AP2127K-1.2, Package_TO_SOT_SMD:SOT-23-5, symbol Regulator_Linear:AP2127K-1.2
- added X1601: ASAAIG-40.000MHZ, ETH3CDAQ1:ASAAIG, symbol ETH3CDAQ1:ASAAIG-xxx
Connections:
- net +3V3: now also C1601.1, C1602.1, C1603.1, C1604.1, C1605.1, C1606.1, C1608.1, D1601.2 (A), R1602.1, R1603.1, R1604.1, R1605.1, R1606.1, R1607.1, R1608.1, R1609.1, U1601.1 (VCCIO_2), U1601.22 (SPI_VCCIO1), U1601.33 (VCCIO_0), U1602.8 (VCC), U1603.1 (VIN), U1603.3 (EN), X1601.4 (VDD)
- net CODE1: now also R1604.2, U1601.2 (IOB_6a)
- net CODE2: now also R1606.2, U1601.3 (IOB_9b)
- net FPGA_CLK: now also R1601.1, U1601.35 (IOT_46b_G0)
- net GND: now also C1601.2, C1602.2, C1603.2, C1604.2, C1605.2, C1606.2, C1607.2, C1608.2, C1609.2, C1610.2, C1611.2, C1612.2, J1601.2 (Pin_2), U1601.49 (GND), U1602.4 (GND), U1603.2 (GND), X1601.2 (GND)
- net iCE_CDONE: now also J1601.5 (Pin_5), R1607.2, U1601.7 (CDONE)
- net iCE_CRESET: now also J1601.6 (Pin_6), R1602.2, U1601.8 (~CRESET)
- net iCE_MISO: now also J1601.8 (Pin_8), U1601.14 (IOB_32a_SPI_SO), U1602.5 (DI(IO0))
- net iCE_MOSI: now also J1601.7 (Pin_7), U1601.17 (IOB_33b_SPI_SI), U1602.2 (DO(IO1))
- net iCE_SCK: now also J1601.9 (Pin_9), R1605.2, U1601.15 (IOB_34a_SPI_SCK), U1602.6 (CLK)
- net iCE_SSn: now also J1601.10 (Pin_10), R1603.2, U1601.16 (IOB_35b_SPI_SS), U1602.1 (~CS)
- new net: C1612.1, D1601.1 (K), U1601.24 (VPP_2V5)
- new net: C1609.1, C1610.1, R1610.1, U1601.29 (VCCPLL)
- new net: C1607.1, C1611.1, R1610.2, U1601.30 (VCC), U1601.5 (VCC), U1603.5 (VOUT)
- new net: R1608.2, U1602.3 (IO2)
- new net: R1609.2, U1602.7 (IO3)
- new net: R1601.2, X1601.3 (OUT)
- new net ADC_COMP3: U1601.47 (IOB_2a)
- new net FGPA3_AD_ID: U1601.44 (IOB_3b_G6)
- new net FGPA3_AD_IRN: U1601.43 (IOT_49a)
- new net FGPA3_AD_IRP: U1601.45 (IOB_5b)
- new net FGPA3_AD_VRH: U1601.37 (IOT_45a_G1)
- new net FGPA3_MISO: U1601.20 (IOB_25b_G3)
- new net FGPA3_MOSI: U1601.19 (IOB_29b)
- new net FGPA3_SCLK: U1601.21 (IOB_23b)
- new net FGPA3_nSS: U1601.23 (IOT_37a)
- new net FPGA3_AD_IIN: U1601.42 (IOT_51a)
- new net FPGA3_MUX_ADIN: U1601.38 (IOT_50b)
- new net FPGA3_MUX_GND: U1601.41 (RGB2)
- new net FPGA3_MUX_N7V: U1601.39 (RGB0)
- new net FPGA3_MUX_P10V: U1601.40 (RGB1)
- new net FPGA3_UART2_RX: U1601.26 (IOT_39a)
- new net FPGA3_UART2_TX: U1601.25 (IOT_36b)

Commit message: Software development.
Connections:
- net FPGA3_CONV_STR: now reaches U1601.12 (IOB_22b)
- no-connect marks 20 -> 19
Changed lines of the file:
@@
 encoding utf-8
 Sheet 16 17
-Title ""
-Date ""
+Title "FPGA 3"
+Date "2021-01-31"
 Rev ""
 Comp ""
@@
 NoConn ~ 3200 2600
 NoConn ~ 3200 2300
-NoConn ~ 3200 2100
 NoConn ~ 3200 1800
 NoConn ~ 3200 1700
@@
 NoConn ~ 3200 1900
 NoConn ~ 3200 2000
+Text HLabel 3150 2100 0    50   BiDi ~ 0
+FPGA3_CONV_STR
+Wire Wire Line
+	3150 2100 3200 2100
 $EndSCHEMATC
