File: hardware/project/ETH3CADC1/SDRAM.sch (KiCad schematic (older format))
At the start: 8 parts, among them U1401 MT48LC16M16A2P-6A

Commit message: SDRAM works, thanks to the website https://medium.com/@pjinwoo123/stm32h7-external-sdram-evaluation-board-cc72444898d8 . Modified the code to work with SDRAM BANK2. SCPI library works.
Parts:
- renumbered C1401 to C901, C1402 to C902, C1403 to C903, C1404 to C904, C1405 to C905, C1406 to C906, C1407 to C907, U1401 to U901
Changed lines of the file:
@@
 $Descr A4 11693 8268
 encoding utf-8
-Sheet 14 15
+Sheet 14 13
 Title "SDRAM"
 Date "2020-03-07"
@@
 D[0..15]
 $Comp
-L Device:C C1401
+L Device:C C901
 U 1 1 5F12988C
 P 1000 7250
-F 0 "C1401" H 1115 7296 50  0000 L CNN
+F 0 "C901" H 1115 7296 50  0000 L CNN
 F 1 "100n" H 1115 7205 50  0000 L CNN
 F 2 "Capacitor_SMD:C_0402_1005Metric_Pad0.74x0.62mm_HandSolder" H 1038 7100 50  0001 C CNN
@@
 $EndComp
 $Comp
-L Device:C C1402
+L Device:C C902
 U 1 1 5F12BD5A
 P 1500 7250
-F 0 "C1402" H 1615 7296 50  0000 L CNN
+F 0 "C902" H 1615 7296 50  0000 L CNN
 F 1 "100n" H 1615 7205 50  0000 L CNN
 F 2 "Capacitor_SMD:C_0402_1005Metric_Pad0.74x0.62mm_HandSolder" H 1538 7100 50  0001 C CNN
@@
 $EndComp
 $Comp
-L Device:C C1403
+L Device:C C903
 U 1 1 5F12CAA5
 P 2000 7250
-F 0 "C1403" H 2115 7296 50  0000 L CNN
+F 0 "C903" H 2115 7296 50  0000 L CNN
 F 1 "100n" H 2115 7205 50  0000 L CNN
 F 2 "Capacitor_SMD:C_0402_1005Metric_Pad0.74x0.62mm_HandSolder" H 2038 7100 50  0001 C CNN
@@
 $EndComp
 $Comp
-L Device:C C1404
+L Device:C C904
 U 1 1 5F12CAAB
 P 2500 7250
-F 0 "C1404" H 2615 7296 50  0000 L CNN
+F 0 "C904" H 2615 7296 50  0000 L CNN
 F 1 "100n" H 2615 7205 50  0000 L CNN
 F 2 "Capacitor_SMD:C_0402_1005Metric_Pad0.74x0.62mm_HandSolder" H 2538 7100 50  0001 C CNN
@@
 $EndComp
 $Comp
-L Device:C C1405
+L Device:C C905
 U 1 1 5F12F1B4
 P 3000 7250
-F 0 "C1405" H 3115 7296 50  0000 L CNN
+F 0 "C905" H 3115 7296 50  0000 L CNN
 F 1 "100n" H 3115 7205 50  0000 L CNN
 F 2 "Capacitor_SMD:C_0402_1005Metric_Pad0.74x0.62mm_HandSolder" H 3038 7100 50  0001 C CNN
@@
 $EndComp
 $Comp
-L Device:C C1406
+L Device:C C906
 U 1 1 5F12F1BA
 P 3500 7250
-F 0 "C1406" H 3615 7296 50  0000 L CNN
+F 0 "C906" H 3615 7296 50  0000 L CNN
 F 1 "100n" H 3615 7205 50  0000 L CNN
 F 2 "Capacitor_SMD:C_0402_1005Metric_Pad0.74x0.62mm_HandSolder" H 3538 7100 50  0001 C CNN
@@
 $EndComp
 $Comp
-L Device:C C1407
+L Device:C C907
 U 1 1 5F12F1C0
 P 4000 7250
-F 0 "C1407" H 4115 7296 50  0000 L CNN
+F 0 "C907" H 4115 7296 50  0000 L CNN
 F 1 "100n" H 4115 7205 50  0000 L CNN
 F 2 "Capacitor_SMD:C_0402_1005Metric_Pad0.74x0.62mm_HandSolder" H 4038 7100 50  0001 C CNN
@@
 	2500 7000 2500 7050
 $Comp
-L power:GND #PWR01402
+L power:GND #PWR0902
 U 1 1 6038237F
 P 2500 7500
-F 0 "#PWR01402" H 2500 7250 50  0001 C CNN
+F 0 "#PWR0902" H 2500 7250 50  0001 C CNN
 F 1 "GND" H 2505 7327 50  0000 C CNN
 F 2 "" H 2500 7500 50  0001 C CNN
@@
 $EndComp
 $Comp
-L power:GND #PWR01404
+L power:GND #PWR0904
 U 1 1 603828AC
 P 5650 4700
-F 0 "#PWR01404" H 5650 4450 50  0001 C CNN
+F 0 "#PWR0904" H 5650 4450 50  0001 C CNN
 F 1 "GND" H 5655 4527 50  0000 C CNN
 F 2 "" H 5650 4700 50  0001 C CNN
@@
 $EndComp
 $Comp
-L power:+3.3V #PWR01403
+L power:+3.3V #PWR0903
 U 1 1 60383841
 P 5650 1700
-F 0 "#PWR01403" H 5650 1550 50  0001 C CNN
+F 0 "#PWR0903" H 5650 1550 50  0001 C CNN
 F 1 "+3.3V" H 5665 1873 50  0000 C CNN
 F 2 "" H 5650 1700 50  0001 C CNN
@@
 $EndComp
 $Comp
-L power:+3.3V #PWR01401
+L power:+3.3V #PWR0901
 U 1 1 60384354
 P 2500 7000
-F 0 "#PWR01401" H 2500 6850 50  0001 C CNN
+F 0 "#PWR0901" H 2500 6850 50  0001 C CNN
 F 1 "+3.3V" H 2515 7173 50  0000 C CNN
 F 2 "" H 2500 7000 50  0001 C CNN
@@
 $EndComp
 $Comp
-L ETH3CDAQ1:MT48LC16M16A2P-6A U1401
+L ETH3CDAQ1:MT48LC16M16A2P-6A U901
 U 1 1 5FD364EC
 P 5650 3200
-F 0 "U1401" H 6400 4550 50  0000 C CNN
+F 0 "U901" H 6400 4550 50  0000 C CNN
 F 1 "MT48LC16M16A2P-6A" H 6400 4450 50  0000 C CNN
 F 2 "ETH3CDAQ1:TSSOP-54" H 5650 3200 50  0001 C CNN
