File: hardware/project/ETH3CADC1/Trigger.sch (KiCad schematic (older format))
At the start: 22 parts, among them U701 TXB0104PW, U702 ADuM5402, U703 74AC125

Commit message: PCB layout
Parts:
- C702, C705, C707: footprint Capacitor_SMD:C_0603_1608Metric_Pad1.08x0.95mm_HandSolder -> Capacitor_SMD:C_0402_1005Metric_Pad0.74x0.62mm_HandSolder
- C709: footprint Capacitor_SMD:C_0402_1005Metric_Pad0.74x0.62mm_HandSolder -> Capacitor_SMD:C_0603_1608Metric_Pad1.08x0.95mm_HandSolder
- R702, R703, R704, R705, R706: footprint Resistor_SMD:R_0402_1005Metric_Pad0.72x0.64mm_HandSolder -> Resistor_SMD:R_0603_1608Metric_Pad0.98x0.95mm_HandSolder
Changed lines of the file:
@@
 $Descr A4 11693 8268
 encoding utf-8
-Sheet 7 13
+Sheet 7 15
 Title "Trigger"
 Date "2020-03-07"
@@
 F 0 "C709" H 9215 5696 50  0000 L CNN
 F 1 "47p" H 9215 5605 50  0000 L CNN
-F 2 "Capacitor_SMD:C_0402_1005Metric_Pad0.74x0.62mm_HandSolder" H 9138 5500 50  0001 C CNN
+F 2 "Capacitor_SMD:C_0603_1608Metric_Pad1.08x0.95mm_HandSolder" H 9138 5500 50  0001 C CNN
 F 3 "~" H 9100 5650 50  0001 C CNN
 	1    9100 5650
@@
 F 0 "R706" H 9170 5996 50  0000 L CNN
 F 1 "51R1" H 9170 5905 50  0000 L CNN
-F 2 "Resistor_SMD:R_0402_1005Metric_Pad0.72x0.64mm_HandSolder" V 9030 5950 50  0001 C CNN
+F 2 "Resistor_SMD:R_0603_1608Metric_Pad0.98x0.95mm_HandSolder" V 9030 5950 50  0001 C CNN
 F 3 "~" H 9100 5950 50  0001 C CNN
 	1    9100 5950
@@
 F 0 "R705" V 8093 5450 50  0000 C CNN
 F 1 "47" V 8184 5450 50  0000 C CNN
-F 2 "Resistor_SMD:R_0402_1005Metric_Pad0.72x0.64mm_HandSolder" V 8230 5450 50  0001 C CNN
+F 2 "Resistor_SMD:R_0603_1608Metric_Pad0.98x0.95mm_HandSolder" V 8230 5450 50  0001 C CNN
 F 3 "~" H 8300 5450 50  0001 C CNN
 	1    8300 5450
@@
 F 0 "R704" H 8020 4446 50  0000 L CNN
 F 1 "1k" H 8020 4355 50  0000 L CNN
-F 2 "Resistor_SMD:R_0402_1005Metric_Pad0.72x0.64mm_HandSolder" V 7880 4400 50  0001 C CNN
+F 2 "Resistor_SMD:R_0603_1608Metric_Pad0.98x0.95mm_HandSolder" V 7880 4400 50  0001 C CNN
 F 3 "~" H 7950 4400 50  0001 C CNN
 	1    7950 4400
@@
 F 0 "R702" V 5893 5450 50  0000 C CNN
 F 1 "14k7" V 5984 5450 50  0000 C CNN
-F 2 "Resistor_SMD:R_0402_1005Metric_Pad0.72x0.64mm_HandSolder" V 6030 5450 50  0001 C CNN
+F 2 "Resistor_SMD:R_0603_1608Metric_Pad0.98x0.95mm_HandSolder" V 6030 5450 50  0001 C CNN
 F 3 "~" H 6100 5450 50  0001 C CNN
 	1    6100 5450
@@
 F 0 "C705" H 4465 1196 50  0000 L CNN
 F 1 "1u" H 4465 1105 50  0000 L CNN
-F 2 "Capacitor_SMD:C_0603_1608Metric_Pad1.08x0.95mm_HandSolder" H 4388 1000 50  0001 C CNN
+F 2 "Capacitor_SMD:C_0402_1005Metric_Pad0.74x0.62mm_HandSolder" H 4388 1000 50  0001 C CNN
 F 3 "~" H 4350 1150 50  0001 C CNN
 	1    4350 1150
@@
 F 0 "C707" H 5615 1196 50  0000 L CNN
 F 1 "1u" H 5615 1105 50  0000 L CNN
-F 2 "Capacitor_SMD:C_0603_1608Metric_Pad1.08x0.95mm_HandSolder" H 5538 1000 50  0001 C CNN
+F 2 "Capacitor_SMD:C_0402_1005Metric_Pad0.74x0.62mm_HandSolder" H 5538 1000 50  0001 C CNN
 F 3 "~" H 5500 1150 50  0001 C CNN
 	1    5500 1150
@@
 F 0 "C702" H 3015 1196 50  0000 L CNN
 F 1 "1u" H 3015 1105 50  0000 L CNN
-F 2 "Capacitor_SMD:C_0603_1608Metric_Pad1.08x0.95mm_HandSolder" H 2938 1000 50  0001 C CNN
+F 2 "Capacitor_SMD:C_0402_1005Metric_Pad0.74x0.62mm_HandSolder" H 2938 1000 50  0001 C CNN
 F 3 "~" H 2900 1150 50  0001 C CNN
 	1    2900 1150
@@
 F 0 "R703" V 6843 5450 50  0000 C CNN
 F 1 "100" V 6934 5450 50  0000 C CNN
-F 2 "Resistor_SMD:R_0402_1005Metric_Pad0.72x0.64mm_HandSolder" V 6980 5450 50  0001 C CNN
+F 2 "Resistor_SMD:R_0603_1608Metric_Pad0.98x0.95mm_HandSolder" V 6980 5450 50  0001 C CNN
 F 3 "~" H 7050 5450 50  0001 C CNN
 	1    7050 5450

Commit message: SDRAM works, thanks to the website https://medium.com/@pjinwoo123/stm32h7-external-sdram-evaluation-board-cc72444898d8 . Modified the code to work with SDRAM BANK2. SCPI library works.
Parts:
- renumbered C701 to C601, C702 to C602, C703 to C603, C704 to C604, C705 to C605, C706 to C606, C707 to C607, C708 to C608, C709 to C609, D701 to D601, D702 to D602, D703 to D603, L701 to L601, R701 to R601, R702 to R602, R703 to R603, R704 to R604, R705 to R605, R706 to R606, U701 to U601, U702 to U602, U703 to U603
