File: hardware/project/ETH3CADC1/VREF.sch (KiCad schematic (older format))
At the start: 16 parts, among them Q301 MMBTA55, Q302 BC847, U301 LT1021-7, U302 LM399H

Commit message: PCB layout
Parts:
- added C302: 100n, Capacitor_SMD:C_0402_1005Metric_Pad0.74x0.62mm_HandSolder, symbol Device:C
- added R310: 6k95/.05%, Resistor_SMD:R_0603_1608Metric_Pad0.98x0.95mm_HandSolder, symbol Device:R
- added R311, R312: 3k01/.1%, Resistor_SMD:R_0603_1608Metric_Pad0.98x0.95mm_HandSolder, symbol Device:R
- added R313: 0, Resistor_SMD:R_0603_1608Metric_Pad0.98x0.95mm_HandSolder, symbol Device:R
- added U303: OPA177, Package_SO:SOIC-8_3.9x4.9mm_P1.27mm, symbol ETH3CDAQ1:OPA177
Connections:
- net -14VF: now also C302.2, U303.4 (V-)
- net AGNDF: now also C302.1, R310.2, U303.7 (V+)
- net VREF_N7V: no longer names the net of R307.1, R309.2, U302.2
- net VREF_N7V: now also R311.2, U303.3 (+)
- new net: R310.1, R312.2, U303.2 (-)
- new net: R311.1, R312.1, R313.2, U303.6
- new net +10VRF: R313.1
- no-connect marks 0 -> 2
Changed lines of the file:
@@
 $Descr A4 11693 8268
 encoding utf-8
-Sheet 3 13
+Sheet 3 15
 Title ""
 Date ""
@@
 $EndComp
 Wire Wire Line
-	7000 3600 7450 3600
+	7000 3600 7200 3600
 $Comp
 L ETH3CDAQ1:+18VF #PWR?
@@
 	1    0    0    -1
 $EndComp
-Wire Wire Line
-	6350 2850 7450 2850
 Connection ~ 6350 3600
 Wire Wire Line
@@
 Wire Wire Line
 	5400 2850 6350 2850
-Connection ~ 6350 2850
 Wire Wire Line
 	6350 2850 6350 3600
-Text HLabel 7450 2850 2    50   Output ~ 0
-VREF_N7V
-Text HLabel 7450 3600 2    50   Output ~ 0
+Text HLabel 7200 3600 2    50   Output ~ 0
 VREF_N7V_LPF
 $Comp
@@
 Wire Wire Line
 	4750 3950 4250 3950
+$Comp
+L ETH3CDAQ1:OPA177 U303
+U 1 1 5FF6771B
+P 9050 2950
+F 0 "U303" H 9200 3200 50  0000 L CNN
+F 1 "OPA177" H 9100 3100 50  0000 L CNN
+F 2 "Package_SO:SOIC-8_3.9x4.9mm_P1.27mm" H 9100 3000 50  0001 C CNN
+F 3 "" H 9100 3100 50  0001 C CNN
+	1    9050 2950
+	1    0    0    -1
+$EndComp
+$Comp
+L ETH3CDAQ1:AGNDF #PWR?
+U 1 1 5FF6AD62
+P 8950 2650
+AR Path="/5FF6AD62" Ref="#PWR?"  Part="1"
+AR Path="/5FCCC067/5FF6AD62" Ref="#PWR?"  Part="1"
+AR Path="/5FD74AB8/5FF6AD62" Ref="#PWR?"  Part="1"
+AR Path="/600E050E/5FF6AD62" Ref="#PWR0310"  Part="1"
+F 0 "#PWR0310" H 8950 2400 50  0001 C CNN
+F 1 "AGNDF" H 8955 2477 50  0000 C CNN
+F 2 "" H 8950 2650 50  0001 C CNN
+F 3 "" H 8950 2650 50  0001 C CNN
+	1    8950 2650
+	-1   0    0    1
+$EndComp
+NoConn ~ 9050 2650
+NoConn ~ 9050 3250
+$Comp
+L ETH3CDAQ1:-14VF #PWR?
+U 1 1 5FF6D953
+P 8950 3450
+AR Path="/5FF6D953" Ref="#PWR?"  Part="1"
+AR Path="/5FCCC067/5FF6D953" Ref="#PWR?"  Part="1"
+AR Path="/5FD74AB8/5FF6D953" Ref="#PWR?"  Part="1"
+AR Path="/600E050E/5FF6D953" Ref="#PWR0311"  Part="1"
+F 0 "#PWR0311" H 8950 3300 50  0001 C CNN
+F 1 "-14VF" H 8965 3623 50  0000 C CNN
+F 2 "" H 8950 3450 50  0001 C CNN
+F 3 "" H 8950 3450 50  0001 C CNN
+	1    8950 3450
+	-1   0    0    1
+$EndComp
+$Comp
+L Device:R R310
+U 1 1 5FF70775
+P 8100 3250
+F 0 "R310" H 8170 3296 50  0000 L CNN
+F 1 "6k95/.05%" H 8170 3205 50  0000 L CNN
+F 2 "Resistor_SMD:R_0603_1608Metric_Pad0.98x0.95mm_HandSolder" V 8030 3250 50  0001 C CNN
+F 3 "~" H 8100 3250 50  0001 C CNN
+	1    8100 3250
+	1    0    0    -1
+$EndComp
+Wire Wire Line
+	8100 3050 8100 3100
+$Comp
+L Device:R R312
+U 1 1 5FF78E6B
+P 9000 4000
+F 0 "R312" V 8793 4000 50  0000 C CNN
+F 1 "3k01/.1%" V 8884 4000 50  0000 C CNN
+F 2 "Resistor_SMD:R_0603_1608Metric_Pad0.98x0.95mm_HandSolder" V 8930 4000 50  0001 C CNN
+F 3 "~" H 9000 4000 50  0001 C CNN
+	1    9000 4000
+	0    1    1    0
+$EndComp
+Wire Wire Line
+	8850 4000 8700 4000
+$Comp
+L Device:R R311
+U 1 1 5FF7B73D
+P 9000 2250
+F 0 "R311" V 8793 2250 50  0000 C CNN
+F 1 "3k01/.1%" V 8884 2250 50  0000 C CNN
+F 2 "Resistor_SMD:R_0603_1608Metric_Pad0.98x0.95mm_HandSolder" V 8930 2250 50  0001 C CNN
+F 3 "~" H 9000 2250 50  0001 C CNN
+	1    9000 2250
+	0    1    1    0
+$EndComp
+Wire Wire Line
+	8850 2250 8700 2250
+Wire Wire Line
+	8700 2250 8700 2850
+Wire Wire Line
+	8700 2850 8750 2850
+Wire Wire Line
+	9150 2250 9750 2250
+Wire Wire Line
+	9750 2250 9750 2950
+$Comp
+L Device:R R313
+U 1 1 5FF7E462
+P 9950 2950
+F 0 "R313" V 9743 2950 50  0000 C CNN
+F 1 "0" V 9834 2950 50  0000 C CNN
+F 2 "Resistor_SMD:R_0603_1608Metric_Pad0.98x0.95mm_HandSolder" V 9880 2950 50  0001 C CNN
+F 3 "~" H 9950 2950 50  0001 C CNN
+	1    9950 2950
+	0    1    1    0
+$EndComp
+$Comp
+L ETH3CDAQ1:AGNDF #PWR?
+U 1 1 5FF802F9
+P 8100 3450
+AR Path="/5FF802F9" Ref="#PWR?"  Part="1"
+AR Path="/5FCCC067/5FF802F9" Ref="#PWR?"  Part="1"
+AR Path="/5FD74AB8/5FF802F9" Ref="#PWR?"  Part="1"
+AR Path="/600E050E/5FF802F9" Ref="#PWR0309"  Part="1"
+F 0 "#PWR0309" H 8100 3200 50  0001 C CNN
+F 1 "AGNDF" H 8105 3277 50  0000 C CNN
+F 2 "" H 8100 3450 50  0001 C CNN
+F 3 "" H 8100 3450 50  0001 C CNN
+	1    8100 3450
+	1    0    0    -1
+$EndComp
+Wire Wire Line
+	8100 3450 8100 3400
+$Comp
+L ETH3CDAQ1:+10VRF #PWR0313
+U 1 1 5FF84F41
+P 10100 2950
+F 0 "#PWR0313" H 10100 2800 50  0001 C CNN
+F 1 "+10VRF" V 10100 3100 50  0000 L CNN
+F 2 "" H 10100 2950 50  0001 C CNN
+F 3 "" H 10100 2950 50  0001 C CNN
+	1    10100 2950
+	0    1    1    0
+$EndComp
+Wire Wire Line
+	8100 3050 8700 3050
+$Comp
+L Device:C C302
+U 1 1 5FF8EAC9
+P 9300 3400
+F 0 "C302" V 9048 3400 50  0000 C CNN
+F 1 "100n" V 9139 3400 50  0000 C CNN
+F 2 "Capacitor_SMD:C_0402_1005Metric_Pad0.74x0.62mm_HandSolder" H 9338 3250 50  0001 C CNN
+F 3 "~" H 9300 3400 50  0001 C CNN
+	1    9300 3400
+	0    1    1    0
+$EndComp
+$Comp
+L ETH3CDAQ1:AGNDF #PWR?
+U 1 1 5FF98DDC
+P 9450 3400
+AR Path="/5FF98DDC" Ref="#PWR?"  Part="1"
+AR Path="/5FCCC067/5FF98DDC" Ref="#PWR?"  Part="1"
+AR Path="/5FD74AB8/5FF98DDC" Ref="#PWR?"  Part="1"
+AR Path="/600E050E/5FF98DDC" Ref="#PWR0312"  Part="1"
+F 0 "#PWR0312" H 9450 3150 50  0001 C CNN
+F 1 "AGNDF" H 9455 3227 50  0000 C CNN
+F 2 "" H 9450 3400 50  0001 C CNN
+F 3 "" H 9450 3400 50  0001 C CNN
+	1    9450 3400
+	0    -1   -1   0
+$EndComp
+Wire Wire Line
+	9150 3400 8950 3400
+Wire Wire Line
+	8950 3400 8950 3250
+Wire Wire Line
+	8950 3450 8950 3400
+Connection ~ 8950 3400
+Wire Wire Line
+	9350 2950 9750 2950
+Wire Wire Line
+	8700 3050 8700 4000
+Connection ~ 8700 3050
+Wire Wire Line
+	8700 3050 8750 3050
+Wire Wire Line
+	9750 4000 9750 2950
+Wire Wire Line
+	9150 4000 9750 4000
+Connection ~ 9750 2950
+Wire Wire Line
+	9800 2950 9750 2950
+Wire Wire Line
+	8700 2850 6350 2850
+Connection ~ 8700 2850
+Connection ~ 6350 2850
 $EndSCHEMATC
